Commit message: added the lower leg joint, not entirely complete

File: urdfs/leg.gazebo.xacro (robot description, xacro)
@@ -3,4 +3,10 @@
         <xacro:macro name="leg_gazebo" params="name robot_name">
         	 <gazebo reference="${name}_bs_joint">
+                        <provideFeedback>true</provideFeedback>
+                 </gazebo>
+                 <gazebo reference="${name}_upper_leg_joint">
+                        <provideFeedback>true</provideFeedback>
+                 </gazebo>
+                 <gazebo reference="${name}_lower_leg_joint">
                         <provideFeedback>true</provideFeedback>
                  </gazebo>

File: urdfs/leg.transmission.xacro (robot description, xacro)
@@ -13,4 +13,26 @@
                         </actuator>
                 </transmission>
+         <!-- Upper leg -->
+                <transmission name="${name}_upper_leg_joint_trans">
+                        <type>transmission_interface/SimpleTransmission</type>
+                        <joint name="${name}_upper_leg_joint">
+                                <hardwareInterface>hardware_interface/EffortJointInterface</hardwareInterface>
+                        </joint>
+                        <actuator name="${name}_upper_leg_joint_motor">
+                                <hardwareInterface>hardware_interface/EffortJointInterface</hardwareInterface>
+                                <mechanicalReduction>1</mechanicalReduction>
+                        </actuator>
+                </transmission>
+         <!-- Lower leg -->
+                <transmission name="${name}_lower_leg_joint_trans">
+                        <type>transmission_interface/SimpleTransmission</type>
+                        <joint name="${name}_lower_leg_joint">
+                                <hardwareInterface>hardware_interface/EffortJointInterface</hardwareInterface>
+                        </joint>
+                        <actuator name="${name}_lower_leg_joint_motor">
+                                <hardwareInterface>hardware_interface/EffortJointInterface</hardwareInterface>
+                                <mechanicalReduction>1</mechanicalReduction>
+                        </actuator>
+                </transmission>
         </xacro:macro>
 </robot>

File: urdfs/leg.xacro (robot description, xacro)
@@ -7,4 +7,8 @@
     <xacro:property name="MAX_TORQUE" value="0" />
     <xacro:property name="VELOCITY" value="0" />
+    <xacro:property name="UPPER_LEG" value="0.15312" />
+    <xacro:property name="LOWER_LEG_x" value="0.22546" />
+    <xacro:property name="LOWER_LEG_y" value="0.00035" />
+    <xacro:property name="LOWER_LEG_z" value="2e-05" />
     <!-- This macro has for purpose to define a leg -->
     <xacro:macro name="leg" params="name parent is_front is_right robot_name *origin">
@@ -88,5 +92,5 @@
                         </xacro:if>
                     </xacro:unless>
-	                <material name="shoulder_collision_color">
+	                <material name="collision_color">
       				<color rgba="0.8 0.8 0.8 1.0"/>
     			</material>
@@ -99,4 +103,261 @@
 	            </inertial>
 	        </link>
+	     <!--UPPER LEG JOINT-->
+            <joint name="${name}_upper_leg_joint" type="revolute">
+                <parent link="${name}_shoulder"/>
+                <child link="${name}_upperleg"/>
+                <xacro:insert_block name="origin"/>
+                <!-- joints rotates around the y-axis -->
+                <!-- limit and placement of the joint -->
+                <xacro:if value="${is_front}">
+                    <xacro:unless value="${is_right}">
+                        <!-- LF_UPPER_LEG_JOINT -->
+                        <axis xyz="0 1 0"/>
+                        <limit effort="${MAX_TORQUE}" lower="-3.14" upper="3.14" velocity="${VELOCITY}"/>
+                        <origin xyz="-${UPPER_LEG} 0 0" rpy="0 0 0" />
+                    </xacro:unless>
+                    <xacro:if value="${is_right}">
+                        <!-- RF_UPPER_LEG_JOINT -->
+                        <axis xyz="-1 0 0"/>
+			<limit effort="${MAX_TORQUE}" lower="-3.14" upper="3.14" velocity="${VELOCITY}"/>
+                        <origin xyz="0 -${UPPER_LEG} 0" rpy="0 0 0" />
+                    </xacro:if>
+                </xacro:if>
+                <xacro:unless value="${is_front}">
+                    <xacro:unless value="${is_right}">
+                        <!-- LH_UPPER_LEG_JOINT -->
+                        <axis xyz="1 0 0"/>
+			<limit effort="${MAX_TORQUE}" lower="-3.14" upper="3.14" velocity="${VELOCITY}"/>
+                        <origin xyz="0 ${UPPER_LEG} 0" rpy="0 0 0" />
+                    </xacro:unless>
+                    <xacro:if value="${is_right}">
+                        <!-- RF_UPPER_LEG_JOINT -->
+                        <axis xyz="0 -1 0"/>
+			<limit effort="${MAX_TORQUE}" lower="-3.14" upper="3.14" velocity="${VELOCITY}"/>
+                        <origin xyz="${UPPER_LEG} 0 0" rpy="0 0 0" />
+                    </xacro:if>
+                </xacro:unless>
+                <!-- pybullet simulation parameters -->
+                <dynamics damping="0.0" friction="0.0"/>
+            </joint>
+	  <!-- UPPER LEG ASSEMBLY -->
+            <link name="${name}_upperleg">
+            	<!--VISUAL-->
+	        <visual>
+	            <origin xyz="0 0 0" rpy="0 0 0" />
+                    <xacro:if value="${is_front}">
+                        <xacro:unless value="${is_right}">
+                            <!-- LF UPPER_LEG -->
+                        	<geometry>
+                        	    <mesh filename="package://starbot_description/meshes/stl/upper_leg.stl"/>
+                        	</geometry>
+                        </xacro:unless>
+                        <xacro:if value="${is_right}">
+                            <!-- RF UPPER_LEG-->
+                        	<geometry>
+                        	    <mesh filename="package://starbot_description/meshes/stl/upper_leg.001.stl"/>
+                        	</geometry>
+                        </xacro:if>
+                    </xacro:if>
+                    <xacro:unless value="${is_front}">
+                        <xacro:unless value="${is_right}">
+                            <!-- LH UPPER_LEG -->
+                        	<geometry>
+                        	    <mesh filename="package://starbot_description/meshes/stl/upper_leg.002.stl"/>
+                        	</geometry>
+                        </xacro:unless>
+                        <xacro:if value="${is_right}">
+                            <!-- RH UPPER_LEG -->
+                        	<geometry>
+                        	    <mesh filename="package://starbot_description/meshes/stl/upper_leg.003.stl"/>
+                        	</geometry>
+                        </xacro:if>
+                    </xacro:unless>
+	                <material name="upper_leg_color">
+                    		<color rgba="0.8 0.8 0.8 1.0"/>
+                	</material>
+	            </visual>
+	            <!--COLLISION-->
+	            <collision>
+	            <origin xyz="0 0 0" rpy="0 0 0" />
+                    <xacro:if value="${is_front}">
+                        <xacro:unless value="${is_right}">
+                            <!-- LF UPPER_LEG -->
+                        	<geometry>
+                        	    <box size="0.30016 0.07002 0.0707"/>
+                        	</geometry>
+                        </xacro:unless>
+                        <xacro:if value="${is_right}">
+                            <!-- RF UPPER_LEG -->
+                        	<geometry>
+                        	    <box size="0.07002 0.30016 0.0707"/>
+                        	</geometry>
+                        </xacro:if>
+                    </xacro:if>
+                    <xacro:unless value="${is_front}">
+                        <xacro:unless value="${is_right}">
+                            <!-- LH UPPER_LEG -->
+                        	<geometry>
+                        	    <box size="0.07002 0.30016 0.0707"/>
+                        	</geometry>
+                        </xacro:unless>
+                        <xacro:if value="${is_right}">
+                            <!-- RH UPPER_LEG-->
+                        	<geometry>
+                        	    <box size="0.30016 0.07002 0.0707"/>
+                        	</geometry>
+                        </xacro:if>
+                    </xacro:unless>
+	                <material name="collision_color">
+      				<color rgba="0.8 0.8 0.8 1.0"/>
+    			</material>
+	            </collision>
+	            <!-- UPPER LEG LINK INERTIAL -->
+            	<xacro:unless value="${is_right}">
+                <!-- Left upper leg inertia -->
+                <inertial>
+                     <origin xyz="0 0 0" rpy="0 0 0"/>
+                    <mass value="2.3"/>
+                    <inertia ixx="0.00148" ixy="0" ixz="0" iyy="0.01286" iyz="0" izz="0.01286"/>
+                </inertial>
+            	</xacro:unless>
+            	<xacro:if value="${is_right}">
+            	<!-- Right upper leg inertia -->
+                <inertial>
+                     <origin xyz="0 0 0" rpy="0 0 0"/>
+                    <mass value="2.3"/>
+                    <inertia ixx="0.01259" ixy="0" ixz="0" iyy="0.00147" iyz="0" izz="0.01259"/>
+                </inertial>
+            	</xacro:if>
+	        </link>
+	     <!--LOWER LEG JOINT-->
+            <joint name="${name}_lower_leg_joint" type="prismatic">
+                <parent link="${name}_upperleg"/>
+                <child link="${name}_lowerleg"/>
+                <xacro:insert_block name="origin"/>
+                <!-- joints rotates around the x-axis -->
+                <!-- limit and placement of the joint -->
+                <xacro:if value="${is_front}">
+                    <xacro:unless value="${is_right}">
+                        <!-- LF_LOWER_LEG_JOINT -->
+                        <axis xyz="1 0 0"/>
+                        <limit effort="${MAX_TORQUE}" lower="-3.14" upper="3.14" velocity="${VELOCITY}"/>
+                        <origin xyz="${LOWER_LEG_x} -${LOWER_LEG_y} -${LOWER_LEG_z}" rpy="0 0 0" />
+                    </xacro:unless>
+                    <xacro:if value="${is_right}">
+                    	<axis xyz="0 1 0"/>
+                        <!-- RF_LOWER_LEG_JOINT -->
+			<limit effort="${MAX_TORQUE}" lower="-3.14" upper="3.14" velocity="${VELOCITY}"/>
+                        <origin xyz="${LOWER_LEG_y} ${LOWER_LEG_x} -${LOWER_LEG_z}" rpy="0 0 0" />
+                    </xacro:if>
+                </xacro:if>
+                <xacro:unless value="${is_front}">
+                    <xacro:unless value="${is_right}">
+                    	<axis xyz="0 -1 0"/>
+                        <!-- LH_LOWER_LEG_JOINT -->
+			<limit effort="${MAX_TORQUE}" lower="-3.14" upper="3.14" velocity="${VELOCITY}"/>
+                        <origin xyz="${LOWER_LEG_y} -${LOWER_LEG_x} -${LOWER_LEG_z}" rpy="0 0 0" />
+                    </xacro:unless>
+                    <xacro:if value="${is_right}">
+                        <!-- RF_LOWER_LEG_JOINT -->
+                        <axis xyz="-1 0 0"/>
+			<limit effort="${MAX_TORQUE}" lower="-3.14" upper="3.14" velocity="${VELOCITY}"/>
+                        <origin xyz="-${LOWER_LEG_x} -${LOWER_LEG_y} -${LOWER_LEG_z}" rpy="0 0 0" />
+                    </xacro:if>
+                </xacro:unless>
+                <!-- pybullet simulation parameters -->
+                <dynamics damping="0.0" friction="0.0"/>
+            </joint>
+	  <!-- LOWER LEG ASSEMBLY -->
+            <link name="${name}_lowerleg">
+            	<!--VISUAL-->
+	        <visual>
+	            <origin xyz="0 0 0" rpy="0 0 0" />
+                    <xacro:if value="${is_front}">
+                        <xacro:unless value="${is_right}">
+                            <!-- LF LOWER_LEG -->
+                            <!--we need mesh geometry otherwise strange behaviour happens-->
+                        	<geometry>
+                        	    <mesh filename="package://starbot_description/meshes/stl/upper_leg.stl" scale="0.7 0.7 0.7"/>
+                        	</geometry>
+                        </xacro:unless>
+                        <xacro:if value="${is_right}">
+                            <!-- RF LOWER_LEG-->
+                        	<geometry>
+                        	    <mesh filename="package://starbot_description/meshes/stl/upper_leg.001.stl" scale="0.7 0.7 0.7"/>
+                        	</geometry>
+                        </xacro:if>
+                    </xacro:if>
+                    <xacro:unless value="${is_front}">
+                        <xacro:unless value="${is_right}">
+                            <!-- LH LOWER_LEG -->
+                        	<geometry>
+                        	    <mesh filename="package://starbot_description/meshes/stl/upper_leg.002.stl" scale="0.7 0.7 0.7"/>
+                        	</geometry>
+                        </xacro:unless>
+                        <xacro:if value="${is_right}">
+                            <!-- RH LOWER_LEG -->
+                        	<geometry>
+                        	    <mesh filename="package://starbot_description/meshes/stl/upper_leg.003.stl" scale="0.7 0.7 0.7"/>
+                        	</geometry>
+                        </xacro:if>
+                    </xacro:unless>
+	                <material name="upper_leg_color">
+                    		<color rgba="0.3 0.3 0.6 1.0"/>
+                	</material>
+	            </visual>
+	            <!--COLLISION-->
+	            <collision>
+	            <origin xyz="0 0 0" rpy="0 0 0" />
+                    <xacro:if value="${is_front}">
+                        <xacro:unless value="${is_right}">
+                            <!-- LF LOWER_LEG -->
+                        	<geometry>
+                        	    <box size="0.25009 0.04058 0.04002"/>
+                        	</geometry>
+                        </xacro:unless>
+                        <xacro:if value="${is_right}">
+                            <!-- RF LOWER_LEG -->
+                        	<geometry>
+                        	    <box size="0.04058 0.25009 0.04002"/>
+                        	</geometry>
+                        </xacro:if>
+                    </xacro:if>
+                    <xacro:unless value="${is_front}">
+                        <xacro:unless value="${is_right}">
+                            <!-- LH LOWER_LEG -->
+                        	<geometry>
+                        	     <box size="0.04058 0.25009 0.04002"/>
+                        	</geometry>
+                        </xacro:unless>
+                        <xacro:if value="${is_right}">
+                            <!-- RH LOWER_LEG-->
+                        	<geometry>
+                        	    <box size="0.25009 0.04058 0.04002"/>
+                        	</geometry>
+                        </xacro:if>
+                    </xacro:unless>
+	                <material name="collision_color">
+      				<color rgba="0.8 0.8 0.8 1.0"/>
+    			</material>
+	            </collision>
+	            <!-- LOWER LEG LINK INERTIAL -->
+            	<xacro:unless value="${is_right}">
+                <!-- Left upper leg inertia -->
+                <inertial>
+                    <origin xyz="0 0 0" rpy="0 0 0"/>
+        	    <mass value="2.36"/>
+        	    <inertia ixx="0.00954" ixy="0" ixz="0" iyy="0.00954" iyz="0" izz="0.01845"/>
+                </inertial>
+            	</xacro:unless>
+            	<xacro:if value="${is_right}">
+            	<!-- Right upper leg inertia -->
+                <inertial>
+                     <origin xyz="0 0 0" rpy="0 0 0"/>
+        	     <mass value="2.36"/>
+        	     <inertia ixx="0.00056" ixy="0" ixz="0" iyy="0.00056" iyz="0" izz="0.00049"/>
+                </inertial>
+            	</xacro:if>
+	        </link>
         <!-- Extensions -->
         <xacro:leg_transmission name="${name}"/>
