Commit message: add joint pew_wheel

File: urdfs/leg.gazebo.xacro (robot description, xacro)
@@ -11,4 +11,7 @@
                         <provideFeedback>true</provideFeedback>
                  </gazebo>
+                <gazebo reference="${name}_pre_wheel_joint">
+                        <provideFeedback>true</provideFeedback>
+                </gazebo>
 		 <!-- HERE WE HAVE FOOT SENSOR AND FRICTION PROPERTIES -->
                  <gazebo reference="${name}_foot">

File: urdfs/leg.transmission.xacro (robot description, xacro)
@@ -35,4 +35,15 @@
                         </actuator>
                 </transmission>
+        <!-- Pre wheel -->
+                <transmission name="${name}_pre_wheel_joint_trans">
+                        <type>transmission_interface/SimpleTransmission</type>
+                        <joint name="${name}_pre_wheel_joint">
+                                <hardwareInterface>hardware_interface/EffortJointInterface</hardwareInterface>
+                        </joint>
+                        <actuator name="${name}_pre_wheel_joint_motor">
+                                <hardwareInterface>hardware_interface/EffortJointInterface</hardwareInterface>
+                                <mechanicalReduction>1</mechanicalReduction>
+                        </actuator>
+                </transmission>
         </xacro:macro>
 </robot>

File: urdfs/leg.xacro (robot description, xacro)
@@ -11,4 +11,5 @@
     <xacro:property name="LOWER_LEG_y" value="0.00035" />
     <xacro:property name="LOWER_LEG_z" value="2e-05" />
+    <xacro:property name="PRE_WHEEL" value="0.10183" />
     <!-- This macro has for purpose to define a leg -->
     <xacro:macro name="leg" params="name parent is_front is_right robot_name *origin">
@@ -360,4 +361,133 @@
             	</xacro:if>
 	        </link>
+        <!--PRE WHEEL JOINT-->
+            <joint name="${name}_pre_wheel_joint" type="revolute">
+                <parent link="${name}_lowerleg"/>
+                <child link="${name}_pre_wheel"/>
+                <xacro:insert_block name="origin"/>
+                <!-- joints rotates around the x-axis (refer to the x-axis align leg) -->
+                <!-- limit and placement of the joint -->
+                <xacro:if value="${is_front}">
+                    <xacro:unless value="${is_right}">
+                        <!-- LF_PRE_WHEEL_JOINT -->
+                        <axis xyz="1 0 0"/>
+                        <limit effort="${MAX_TORQUE}" lower="-3.14" upper="3.14" velocity="${VELOCITY}"/>
+                        <origin xyz="0 ${PRE_WHEEL} 0" rpy="0 0 0" />
+                    </xacro:unless>
+                    <xacro:if value="${is_right}">
+                    	<axis xyz="0 1 0"/>
+                        <!-- RF_PRE_WHEEL_JOINT -->
+			<limit effort="${MAX_TORQUE}" lower="-3.14" upper="3.14" velocity="${VELOCITY}"/>
+                        <origin xyz="${PRE_WHEEL} 0 0" rpy="0 0 0" />
+                    </xacro:if>
+                </xacro:if>
+                <xacro:unless value="${is_front}">
+                    <xacro:unless value="${is_right}">
+                    	<axis xyz="0 -1 0"/>
+                        <!-- LH_PRE_WHEEL_JOINT -->
+			<limit effort="${MAX_TORQUE}" lower="-3.14" upper="3.14" velocity="${VELOCITY}"/>
+                        <origin xyz="$-{PRE_WHEEL} 0 0" rpy="0 0 0" />
+                    </xacro:unless>
+                    <xacro:if value="${is_right}">
+                        <!-- RF_PRE_WHEEL_JOINT -->
+                        <axis xyz="-1 0 0"/>
+			<limit effort="${MAX_TORQUE}" lower="-3.14" upper="3.14" velocity="${VELOCITY}"/>
+                        <origin xyz="0 -${PRE_WHEEL} 0" rpy="0 0 0" />
+                    </xacro:if>
+                </xacro:unless>
+                <!-- pybullet simulation parameters -->
+                <dynamics damping="0.0" friction="0.0"/>
+            </joint>
+	  <!-- PRE WHEEL ASSEMBLY -->
+            <link name="${name}_pre_wheel">
+            	<!--VISUAL-->
+	        <visual>
+	            <origin xyz="0 0 0" rpy="0 0 0" />
+                    <xacro:if value="${is_front}">
+                        <xacro:unless value="${is_right}">
+                            <!-- LF PRE_WHEEL -->
+                            <!--we need mesh geometry otherwise strange behaviour happens-->
+                        	<geometry>
+                        	    <mesh filename="package://starbot_description/meshes/stl/upper_leg_y.stl" scale = "0.5 0.5 0.5"/>
+                        	</geometry>
+                        </xacro:unless>
+                        <xacro:if value="${is_right}">
+                            <!-- RF PRE_WHEEL-->
+                        	<geometry>
+                        	    <mesh filename="package://starbot_description/meshes/stl/upper_leg_x.stl" scale = "0.5 0.5 0.5"/>
+                        	</geometry>
+                        </xacro:if>
+                    </xacro:if>
+                    <xacro:unless value="${is_front}">
+                        <xacro:unless value="${is_right}">
+                            <!-- LH PRE_WHEEL -->
+                        	<geometry>
+                        	    <mesh filename="package://starbot_description/meshes/stl/upper_leg_nx.stl" scale = "0.5 0.5 0.5"/>
+                        	</geometry>
+                        </xacro:unless>
+                        <xacro:if value="${is_right}">
+                            <!-- RH PRE_WHEEL -->
+                        	<geometry>
+                        	    <mesh filename="package://starbot_description/meshes/stl/upper_leg_ny.stl" scale = "0.5 0.5 0.5"/>
+                        	</geometry>
+                        </xacro:if>
+                    </xacro:unless>
+	                <material name="upper_leg_color">
+                    		<color rgba="0.3 0.3 0.6 1.0"/>
+                	</material>
+	            </visual>
+            <!--COLLISION-->
+	            <collision>
+	            <origin xyz="0 0 0" rpy="0 0 0" />
+                    <xacro:if value="${is_front}">
+                        <xacro:unless value="${is_right}">
+                            <!-- LF PRE_WHEEL -->
+                        	<geometry>
+                        	    <mesh filename="package://starbot_description/meshes/stl/upper_leg_ny.stl" scale = "0.5 0.5 0.5"/>
+                        	</geometry>
+                        </xacro:unless>
+                        <xacro:if value="${is_right}">
+                            <!-- RF PRE_WHEEL -->
+                        	<geometry>
+                        	    <mesh filename="package://starbot_description/meshes/stl/upper_leg_ny.stl" scale = "0.5 0.5 0.5"/>
+                        	</geometry>
+                        </xacro:if>
+                    </xacro:if>
+                    <xacro:unless value="${is_front}">
+                        <xacro:unless value="${is_right}">
+                            <!-- LH PRE_WHEEL -->
+                        	<geometry>
+                        	     <mesh filename="package://starbot_description/meshes/stl/upper_leg_ny.stl" scale = "0.5 0.5 0.5"/>
+                        	</geometry>
+                        </xacro:unless>
+                        <xacro:if value="${is_right}">
+                            <!-- RH PRE_WHEEL-->
+                        	<geometry>
+                        	    <mesh filename="package://starbot_description/meshes/stl/upper_leg_ny.stl" scale = "0.5 0.5 0.5"/>
+                        	</geometry>
+                        </xacro:if>
+                    </xacro:unless>
+	                <material name="collision_color">
+      				<color rgba="0.8 0.8 0.8 1.0"/>
+    			</material>
+	            </collision>
+	            <!-- PRE WHEEL LINK INERTIAL -->
+            	<xacro:unless value="${is_right}">
+                <!-- Left pre_wheel inertia -->
+                <inertial>
+                    <origin xyz="0 0 0" rpy="0 0 0"/>
+                    <mass value="0.66"/>
+                    <inertia ixx="0.00015" ixy="0" ixz="0" iyy="0.00015" iyz="0" izz="0.00013"/>
+                </inertial>
+            	</xacro:unless>
+            	<xacro:if value="${is_right}">
+            	<!-- Right pre_wheel inertia -->
+                <inertial>
+                     <origin xyz="0 0 0" rpy="0 0 0"/>
+                    <mass value="0.66"/>
+                    <inertia ixx="0.00029" ixy="0" ixz="0" iyy="0.00029" iyz="0" izz="0.00041"/>
+                </inertial>
+            	</xacro:if>
+	        </link>
         <!-- Extensions -->
         <xacro:leg_transmission name="${name}"/>

Commit message: add wheel joint and link

File: urdfs/leg.gazebo.xacro (robot description, xacro)
@@ -1,41 +1,44 @@
 <?xml version="1.0"?>
 <robot xmlns:xacro="http://ros.org/wiki/xacro">
-        <xacro:macro name="leg_gazebo" params="name robot_name">
-        	 <gazebo reference="${name}_bs_joint">
-                        <provideFeedback>true</provideFeedback>
-                 </gazebo>
-                 <gazebo reference="${name}_upper_leg_joint">
-                        <provideFeedback>true</provideFeedback>
-                 </gazebo>
-                 <gazebo reference="${name}_lower_leg_joint">
-                        <provideFeedback>true</provideFeedback>
-                 </gazebo>
-                <gazebo reference="${name}_pre_wheel_joint">
-                        <provideFeedback>true</provideFeedback>
-                </gazebo>
-		 <!-- HERE WE HAVE FOOT SENSOR AND FRICTION PROPERTIES -->
-                 <gazebo reference="${name}_foot">
-                        <kp>1000000.0</kp>
-                        <kd>100.0</kd>
-                        <mu1>0.8</mu1>
-                        <mu2>0.8</mu2>
-                        <maxVel>1.0</maxVel>
-                        <maxContacts>1</maxContacts>
-                        <sensor name="${name}_foot_contact_sensor" type="contact">
-                                <always_on>true</always_on>
-                                <update_rate>1000.0</update_rate>
-                                <contact>
-                                        <collision>${name}_XXXX</collision>
-                                </contact>
-                                <!-- the sensor readings in terms of force torques are expressed in the lowerleg frame
-                                because gazebo lumps the fake footframe with the real parent link, the normals are in the world frame-->
-                                <plugin name="${name}_foot_bumper" filename="libgazebo_ros_bumper.so">
-                                        <bumperTopicName>/${robot_name}/${name}_foot_bumper</bumperTopicName>
-                                        <!--robotNamespace>solo</robotNamespace-->
-                                        <frameName>${name}_foot</frameName>
-                                </plugin>
-                        </sensor>
-                        <material>Gazebo/Black</material>
-                </gazebo>
-        </xacro:macro>
+    <xacro:macro name="leg_gazebo" params="name robot_name">
+        <gazebo reference="${name}_bs_joint">
+            <provideFeedback>true</provideFeedback>
+        </gazebo>
+        <gazebo reference="${name}_upper_leg_joint">
+            <provideFeedback>true</provideFeedback>
+        </gazebo>
+        <gazebo reference="${name}_lower_leg_joint">
+            <provideFeedback>true</provideFeedback>
+        </gazebo>
+        <gazebo reference="${name}_pre_wheel_joint">
+            <provideFeedback>true</provideFeedback>
+        </gazebo>
+        <gazebo reference="${name}_wheel_joint">
+            <provideFeedback>true</provideFeedback>
+        </gazebo>
+        <!-- HERE WE HAVE FOOT SENSOR AND FRICTION PROPERTIES -->
+        <gazebo reference="${name}_foot">
+            <kp>1000000.0</kp>
+            <kd>100.0</kd>
+            <mu1>0.8</mu1>
+            <mu2>0.8</mu2>
+            <maxVel>1.0</maxVel>
+            <maxContacts>1</maxContacts>
+            <sensor name="${name}_foot_contact_sensor" type="contact">
+                <always_on>true</always_on>
+                <update_rate>1000.0</update_rate>
+                <contact>
+                    <collision>${name}_XXXX</collision>
+                </contact>
+                <!-- the sensor readings in terms of force torques are expressed in the lowerleg frame
+                because gazebo lumps the fake footframe with the real parent link, the normals are in the world frame-->
+                <plugin name="${name}_foot_bumper" filename="libgazebo_ros_bumper.so">
+                    <bumperTopicName>/${robot_name}/${name}_foot_bumper</bumperTopicName>
+                    <!--robotNamespace>solo</robotNamespace-->
+                    <frameName>${name}_foot</frameName>
+                </plugin>
+            </sensor>
+            <material>Gazebo/Black</material>
+        </gazebo>
+    </xacro:macro>
 </robot>

File: urdfs/leg.transmission.xacro (robot description, xacro)
@@ -2,5 +2,5 @@
 <robot xmlns:xacro="http://ros.org/wiki/xacro">
         <xacro:macro name="leg_transmission" params="name">
-        <!-- body_shoulder joint -->
+                <!-- body_shoulder joint -->
                 <transmission name="${name}_bs_joint_trans">
                         <type>transmission_interface/SimpleTransmission</type>
@@ -13,5 +13,5 @@
                         </actuator>
                 </transmission>
-         <!-- Upper leg -->
+                <!-- Upper leg -->
                 <transmission name="${name}_upper_leg_joint_trans">
                         <type>transmission_interface/SimpleTransmission</type>
@@ -24,5 +24,5 @@
                         </actuator>
                 </transmission>
-         <!-- Lower leg -->
+                <!-- Lower leg -->
                 <transmission name="${name}_lower_leg_joint_trans">
                         <type>transmission_interface/SimpleTransmission</type>
@@ -35,5 +35,5 @@
                         </actuator>
                 </transmission>
-        <!-- Pre wheel -->
+                <!-- Pre wheel -->
                 <transmission name="${name}_pre_wheel_joint_trans">
                         <type>transmission_interface/SimpleTransmission</type>
@@ -46,4 +46,15 @@
                         </actuator>
                 </transmission>
+                <!-- Wheel -->
+                <transmission name="${name}_wheel_joint_trans">
+                        <type>transmission_interface/SimpleTransmission</type>
+                        <joint name="${name}_wheel_joint">
+                                <hardwareInterface>hardware_interface/EffortJointInterface</hardwareInterface>
+                        </joint>
+                        <actuator name="${name}_wheel_joint_motor">
+                                <hardwareInterface>hardware_interface/EffortJointInterface</hardwareInterface>
+                                <mechanicalReduction>1</mechanicalReduction>
+                        </actuator>
+                </transmission>
         </xacro:macro>
 </robot>
