Commit message: add wheel joint and link

File: urdfs/leg.xacro (robot description, xacro)
@@ -11,467 +11,468 @@
     <xacro:property name="LOWER_LEG_y" value="0.00035" />
     <xacro:property name="LOWER_LEG_z" value="2e-05" />
-    <xacro:property name="PRE_WHEEL" value="0.10183" />
+    <xacro:property name="PRE_WHEEL_pos" value="0.16173" />
+    <xacro:property name="WHEEL_pos" value="0.10183" />
     <!-- This macro has for purpose to define a leg -->
     <xacro:macro name="leg" params="name parent is_front is_right robot_name *origin">
-          <!-- Starbot 1.0 -->
-	  <!--BS_JOINT: Joint between the body and the shoulder -->
-            <joint name="${name}_bs_joint" type="revolute">
-                <parent link="${parent}"/>
-                <child link="${name}_shoulder"/>
-                <xacro:insert_block name="origin"/>
-                <!-- joints rotates around the z-axis -->
-                <axis xyz="0 0 1"/>
-                <!-- limit of the joint -->
-                <limit effort="${MAX_TORQUE}" lower="-3.14" upper="3.14" velocity="${VELOCITY}"/>
-            </joint>
-	  <!-- SHOULDER ASSEMBLY -->
-            <link name="${name}_shoulder">
-            	<!-- create a dummy shoulder_assembly link to join the two joints -->
-            	<!--VISUAL-->
-	        <visual>
-                    <xacro:if value="${is_front}">
-                        <xacro:unless value="${is_right}">
-                            <!-- LF SHOULDER -->
-                        	<geometry>
-                        	    <mesh filename="package://starbot_description/meshes/stl/shoulder_y.stl"/>
-                        	</geometry>
-                        </xacro:unless>
-                        <xacro:if value="${is_right}">
-                            <!-- RF SHOULDER-->
-                        	<geometry>
-                        	    <mesh filename="package://starbot_description/meshes/stl/shoulder_x.stl"/>
-                        	</geometry>
+        <!-- Starbot 1.0 -->
+        <!--BS_JOINT: Joint between the body and the shoulder -->
+        <joint name="${name}_bs_joint" type="revolute">
+            <parent link="${parent}"/>
+            <child link="${name}_shoulder"/>
+            <xacro:insert_block name="origin"/>
+            <!-- joints rotates around the z-axis -->
+            <axis xyz="0 0 1"/>
+            <!-- limit of the joint -->
+            <limit effort="${MAX_TORQUE}" lower="-3.14" upper="3.14" velocity="${VELOCITY}"/>
+        </joint>
+        <!-- SHOULDER ASSEMBLY -->
+        <link name="${name}_shoulder">
+            <!-- create a dummy shoulder_assembly link to join the two joints -->
+            <!--VISUAL-->
+            <visual>
+                <xacro:if value="${is_front}">
+                    <xacro:unless value="${is_right}">
+                        <!-- LF SHOULDER -->
+                        <geometry>
+                            <mesh filename="package://starbot_description/meshes/stl/shoulder_y.stl"/>
+                        </geometry>
+                    </xacro:unless>
+                <xacro:if value="${is_right}">
+                    <!-- RF SHOULDER-->
+                    <geometry>
+                        <mesh filename="package://starbot_description/meshes/stl/shoulder_x.stl"/>
+                    </geometry>
+                    </xacro:if>
+                </xacro:if>
+                <xacro:unless value="${is_front}">
+                    <xacro:unless value="${is_right}">
+                        <!-- LH SHOULDER -->
+                        <geometry>
+                            <mesh filename="package://starbot_description/meshes/stl/shoulder_nx.stl"/>
+                        </geometry>
+                    </xacro:unless>
+                    <xacro:if value="${is_right}">
+                        <!-- RH SHOULDER -->
+                        <geometry>
+                            <mesh filename="package://starbot_description/meshes/stl/shoulder_ny.stl"/>
+                        </geometry>
+                    </xacro:if>
+                </xacro:unless>
+                <material name="shoulder_color">
+                    <color rgba="0.8 0.8 0.8 1.0"/>
+                </material>
+            </visual>
+            <!--COLLISION-->
+            <collision>
+                <origin xyz="0 0 0" rpy="0 0 0" />
+                <xacro:if value="${is_front}">
+                    <xacro:unless value="${is_right}">
+                        <!-- LF_BS -->
+                        <geometry>
+                            <mesh filename="package://starbot_description/meshes/stl/shoulder_y.stl"/>
+                        </geometry>
+                    </xacro:unless>
+                    <xacro:if value="${is_right}">
+                        <!-- RF_BS -->
+                        <geometry>
+                            <mesh filename="package://starbot_description/meshes/stl/shoulder_x.stl"/>
+                        </geometry>
+                    </xacro:if>
+                </xacro:if>
+                <xacro:unless value="${is_front}">
+                    <xacro:unless value="${is_right}">
+                        <!-- LH_BS -->
+                        <geometry>
+                            <mesh filename="package://starbot_description/meshes/stl/shoulder_nx.stl"/>
+                        </geometry>
+                    </xacro:unless>
+                    <xacro:if value="${is_right}">
+                        <!-- RH_BS -->
+                        <geometry>
+                            <mesh filename="package://starbot_description/meshes/stl/shoulder_ny.stl"/>
+                        </geometry>
+                    </xacro:if>
+                </xacro:unless>
+                <material name="collision_color">
+                    <color rgba="0.8 0.8 0.8 1.0"/>
+                </material>
+            </collision>
+            <!--INERTIAL -->
+            <inertial>
+                <origin xyz="0 0 0" rpy="0 0 0" />
+                <mass value="0.0001"/>
+                <inertia ixx="0" ixy="0" ixz="0" iyy="0" iyz="0" izz="0"/>
+            </inertial>
+        </link>
+        <!--UPPER LEG JOINT-->
+        <joint name="${name}_upper_leg_joint" type="revolute">
+            <parent link="${name}_shoulder"/>
+            <child link="${name}_upperleg"/>
+            <xacro:insert_block name="origin"/>
+            <!-- joints rotates around the y-axis -->
+            <!-- limit and placement of the joint -->
+            <xacro:if value="${is_front}">
+                <xacro:unless value="${is_right}">
+                    <!-- LF_UPPER_LEG_JOINT -->
+                    <axis xyz="1 0 0"/>
+                    <limit effort="${MAX_TORQUE}" lower="-3.14" upper="3.14" velocity="${VELOCITY}"/>
+                    <origin xyz="0 ${UPPER_LEG}  0" rpy="0 0 0" />
+                </xacro:unless>
+                <xacro:if value="${is_right}">
+                    <!-- RF_UPPER_LEG_JOINT -->
+                    <axis xyz="0 1 0"/>
+                    <limit effort="${MAX_TORQUE}" lower="-3.14" upper="3.14" velocity="${VELOCITY}"/>
+                    <origin xyz="${UPPER_LEG} 0 0" rpy="0 0 0" />
+                </xacro:if>
+            </xacro:if>
+            <xacro:unless value="${is_front}">
+                <xacro:unless value="${is_right}">
+                    <!-- LH_UPPER_LEG_JOINT -->
+                    <axis xyz="0 -1 0"/>
+                    <limit effort="${MAX_TORQUE}" lower="-3.14" upper="3.14" velocity="${VELOCITY}"/>
+                    <origin xyz="-${UPPER_LEG} 0 0" rpy="0 0 0" />
+                </xacro:unless>
+                <xacro:if value="${is_right}">
+                    <!-- RH_UPPER_LEG_JOINT -->
+                    <axis xyz="-1 0 0"/>
+                    <limit effort="${MAX_TORQUE}" lower="-3.14" upper="3.14" velocity="${VELOCITY}"/>
+                    <origin xyz="0 -${UPPER_LEG} 0" rpy="0 0 0" />
+                </xacro:if>
+            </xacro:unless>
+            <!-- pybullet simulation parameters -->
+            <dynamics damping="0.0" friction="0.0"/>
+        </joint>
+        <!-- UPPER LEG ASSEMBLY -->
+        <link name="${name}_upperleg">
+            <!--VISUAL-->
+            <visual>
+                <origin xyz="0 0 0" rpy="0 0 0" />
+                <xacro:if value="${is_front}">
+                    <xacro:unless value="${is_right}">
+                        <!-- LF UPPER_LEG -->
+                        <geometry>
+                            <mesh filename="package://starbot_description/meshes/stl/upper_leg_y.stl"/>
+                        </geometry>
+                    </xacro:unless>
+                    <xacro:if value="${is_right}">
+                        <!-- RF UPPER_LEG-->
+                        <geometry>
+                            <mesh filename="package://starbot_description/meshes/stl/upper_leg_x.stl"/>
+                        </geometry>
                         </xacro:if>
-                    </xacro:if>
-                    <xacro:unless value="${is_front}">
-                        <xacro:unless value="${is_right}">
-                            <!-- LH SHOULDER -->
-                        	<geometry>
-                        	    <mesh filename="package://starbot_description/meshes/stl/shoulder_nx.stl"/>
-                        	</geometry>
-                        </xacro:unless>
-                        <xacro:if value="${is_right}">
-                            <!-- RH SHOULDER -->
-                        	<geometry>
-                        	    <mesh filename="package://starbot_description/meshes/stl/shoulder_ny.stl"/>
-                        	</geometry>
-                        </xacro:if>
-                    </xacro:unless>
-	                <material name="shoulder_color">
-                    		<color rgba="0.8 0.8 0.8 1.0"/>
-                	</material>
-	            </visual>
-	            <!--COLLISION-->
-	            <collision>
-	            <origin xyz="0 0 0" rpy="0 0 0" />
-                    <xacro:if value="${is_front}">
-                        <xacro:unless value="${is_right}">
-                            <!-- LF_BS -->
-                        	<geometry>
-                        	    <box size="0.0707 0.00651 0.07002"/>
-                        	</geometry>
-                        </xacro:unless>
-                        <xacro:if value="${is_right}">
-                            <!-- RF_BS -->
-                        	<geometry>
-                        	    <box size="0.00651 0.0707 0.07002"/>
-                        	</geometry>
-                        </xacro:if>
-                    </xacro:if>
-                    <xacro:unless value="${is_front}">
-                        <xacro:unless value="${is_right}">
-                            <!-- LH_BS -->
-                        	<geometry>
-                        	    <box size="0.00651 0.0707 0.07002"/>
-                        	</geometry>
-                        </xacro:unless>
-                        <xacro:if value="${is_right}">
-                            <!-- RH_BS -->
-                        	<geometry>
-                        	    <box size="0.0707 0.00651 0.07002"/>
-                        	</geometry>
-                        </xacro:if>
-                    </xacro:unless>
-	                <material name="collision_color">
-      				<color rgba="0.8 0.8 0.8 1.0"/>
-    			</material>
-	            </collision>
-	            <!--INERTIAL -->
-	            <inertial>
-	            	<origin xyz="0 0 0" rpy="0 0 0" />
-	                <mass value="0.0001"/>
-	                <inertia ixx="0" ixy="0" ixz="0" iyy="0" iyz="0" izz="0"/>
-	            </inertial>
-	        </link>
-	     <!--UPPER LEG JOINT-->
-            <joint name="${name}_upper_leg_joint" type="revolute">
-                <parent link="${name}_shoulder"/>
-                <child link="${name}_upperleg"/>
-                <xacro:insert_block name="origin"/>
-                <!-- joints rotates around the y-axis -->
-                <!-- limit and placement of the joint -->
-                <xacro:if value="${is_front}">
-                    <xacro:unless value="${is_right}">
-                        <!-- LF_UPPER_LEG_JOINT -->
-                        <axis xyz="1 0 0"/>
-                        <limit effort="${MAX_TORQUE}" lower="-3.14" upper="3.14" velocity="${VELOCITY}"/>
-                        <origin xyz="0 ${UPPER_LEG}  0" rpy="0 0 0" />
-                    </xacro:unless>
-                    <xacro:if value="${is_right}">
-                        <!-- RF_UPPER_LEG_JOINT -->
-                        <axis xyz="0 1 0"/>
-			<limit effort="${MAX_TORQUE}" lower="-3.14" upper="3.14" velocity="${VELOCITY}"/>
-                        <origin xyz="${UPPER_LEG} 0 0" rpy="0 0 0" />
-                    </xacro:if>
-                </xacro:if>
-                <xacro:unless value="${is_front}">
-                    <xacro:unless value="${is_right}">
-                        <!-- LH_UPPER_LEG_JOINT -->
-                        <axis xyz="0 -1 0"/>
-			<limit effort="${MAX_TORQUE}" lower="-3.14" upper="3.14" velocity="${VELOCITY}"/>
-                        <origin xyz="-${UPPER_LEG} 0 0" rpy="0 0 0" />
-                    </xacro:unless>
-                    <xacro:if value="${is_right}">
-                        <!-- RH_UPPER_LEG_JOINT -->
-                        <axis xyz="-1 0 0"/>
-			<limit effort="${MAX_TORQUE}" lower="-3.14" upper="3.14" velocity="${VELOCITY}"/>
-                        <origin xyz="0 -${UPPER_LEG} 0" rpy="0 0 0" />
-                    </xacro:if>
-                </xacro:unless>
-                <!-- pybullet simulation parameters -->
-                <dynamics damping="0.0" friction="0.0"/>
-            </joint>
-	  <!-- UPPER LEG ASSEMBLY -->
-            <link name="${name}_upperleg">
-            	<!--VISUAL-->
-	        <visual>
-	            <origin xyz="0 0 0" rpy="0 0 0" />
-                    <xacro:if value="${is_front}">
-                        <xacro:unless value="${is_right}">
-                            <!-- LF UPPER_LEG -->
-                        	<geometry>
-                        	    <mesh filename="package://starbot_description/meshes/stl/upper_leg_y.stl"/>
-                        	</geometry>
-                        </xacro:unless>
-                        <xacro:if value="${is_right}">
-                            <!-- RF UPPER_LEG-->
-                        	<geometry>
-                        	    <mesh filename="package://starbot_description/meshes/stl/upper_leg_x.stl"/>
-                        	</geometry>
-                        </xacro:if>
-                    </xacro:if>
-                    <xacro:unless value="${is_front}">
-                        <xacro:unless value="${is_right}">
-                            <!-- LH UPPER_LEG -->
-                        	<geometry>
-                        	    <mesh filename="package://starbot_description/meshes/stl/upper_leg_nx.stl"/>
-                        	</geometry>
-                        </xacro:unless>
-                        <xacro:if value="${is_right}">
-                            <!-- RH UPPER_LEG -->
-                        	<geometry>
-                        	    <mesh filename="package://starbot_description/meshes/stl/upper_leg_ny.stl"/>
-                        	</geometry>
-                        </xacro:if>
-                    </xacro:unless>
-	                <material name="upper_leg_color">
-                    		<color rgba="0.8 0.8 0.8 1.0"/>
-                	</material>
-	            </visual>
-	            <!--COLLISION-->
-	            <collision>
-	            <origin xyz="0 0 0" rpy="0 0 0" />
-                    <xacro:if value="${is_front}">
-                        <xacro:unless value="${is_right}">
-                            <!-- LF UPPER_LEG -->
-                        	<geometry>
-                        	    <box size="0.07002 0.30016 0.0707"/>
-                        	</geometry>
-                        </xacro:unless>
-                        <xacro:if value="${is_right}">
-                            <!-- RF UPPER_LEG -->
-                        	<geometry>
-                        	    <box size="0.30016 0.07002 0.0707"/>
-                        	</geometry>
-                        </xacro:if>
-                    </xacro:if>
-                    <xacro:unless value="${is_front}">
-                        <xacro:unless value="${is_right}">
-                            <!-- LH UPPER_LEG -->
-                        	<geometry>
-                        	    <box size="0.30016 0.07002 0.0707"/>
-                        	</geometry>
-                        </xacro:unless>
-                        <xacro:if value="${is_right}">
-                            <!-- RH UPPER_LEG-->
-                        	<geometry>
-                        	    <box size="0.07002 0.30016 0.0707"/>
-                        	</geometry>
-                        </xacro:if>
-                    </xacro:unless>
-	                <material name="collision_color">
-      				<color rgba="0.8 0.8 0.8 1.0"/>
-    			</material>
-	            </collision>
-	            <!-- UPPER LEG LINK INERTIAL -->
-            	<xacro:unless value="${is_right}">
+                </xacro:if>
+                <xacro:unless value="${is_front}">
+                    <xacro:unless value="${is_right}">
+                        <!-- LH UPPER_LEG -->
+                        <geometry>
+                            <mesh filename="package://starbot_description/meshes/stl/upper_leg_nx.stl"/>
+                        </geometry>
+                    </xacro:unless>
+                    <xacro:if value="${is_right}">
+                        <!-- RH UPPER_LEG -->
+                        <geometry>
+                            <mesh filename="package://starbot_description/meshes/stl/upper_leg_ny.stl"/>
+                        </geometry>
+                    </xacro:if>
+                </xacro:unless>
+                <material name="upper_leg_color">
+                <color rgba="0.8 0.8 0.8 1.0"/>
+                </material>
+            </visual>
+            <!--COLLISION-->
+            <collision>
+                <origin xyz="0 0 0" rpy="0 0 0" />
+                <xacro:if value="${is_front}">
+                    <xacro:unless value="${is_right}">
+                        <!-- LF UPPER_LEG -->
+                        <geometry>
+                            <mesh filename="package://starbot_description/meshes/stl/upper_leg_y.stl"/>
+                        </geometry>
+                    </xacro:unless>
+                    <xacro:if value="${is_right}">
+                        <!-- RF UPPER_LEG -->
+                        <geometry>
+                            <mesh filename="package://starbot_description/meshes/stl/upper_leg_x.stl"/>
+                        </geometry>
+                    </xacro:if>
+                </xacro:if>
+                <xacro:unless value="${is_front}">
+                    <xacro:unless value="${is_right}">
+                        <!-- LH UPPER_LEG -->
+                        <geometry>
+                            <mesh filename="package://starbot_description/meshes/stl/upper_leg_nx.stl"/>
+                        </geometry>
+                    </xacro:unless>
+                    <xacro:if value="${is_right}">
+                        <!-- RH UPPER_LEG-->
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