Commit message: fix urdf with new meshes

File: urdfs/leg.xacro (robot description, xacro)
@@ -244,5 +244,5 @@
                     <!-- LF_LOWER_LEG_JOINT -->
                     <axis xyz="0 1 0"/>
-                    <limit effort="${MAX_TORQUE}" lower="-3.14" upper="3.14" velocity="${VELOCITY}"/>
+                    <limit effort="${MAX_TORQUE}" lower="0" upper="0" velocity="${VELOCITY}"/>
                     <origin xyz="${LOWER_LEG_y} ${LOWER_LEG_x} -${LOWER_LEG_z}" rpy="0 0 0" />
                 </xacro:unless>
@@ -250,5 +250,5 @@
                     <axis xyz="1 0 0"/>
                     <!-- RF_LOWER_LEG_JOINT -->
-                    <limit effort="${MAX_TORQUE}" lower="-3.14" upper="3.14" velocity="${VELOCITY}"/>
+                    <limit effort="${MAX_TORQUE}" lower="0" upper="0" velocity="${VELOCITY}"/>
                     <origin xyz="${LOWER_LEG_x} -${LOWER_LEG_y} -${LOWER_LEG_z}" rpy="0 0 0" />
                 </xacro:if>
@@ -258,5 +258,5 @@
                     <axis xyz="-1 0 0"/>
                     <!-- LH_LOWER_LEG_JOINT -->
-                    <limit effort="${MAX_TORQUE}" lower="-3.14" upper="3.14" velocity="${VELOCITY}"/>
+                    <limit effort="${MAX_TORQUE}" lower="0" upper="0" velocity="${VELOCITY}"/>
                     <origin xyz="$-{LOWER_LEG_x} -${LOWER_LEG_y} -${LOWER_LEG_z}" rpy="0 0 0" />
                 </xacro:unless>
@@ -264,5 +264,5 @@
                     <!-- RF_LOWER_LEG_JOINT -->
                     <axis xyz="0 -1 0"/>
-                    <limit effort="${MAX_TORQUE}" lower="-3.14" upper="3.14" velocity="${VELOCITY}"/>
+                    <limit effort="${MAX_TORQUE}" lower="0" upper="0" velocity="${VELOCITY}"/>
                     <origin xyz="${LOWER_LEG_y} -${LOWER_LEG_x} -${LOWER_LEG_z}" rpy="0 0 0" />
                 </xacro:if>
@@ -281,5 +281,5 @@
                         <!--we need mesh geometry otherwise strange behaviour happens-->
                         <geometry>
-                            <mesh filename="package://starbot_description/meshes/stl/upper_leg_y.stl" scale = "0.8 0.8 0.8"/>
+                            <mesh filename="package://starbot_description/meshes/stl/lower_leg_y.stl"/>
                         </geometry>
                     </xacro:unless>
@@ -287,5 +287,5 @@
                         <!-- RF LOWER_LEG-->
                         <geometry>
-                            <mesh filename="package://starbot_description/meshes/stl/upper_leg_x.stl" scale = "0.8 0.8 0.8"/>
+                            <mesh filename="package://starbot_description/meshes/stl/lower_leg_x.stl"/>
                         </geometry>
                     </xacro:if>
@@ -295,5 +295,5 @@
                         <!-- LH LOWER_LEG -->
                         <geometry>
-                            <mesh filename="package://starbot_description/meshes/stl/upper_leg_nx.stl" scale = "0.8 0.8 0.8"/>
+                            <mesh filename="package://starbot_description/meshes/stl/lower_leg_nx.stl"/>
                         </geometry>
                     </xacro:unless>
@@ -301,5 +301,5 @@
                         <!-- RH LOWER_LEG -->
                         <geometry>
-                            <mesh filename="package://starbot_description/meshes/stl/upper_leg_ny.stl" scale = "0.8 0.8 0.8"/>
+                            <mesh filename="package://starbot_description/meshes/stl/lower_leg_ny.stl"/>
                         </geometry>
                     </xacro:if>
@@ -316,5 +316,5 @@
                         <!-- LF LOWER_LEG -->
                         <geometry>
-                            <mesh filename="package://starbot_description/meshes/stl/upper_leg_y.stl" scale = "0.8 0.8 0.8"/>
+                            <mesh filename="package://starbot_description/meshes/stl/lower_leg_y.stl"/>
                         </geometry>
                     </xacro:unless>
@@ -322,5 +322,5 @@
                         <!-- RF LOWER_LEG -->
                         <geometry>
-                            <mesh filename="package://starbot_description/meshes/stl/upper_leg_x.stl" scale = "0.8 0.8 0.8"/>
+                            <mesh filename="package://starbot_description/meshes/stl/lower_leg_x.stl"/>
                         </geometry>
                     </xacro:if>
@@ -330,5 +330,5 @@
                         <!-- LH LOWER_LEG -->
                         <geometry>
-                            <mesh filename="package://starbot_description/meshes/stl/upper_leg_nx.stl" scale = "0.8 0.8 0.8"/>
+                            <mesh filename="package://starbot_description/meshes/stl/lower_leg_nx.stl"/>
                         </geometry>
                     </xacro:unless>
@@ -336,5 +336,5 @@
                         <!-- RH LOWER_LEG-->
                         <geometry>
-                            <mesh filename="package://starbot_description/meshes/stl/upper_leg_ny.stl" scale = "0.8 0.8 0.8"/>
+                            <mesh filename="package://starbot_description/meshes/stl/lower_leg_ny.stl"/>
                         </geometry>
                     </xacro:if>
@@ -410,5 +410,5 @@
                         <!--we need mesh geometry otherwise strange behaviour happens-->
                         <geometry>
-                            <mesh filename="package://starbot_description/meshes/stl/upper_leg_y.stl" scale = "0.5 0.5 0.5"/>
+                            <mesh filename="package://starbot_description/meshes/stl/joint_wheel_y.stl"/>
                         </geometry>
                     </xacro:unless>
@@ -416,5 +416,5 @@
                         <!-- RF PRE_WHEEL-->
                         <geometry>
-                            <mesh filename="package://starbot_description/meshes/stl/upper_leg_x.stl" scale = "0.5 0.5 0.5"/>
+                            <mesh filename="package://starbot_description/meshes/stl/joint_wheel_x.stl"/>
                         </geometry>
                     </xacro:if>
@@ -424,5 +424,5 @@
                         <!-- LH PRE_WHEEL -->
                         <geometry>
-                            <mesh filename="package://starbot_description/meshes/stl/upper_leg_nx.stl" scale = "0.5 0.5 0.5"/>
+                            <mesh filename="package://starbot_description/meshes/stl/joint_wheel_nx.stl"/>
                         </geometry>
                     </xacro:unless>
@@ -430,5 +430,5 @@
                         <!-- RH PRE_WHEEL -->
                         <geometry>
-                            <mesh filename="package://starbot_description/meshes/stl/upper_leg_ny.stl" scale = "0.5 0.5 0.5"/>
+                            <mesh filename="package://starbot_description/meshes/stl/joint_wheel_ny.stl"/>
                         </geometry>
                     </xacro:if>
@@ -445,5 +445,5 @@
                         <!-- LF PRE_WHEEL -->
                         <geometry>
-                            <mesh filename="package://starbot_description/meshes/stl/upper_leg_ny.stl" scale = "0.5 0.5 0.5"/>
+                            <mesh filename="package://starbot_description/meshes/stl/joint_wheel_y.stl"/>
                         </geometry>
                     </xacro:unless>
@@ -451,5 +451,5 @@
                         <!-- RF PRE_WHEEL -->
                         <geometry>
-                            <mesh filename="package://starbot_description/meshes/stl/upper_leg_ny.stl" scale = "0.5 0.5 0.5"/>
+                            <mesh filename="package://starbot_description/meshes/stl/joint_wheel_x.stl"/>
                         </geometry>
                     </xacro:if>
@@ -459,5 +459,5 @@
                         <!-- LH PRE_WHEEL -->
                         <geometry>
-                            <mesh filename="package://starbot_description/meshes/stl/upper_leg_ny.stl" scale = "0.5 0.5 0.5"/>
+                            <mesh filename="package://starbot_description/meshes/stl/joint_wheel_nx.stl"/>
                         </geometry>
                     </xacro:unless>
@@ -465,5 +465,5 @@
                         <!-- RH PRE_WHEEL-->
                         <geometry>
-                            <mesh filename="package://starbot_description/meshes/stl/upper_leg_ny.stl" scale = "0.5 0.5 0.5"/>
+                            <mesh filename="package://starbot_description/meshes/stl/joint_wheel_ny.stl"/>
                         </geometry>
                     </xacro:if>
@@ -539,5 +539,5 @@
                         <!--we need mesh geometry otherwise strange behaviour happens-->
                         <geometry>
-                            <mesh filename="package://starbot_description/meshes/stl/upper_leg_y.stl" scale = "0.4 0.4 0.4"/>
+                            <mesh filename="package://starbot_description/meshes/stl/wheel_y.stl"/>
                         </geometry>
                     </xacro:unless>
@@ -545,5 +545,5 @@
                         <!-- RF WHEEL-->
                         <geometry>
-                            <mesh filename="package://starbot_description/meshes/stl/upper_leg_x.stl" scale = "0.4 0.4 0.4"/>
+                            <mesh filename="package://starbot_description/meshes/stl/wheel_x.stl"/>
                         </geometry>
                     </xacro:if>
@@ -553,5 +553,5 @@
                         <!-- LH WHEEL -->
                         <geometry>
-                            <mesh filename="package://starbot_description/meshes/stl/upper_leg_nx.stl" scale = "0.4 0.4 0.4"/>
+                            <mesh filename="package://starbot_description/meshes/stl/wheel_nx.stl"/>
                         </geometry>
                     </xacro:unless>
@@ -559,5 +559,5 @@
                         <!-- RH WHEEL -->
                         <geometry>
-                            <mesh filename="package://starbot_description/meshes/stl/upper_leg_ny.stl" scale = "0.4 0.4 0.4"/>
+                            <mesh filename="package://starbot_description/meshes/stl/wheel_ny.stl"/>
                         </geometry>
                     </xacro:if>
@@ -574,5 +574,5 @@
                         <!-- LF WHEEL -->
                         <geometry>
-                            <mesh filename="package://starbot_description/meshes/stl/upper_leg_ny.stl" scale = "0.4 0.4 0.4"/>
+                            <mesh filename="package://starbot_description/meshes/stl/wheel_y.stl"/>
                         </geometry>
                     </xacro:unless>
@@ -580,5 +580,5 @@
                         <!-- RF WHEEL -->
                         <geometry>
-                            <mesh filename="package://starbot_description/meshes/stl/upper_leg_ny.stl" scale = "0.4 0.4 0.4"/>
+                            <mesh filename="package://starbot_description/meshes/stl/wheel_x.stl"/>
                         </geometry>
                     </xacro:if>
@@ -588,5 +588,5 @@
                         <!-- LH WHEEL -->
                         <geometry>
-                            <mesh filename="package://starbot_description/meshes/stl/upper_leg_ny.stl" scale = "0.4 0.4 0.4"/>
+                            <mesh filename="package://starbot_description/meshes/stl/wheel_nx.stl"/>
                         </geometry>
                     </xacro:unless>
@@ -594,5 +594,5 @@
                         <!-- RH WHEEL-->
                         <geometry>
-                            <mesh filename="package://starbot_description/meshes/stl/upper_leg_ny.stl" scale = "0.4 0.4 0.4"/>
+                            <mesh filename="package://starbot_description/meshes/stl/wheel_ny.stl"/>
                         </geometry>
                     </xacro:if>

Commit message: fixed bs and prewheel joint

File: urdfs/leg.xacro (robot description, xacro)
@@ -143,13 +143,13 @@
                 <xacro:unless value="${is_right}">
                     <!-- LF_UPPER_LEG_JOINT -->
-                    <axis xyz="1 0 0"/>
+                    <axis xyz="0 0 1"/>
                     <limit effort="${MAX_TORQUE}" lower="-0.785" upper="0.785" velocity="${VELOCITY}"/>
-                    <origin xyz="0 ${UPPER_LEG}  0" rpy="0 0 0" />
+                    <origin xyz="0 0  0" rpy="0 0 0" />
                 </xacro:unless>
                 <xacro:if value="${is_right}">
                     <!-- RF_UPPER_LEG_JOINT -->
-                    <axis xyz="0 1 0"/>
+                    <axis xyz="0 0 1"/>
                     <limit effort="${MAX_TORQUE}" lower="-0.785" upper="0.785" velocity="${VELOCITY}"/>
-                    <origin xyz="${UPPER_LEG} 0 0" rpy="0 0 0" />
+                    <origin xyz="0 0 0" rpy="0 0 0" />
                 </xacro:if>
             </xacro:if>
@@ -157,13 +157,13 @@
                 <xacro:unless value="${is_right}">
                     <!-- LH_UPPER_LEG_JOINT -->
-                    <axis xyz="0 -1 0"/>
+                    <axis xyz="0 0 1"/>
                     <limit effort="${MAX_TORQUE}" lower="-0.785" upper="0.785" velocity="${VELOCITY}"/>
-                    <origin xyz="-${UPPER_LEG} 0 0" rpy="0 0 0" />
+                    <origin xyz="0 0 0" rpy="0 0 0" />
                 </xacro:unless>
                 <xacro:if value="${is_right}">
                     <!-- RH_UPPER_LEG_JOINT -->
-                    <axis xyz="-1 0 0"/>
+                    <axis xyz="0 0 1"/>
                     <limit effort="${MAX_TORQUE}" lower="-0.785" upper="0.785" velocity="${VELOCITY}"/>
-                    <origin xyz="0 -${UPPER_LEG} 0" rpy="0 0 0" />
+                    <origin xyz="0 0 0" rpy="0 0 0" />
                 </xacro:if>
             </xacro:unless>
@@ -175,8 +175,8 @@
             <!--VISUAL-->
             <visual>
-                <origin xyz="0 0 0" rpy="0 0 0" />
-                <xacro:if value="${is_front}">
-                    <xacro:unless value="${is_right}">
-                        <!-- LF UPPER_LEG -->
+                <xacro:if value="${is_front}">
+                    <xacro:unless value="${is_right}">
+			<!-- LF UPPER_LEG -->
+                      		<origin xyz="0 ${UPPER_LEG} 0" rpy="0 0 0" />
                         <geometry>
                             <mesh filename="package://starbot_description/meshes/stl/upper_leg_y.stl"/>
@@ -184,5 +184,6 @@
                     </xacro:unless>
                     <xacro:if value="${is_right}">
-                        <!-- RF UPPER_LEG-->
+			<!-- RF UPPER_LEG-->
+                        <origin xyz="${UPPER_LEG} 0 0" rpy="0 0 0" />
                         <geometry>
                             <mesh filename="package://starbot_description/meshes/stl/upper_leg_x.stl"/>
@@ -192,5 +193,6 @@
                 <xacro:unless value="${is_front}">
                     <xacro:unless value="${is_right}">
-                        <!-- LH UPPER_LEG -->
+			<!-- LH UPPER_LEG -->
+			<origin xyz="-${UPPER_LEG} 0  0" rpy="0 0 0" />
                         <geometry>
                             <mesh filename="package://starbot_description/meshes/stl/upper_leg_nx.stl"/>
@@ -198,5 +200,6 @@
                     </xacro:unless>
                     <xacro:if value="${is_right}">
-                        <!-- RH UPPER_LEG -->
+		        <!-- RH UPPER_LEG -->
+					<origin xyz=" 0 -${UPPER_LEG} 0" rpy="0 0 0" />
                         <geometry>
                             <mesh filename="package://starbot_description/meshes/stl/upper_leg_ny.stl"/>
@@ -208,8 +211,8 @@
             <!--COLLISION-->
             <collision>
-                <origin xyz="0 0 0" rpy="0 0 0" />
                 <xacro:if value="${is_front}">
                     <xacro:unless value="${is_right}">
                         <!-- LF UPPER_LEG -->
+			<origin xyz="0 ${UPPER_LEG}  0" rpy="0 0 0" />
                         <geometry>
                             <mesh filename="package://starbot_description/meshes/stl/upper_leg_y.stl"/>
@@ -218,4 +221,5 @@
                     <xacro:if value="${is_right}">
                         <!-- RF UPPER_LEG -->
+       			<origin xyz="${UPPER_LEG} 0 0" rpy="0 0 0" />
                         <geometry>
                             <mesh filename="package://starbot_description/meshes/stl/upper_leg_x.stl"/>
@@ -226,4 +230,5 @@
                     <xacro:unless value="${is_right}">
                         <!-- LH UPPER_LEG -->
+			<origin xyz="-${UPPER_LEG} 0  0" rpy="0 0 0" />
                         <geometry>
                             <mesh filename="package://starbot_description/meshes/stl/upper_leg_nx.stl"/>
@@ -232,4 +237,5 @@
                     <xacro:if value="${is_right}">
                         <!-- RH UPPER_LEG-->
+			<origin xyz=" 0 -${UPPER_LEG} 0" rpy="0 0 0" />
                         <geometry>
                             <mesh filename="package://starbot_description/meshes/stl/upper_leg_ny.stl"/>
@@ -285,4 +291,5 @@
                 <xacro:unless value="${is_right}">
                     <!-- LF_LOWER_LEG_JOINT -->
+			<origin xyz="0 ${UPPER_LEG} 0" rpy="0 0 0" />
                     <axis xyz="0 1 0"/>
                     <limit effort="${MAX_TORQUE}" lower="0" upper="0.20" velocity="${VELOCITY}"/>
@@ -292,4 +299,5 @@
                     <axis xyz="1 0 0"/>
                     <!-- RF_LOWER_LEG_JOINT -->
+		<origin xyz="${UPPER_LEG} 0 0" rpy="0 0 0" />
                     <limit effort="${MAX_TORQUE}" lower="0" upper="0.20" velocity="${VELOCITY}"/>
                     <origin xyz="${LOWER_LEG_pos} 0 0" rpy="0 0 0" />
@@ -300,4 +308,5 @@
                     <axis xyz="-1 0 0"/>
                     <!-- LH_LOWER_LEG_JOINT -->
+		<origin xyz="-${UPPER_LEG} 0  0" rpy="0 0 0" />
                     <limit effort="${MAX_TORQUE}" lower="0" upper="0.20" velocity="${VELOCITY}"/>
                     <origin xyz="-${LOWER_LEG_pos} 0 0" rpy="0 0 0" />
@@ -305,4 +314,5 @@
                 <xacro:if value="${is_right}">
                     <!-- RF_LOWER_LEG_JOINT -->
+			<origin xyz=" 0 -${UPPER_LEG} 0" rpy="0 0 0" />
                     <axis xyz="0 -1 0"/>
                     <limit effort="${MAX_TORQUE}" lower="0" upper="0.20" velocity="${VELOCITY}"/>
@@ -317,9 +327,9 @@
             <!--VISUAL-->
             <visual>
-                <origin xyz="0 0 0" rpy="0 0 0" />
                 <xacro:if value="${is_front}">
                     <xacro:unless value="${is_right}">
                         <!-- LF LOWER_LEG -->
-                        <!--we need mesh geometry otherwise strange behaviour happens-->
+			<origin xyz="0 ${UPPER_LEG}  0" rpy="0 0 0" />
+           <!--we need mesh geometry otherwise strange behaviour happens-->
                         <geometry>
                             <mesh filename="package://starbot_description/meshes/stl/lower_leg_y.stl"/>
@@ -428,10 +438,10 @@
                 <xacro:unless value="${is_right}">
                     <!-- LF_PRE_WHEEL_JOINT -->
-                    <axis xyz="1 0 0"/>
+                    <axis xyz="0 1 0"/>
                     <limit effort="${MAX_TORQUE}" lower="-1.57" upper="1.57" velocity="${VELOCITY}"/>
                     <origin xyz="0 ${PRE_WHEEL_pos} 0" rpy="0 0 0" />
                 </xacro:unless>
                 <xacro:if value="${is_right}">
-                    <axis xyz="0 1 0"/>
+                    <axis xyz="1 0 0"/>
                     <!-- RF_PRE_WHEEL_JOINT -->
                     <limit effort="${MAX_TORQUE}" lower="-1.57" upper="1.57" velocity="${VELOCITY}"/>
@@ -441,5 +451,5 @@
             <xacro:unless value="${is_front}">
                 <xacro:unless value="${is_right}">
-                    <axis xyz="0 -1 0"/>
+                    <axis xyz="-1 0  0"/>
                     <!-- LH_PRE_WHEEL_JOINT -->
                     <limit effort="${MAX_TORQUE}" lower="-1.57" upper="1.57" velocity="${VELOCITY}"/>
@@ -448,5 +458,5 @@
                 <xacro:if value="${is_right}">
                     <!-- RF_PRE_WHEEL_JOINT -->
-                    <axis xyz="-1 0 0"/>
+                    <axis xyz="0  -1 0"/>
                     <limit effort="${MAX_TORQUE}" lower="-1.57" upper="1.57" velocity="${VELOCITY}"/>
                     <origin xyz="0 -${PRE_WHEEL_pos} 0" rpy="0 0 0" />

Commit message: bugfix MAX TORQUE and velocity was set  to zero!!!

File: urdfs/leg.xacro (robot description, xacro)
@@ -5,5 +5,6 @@
     <xacro:include filename="$(find starbot_description)/urdfs/leg.gazebo.xacro"/>
     <!-- These are absoulte distance value, the sign are decided below -->
-    <xacro:property name="MAX_TORQUE" value="0" />
+    <xacro:property name="MAX_TORQUE" value="300" />
+    <xacro:property name="MAX_FORCE_LOWERLEG" value="10000" />
     <xacro:property name="SHOULDER" value="0.14142" />
     <xacro:property name="VELOCITY" value="0" />
@@ -289,5 +290,5 @@
                     <!-- LF_LOWER_LEG_JOINT -->
                     <axis xyz="0 1 0"/>
-                    <limit effort="${MAX_TORQUE}" lower="0.02" upper="0.20" velocity="${VELOCITY}"/>
+                    <limit effort="${MAX_FORCE_LOWERLEG}" lower="0.02" upper="0.20" velocity="${VELOCITY}"/>
                     <origin xyz="0 ${LOWER_LEG_pos} 0" rpy="0 0 0" />
                 </xacro:unless>
@@ -295,5 +296,5 @@
                     <axis xyz="1 0 0"/>
                     <!-- RF_LOWER_LEG_JOINT -->
-                    <limit effort="${MAX_TORQUE}" lower="0.02" upper="0.20" velocity="${VELOCITY}"/>
+                    <limit effort="${MAX_FORCE_LOWERLEG}" lower="0.02" upper="0.20" velocity="${VELOCITY}"/>
                     <origin xyz="${LOWER_LEG_pos} 0 0" rpy="0 0 0" />
                 </xacro:if>
@@ -303,5 +304,5 @@
                     <axis xyz="-1 0 0"/>
                     <!-- LH_LOWER_LEG_JOINT -->
-                    <limit effort="${MAX_TORQUE}" lower="0.02" upper="0.20" velocity="${VELOCITY}"/>
+                    <limit effort="${MAX_FORCE_LOWERLEG}" lower="0.02" upper="0.20" velocity="${VELOCITY}"/>
                     <origin xyz="-${LOWER_LEG_pos} 0 0" rpy="0 0 0" />
                 </xacro:unless>
@@ -309,5 +310,5 @@
                     <!-- RF_LOWER_LEG_JOINT -->
                     <axis xyz="0 -1 0"/>
-                    <limit effort="${MAX_TORQUE}" lower="0.02" upper="0.20" velocity="${VELOCITY}"/>
+                    <limit effort="${MAX_FORCE_LOWERLEG}" lower="0.02" upper="0.20" velocity="${VELOCITY}"/>
                     <origin xyz="0 -${LOWER_LEG_pos} 0" rpy="0 0 0" />
                 </xacro:if>
