Commit message: common file added

File: urdfs/leg.xacro (robot description, xacro)
@@ -4,22 +4,5 @@
     <xacro:include filename="$(find starbot_description)/urdfs/leg.transmission.xacro"/>
     <xacro:include filename="$(find starbot_description)/urdfs/leg.gazebo.xacro"/>
-    <!-- These are absoulte distance value, the sign are decided below -->
-    <xacro:property name="MAX_TORQUE" value="300" />
-    <xacro:property name="MAX_FORCE_LOWERLEG" value="10000" />
-    <xacro:property name="SHOULDER" value="0.14142" />
-    <xacro:property name="VELOCITY" value="0" />
-    <xacro:property name="UPPER_LEG" value="0.15312" />
-    <xacro:property name="LOWER_LEG_pos" value="0.02546" />
-    <xacro:property name="PRE_WHEEL_pos" value="0.16173" />
-    <xacro:property name="WHEEL_pos" value="0.10183" />
-    <material name="orange">
-     <color rgba="0.800 0.331 0.183 1.0"/>
-    </material>
-    <material name="blue">
-     <color rgba="0.051 0.144 0.800 1.0"/>
-    </material>
-    <material name="gray">
-     <color rgba="0.638 0.779 0.819 1.0"/>
-    </material>
+    <xacro:include filename="$(find starbot_description)/urdfs/common.xacro"/>
     <!-- This macro has for purpose to define a leg -->
     <xacro:macro name="leg" params="name parent is_front is_right robot_name">
@@ -34,12 +17,12 @@
                     <!-- LF_UPPER_LEG_JOINT -->
                     <axis xyz="1 0 0"/>
-                    <limit effort="${MAX_TORQUE}" lower="-0.785" upper="0.785" velocity="${VELOCITY}"/>
-                    <origin xyz="0 ${SHOULDER}  0" rpy="0 0 0" />
+                    <limit effort="${MAX_TORQUE_SHOULDER}" lower="-${REV_LIMIT}" upper="${REV_LIMIT}" velocity="${VELOCITY}"/>
+                    <origin xyz="0 ${SHOULDER_pos}  0" rpy="0 0 0" />
                 </xacro:unless>
                 <xacro:if value="${is_right}">
                     <!-- RF_UPPER_LEG_JOINT -->
                     <axis xyz="0 1 0"/>
-                    <limit effort="${MAX_TORQUE}" lower="-0.785" upper="0.785" velocity="${VELOCITY}"/>
-                    <origin xyz="${SHOULDER} 0 0" rpy="0 0 0" />
+                    <limit effort="${MAX_TORQUE_SHOULDER}" lower="-${REV_LIMIT}" upper="${REV_LIMIT}" velocity="${VELOCITY}"/>
+                    <origin xyz="${SHOULDER_pos} 0 0" rpy="0 0 0" />
                 </xacro:if>
             </xacro:if>
@@ -48,12 +31,12 @@
                     <!-- LH_UPPER_LEG_JOINT -->
                     <axis xyz="0 -1 0"/>
-                    <limit effort="${MAX_TORQUE}" lower="-0.785" upper="0.785" velocity="${VELOCITY}"/>
-                    <origin xyz="-${SHOULDER} 0 0" rpy="0 0 0" />
+                    <limit effort="${MAX_TORQUE_SHOULDER}" lower="-${REV_LIMIT}" upper="${REV_LIMIT}" velocity="${VELOCITY}"/>
+                    <origin xyz="-${SHOULDER_pos} 0 0" rpy="0 0 0" />
                 </xacro:unless>
                 <xacro:if value="${is_right}">
                     <!-- RH_UPPER_LEG_JOINT -->
                     <axis xyz="-1 0 0"/>
-                    <limit effort="${MAX_TORQUE}" lower="-0.785" upper="0.785" velocity="${VELOCITY}"/>
-                    <origin xyz="0 -${SHOULDER} 0" rpy="0 0 0" />
+                    <limit effort="${MAX_TORQUE_SHOULDER}" lower="-${REV_LIMIT}" upper="${REV_LIMIT}" velocity="${VELOCITY}"/>
+                    <origin xyz="0 -${SHOULDER_pos} 0" rpy="0 0 0" />
                 </xacro:if>
             </xacro:unless>
@@ -146,12 +129,12 @@
                     <!-- LF_UPPER_LEG_JOINT -->
                     <axis xyz="0 0 1"/>
-                    <limit effort="${MAX_TORQUE}" lower="-0.785" upper="0.785" velocity="${VELOCITY}"/>
-                    <origin xyz="0 ${UPPER_LEG} 0" rpy="0 0 0" />
+                    <limit effort="${MAX_TORQUE_UPPER}" lower="-${REV_LIMIT}" upper="${REV_LIMIT}" velocity="${VELOCITY}"/>
+                    <origin xyz="0 ${UPPER_LEG_pos} 0" rpy="0 0 0" />
                 </xacro:unless>
                 <xacro:if value="${is_right}">
                     <!-- RF_UPPER_LEG_JOINT -->
                     <axis xyz="0 0 1"/>
-                    <limit effort="${MAX_TORQUE}" lower="-0.785" upper="0.785" velocity="${VELOCITY}"/>
-                    <origin xyz="${UPPER_LEG} 0 0" rpy="0 0 0" />
+                    <limit effort="${MAX_TORQUE_UPPER}" lower="-${REV_LIMIT}" upper="${REV_LIMIT}" velocity="${VELOCITY}"/>
+                    <origin xyz="${UPPER_LEG_pos} 0 0" rpy="0 0 0" />
                 </xacro:if>
             </xacro:if>
@@ -160,12 +143,12 @@
                     <!-- LH_UPPER_LEG_JOINT -->
                     <axis xyz="0 0 1"/>
-                    <limit effort="${MAX_TORQUE}" lower="-0.785" upper="0.785" velocity="${VELOCITY}"/>
-                    <origin xyz="-${UPPER_LEG} 0 0" rpy="0 0 0" />
+                    <limit effort="${MAX_TORQUE_UPPER}" lower="-${REV_LIMIT}" upper="${REV_LIMIT}" velocity="${VELOCITY}"/>
+                    <origin xyz="-${UPPER_LEG_pos} 0 0" rpy="0 0 0" />
                 </xacro:unless>
                 <xacro:if value="${is_right}">
                     <!-- RH_UPPER_LEG_JOINT -->
                     <axis xyz="0 0 1"/>
-                    <limit effort="${MAX_TORQUE}" lower="-0.785" upper="0.785" velocity="${VELOCITY}"/>
-                    <origin xyz="0 -${UPPER_LEG} 0" rpy="0 0 0" />
+                    <limit effort="${MAX_TORQUE_UPPER}" lower="-${REV_LIMIT}" upper="${REV_LIMIT}" velocity="${VELOCITY}"/>
+                    <origin xyz="0 -${UPPER_LEG_pos} 0" rpy="0 0 0" />
                 </xacro:if>
             </xacro:unless>
@@ -248,5 +231,5 @@
                         <!-- LF UPPER_LEG -->
                         <inertial>
-                    		<origin xyz="0 ${UPPER_LEG} 0" rpy="0 0 0"/>
+                    		<origin xyz="0 ${CM_XY_UPPER} ${CM_Z_UPPER}" rpy="0 0 0"/>
                     		<mass value="2.3"/>
                     		<inertia ixx="0.01246" ixy="0" ixz="0" iyy="0.00148" iyz="0" izz="0.01246"/>
@@ -256,5 +239,5 @@
                         <!-- RF UPPER_LEG -->
                         <inertial>
-                    		<origin xyz="${UPPER_LEG} 0 0" rpy="0 0 0"/>
+                    		<origin xyz="${CM_XY_UPPER} 0 ${CM_Z_UPPER}" rpy="0 0 0"/>
                     		<mass value="2.3"/>
                     		<inertia ixx="0.00148" ixy="0" ixz="0" iyy="0.01246" iyz="0" izz="0.00148"/>
@@ -266,5 +249,5 @@
                         <!-- LH UPPER_LEG -->
                         <inertial>
-                    		<origin xyz="-${UPPER_LEG} 0 0" rpy="0 0 0"/>
+                    		<origin xyz="-${CM_XY_UPPER} 0 ${CM_Z_UPPER}" rpy="0 0 0"/>
                     		<mass value="2.3"/>
                     		<inertia ixx="0.00148" ixy="0" ixz="0" iyy="0.01246" iyz="0" izz="0.00148"/>
@@ -274,5 +257,5 @@
                         <!-- RH UPPER_LEG-->
                         <inertial>
-                    		<origin xyz="0 -${UPPER_LEG} 0" rpy="0 0 0"/>
+                    		<origin xyz="0 -${CM_XY_UPPER} ${CM_Z_UPPER}" rpy="0 0 0"/>
                     		<mass value="2.3"/>
                     		<inertia ixx="0.01246" ixy="0" ixz="0" iyy="0.00148" iyz="0" izz="0.01246"/>
@@ -290,5 +273,5 @@
                     <!-- LF_LOWER_LEG_JOINT -->
                     <axis xyz="0 1 0"/>
-                    <limit effort="${MAX_FORCE_LOWERLEG}" lower="0.02" upper="0.20" velocity="${VELOCITY}"/>
+                    <limit effort="${MAX_FORCE_LOWERLEG}" lower="${LOWER_LIMIT_PRI}" upper="${UPPER_LIMIT_PRI}" velocity="${VELOCITY}"/>
                     <origin xyz="0 ${LOWER_LEG_pos} 0" rpy="0 0 0" />
                 </xacro:unless>
@@ -296,5 +279,5 @@
                     <axis xyz="1 0 0"/>
                     <!-- RF_LOWER_LEG_JOINT -->
-                    <limit effort="${MAX_FORCE_LOWERLEG}" lower="0.02" upper="0.20" velocity="${VELOCITY}"/>
+                    <limit effort="${MAX_FORCE_LOWERLEG}" lower="${LOWER_LIMIT_PRI}" upper="${UPPER_LIMIT_PRI}" velocity="${VELOCITY}"/>
                     <origin xyz="${LOWER_LEG_pos} 0 0" rpy="0 0 0" />
                 </xacro:if>
@@ -304,5 +287,5 @@
                     <axis xyz="-1 0 0"/>
                     <!-- LH_LOWER_LEG_JOINT -->
-                    <limit effort="${MAX_FORCE_LOWERLEG}" lower="0.02" upper="0.20" velocity="${VELOCITY}"/>
+                    <limit effort="${MAX_FORCE_LOWERLEG}" lower="${LOWER_LIMIT_PRI}" upper="${UPPER_LIMIT_PRI}" velocity="${VELOCITY}"/>
                     <origin xyz="-${LOWER_LEG_pos} 0 0" rpy="0 0 0" />
                 </xacro:unless>
@@ -310,5 +293,5 @@
                     <!-- RF_LOWER_LEG_JOINT -->
                     <axis xyz="0 -1 0"/>
-                    <limit effort="${MAX_FORCE_LOWERLEG}" lower="0.02" upper="0.20" velocity="${VELOCITY}"/>
+                    <limit effort="${MAX_FORCE_LOWERLEG}" lower="${LOWER_LIMIT_PRI}" upper="${UPPER_LIMIT_PRI}" velocity="${VELOCITY}"/>
                     <origin xyz="0 -${LOWER_LEG_pos} 0" rpy="0 0 0" />
                 </xacro:if>
@@ -389,5 +372,5 @@
                         <!-- LF LOWER_LEG -->
                         <inertial>
-                    		<origin xyz="0 ${LOWER_LEG_pos} 0" rpy="0 0 0"/>
+                    		<origin xyz="0 ${CM_XY_LOWER} ${CM_Z_LOWER}" rpy="0 0 0"/>
                     		<mass value="2.36"/>
                     		<inertia ixx="0.00767" ixy="0" ixz="0" iyy="0.00056" iyz="0" izz="0.00767"/>
@@ -397,5 +380,5 @@
                         <!-- RF LOWER_LEG -->
                         <inertial>
-                    		<origin xyz="${LOWER_LEG_pos} 0 0" rpy="0 0 0"/>
+                    		<origin xyz="${CM_XY_LOWER} 0 ${CM_Z_LOWER}" rpy="0 0 0"/>
                     		<mass value="2.36"/>
                     		<inertia ixx="0.00056" ixy="0" ixz="0" iyy="0.00767" iyz="0" izz="0.00056"/>
@@ -407,5 +390,5 @@
                         <!-- LH LOWER_LEG -->
                         <inertial>
-                    		<origin xyz="-${LOWER_LEG_pos} 0 0" rpy="0 0 0"/>
+                    		<origin xyz="-${CM_XY_LOWER} 0 ${CM_Z_LOWER}" rpy="0 0 0"/>
                     		<mass value="2.36"/>
                     		<inertia ixx="0.00056" ixy="0" ixz="0" iyy="0.00767" iyz="0" izz="0.00056"/>
@@ -415,5 +398,5 @@
                         <!-- RH LOWER_LEG-->
                         <inertial>
-                    		<origin xyz="0 -${LOWER_LEG_pos} 0" rpy="0 0 0"/>
+                    		<origin xyz="0 -${CM_XY_LOWER} ${CM_Z_LOWER}" rpy="0 0 0"/>
                     		<mass value="2.36"/>
                     		<inertia ixx="0.00767" ixy="0" ixz="0" iyy="0.00056" iyz="0" izz="0.00767"/>
@@ -432,5 +415,5 @@
                     <!-- LF_PRE_WHEEL_JOINT -->
                     <axis xyz="0 1 0"/>
-                    <limit effort="${MAX_TORQUE}" lower="-1.57" upper="1.57" velocity="${VELOCITY}"/>
+                    <limit effort="${MAX_TORQUE_PRE_WHEEL}" lower="-${REV_LIMIT_PRE_WHEEL}" upper="${REV_LIMIT_PRE_WHEEL}" velocity="${VELOCITY}"/>
                     <origin xyz="0 ${PRE_WHEEL_pos} 0" rpy="0 0 0" />
                 </xacro:unless>
@@ -438,5 +421,5 @@
                     <axis xyz="1 0 0"/>
                     <!-- RF_PRE_WHEEL_JOINT -->
-                    <limit effort="${MAX_TORQUE}" lower="-1.57" upper="1.57" velocity="${VELOCITY}"/>
+                    <limit effort="${MAX_TORQUE_PRE_WHEEL}" lower="-${REV_LIMIT_PRE_WHEEL}" upper="${REV_LIMIT_PRE_WHEEL}" velocity="${VELOCITY}"/>
                     <origin xyz="${PRE_WHEEL_pos} 0 0" rpy="0 0 0" />
                 </xacro:if>
@@ -446,5 +429,5 @@
                     <axis xyz="-1 0  0"/>
                     <!-- LH_PRE_WHEEL_JOINT -->
-                    <limit effort="${MAX_TORQUE}" lower="-1.57" upper="1.57" velocity="${VELOCITY}"/>
+                    <limit effort="${MAX_TORQUE_PRE_WHEEL}" lower="-${REV_LIMIT_PRE_WHEEL}" upper="${REV_LIMIT_PRE_WHEEL}" velocity="${VELOCITY}"/>
                     <origin xyz="-${PRE_WHEEL_pos} 0 0" rpy="0 0 0" />
                 </xacro:unless>
@@ -452,5 +435,5 @@
                     <!-- RF_PRE_WHEEL_JOINT -->
                     <axis xyz="0  -1 0"/>
-                    <limit effort="${MAX_TORQUE}" lower="-1.57" upper="1.57" velocity="${VELOCITY}"/>
+                    <limit effort="${MAX_TORQUE_PRE_WHEEL}" lower="-${REV_LIMIT_PRE_WHEEL}" upper="${REV_LIMIT_PRE_WHEEL}" velocity="${VELOCITY}"/>
                     <origin xyz="0 -${PRE_WHEEL_pos} 0" rpy="0 0 0" />
                 </xacro:if>
@@ -467,5 +450,4 @@
                     <xacro:unless value="${is_right}">
                         <!-- LF PRE_WHEEL -->
-                        <!--we need mesh geometry otherwise strange behaviour happens-->
                         <geometry>
                             <mesh filename="package://starbot_description/meshes/stl/joint_wheel_y.stl"/>
@@ -532,5 +514,5 @@
                         <!-- PRE_WHEEL_LEG -->
                         <inertial>
-                    		<origin xyz="0 ${PRE_WHEEL_pos} 0" rpy="0 0 0"/>
+                    		<origin xyz="0 ${CM_XY_PRE_WHEEL} ${CM_Z_PRE_WHEEL}" rpy="0 0 0"/>
                     		<mass value="0.66"/>
                     		<inertia ixx="0.00024" ixy="0" ixz="0" iyy="0.00016" iyz="0" izz="0.00024"/>
@@ -540,5 +522,5 @@
                         <!-- PRE_WHEEL_LEG -->
                         <inertial>
-                    		<origin xyz="${PRE_WHEEL_pos} 0 0" rpy="0 0 0"/>
+                    		<origin xyz="${CM_XY_PRE_WHEEL} 0 ${CM_Z_PRE_WHEEL}" rpy="0 0 0"/>
                     		<mass value="0.66"/>
                     		<inertia ixx="0.00016" ixy="0" ixz="0" iyy="0.00024" iyz="0" izz="0.00016"/>
@@ -550,5 +532,5 @@
                         <!-- PRE_WHEEL_LEG -->
                         <inertial>
-                    		<origin xyz="-${PRE_WHEEL_pos} 0 0" rpy="0 0 0"/>
+                    		<origin xyz="-${CM_XY_PRE_WHEEL} 0 ${CM_Z_PRE_WHEEL}" rpy="0 0 0"/>
                     		<mass value="0.66"/>
                     		<inertia ixx="0.00016" ixy="0" ixz="0" iyy="0.00024" iyz="0" izz="0.00016"/>
@@ -558,5 +540,5 @@
                         <!-- PRE_WHEEL_LEG-->
                         <inertial>
-                    		<origin xyz="0 -${PRE_WHEEL_pos} 0" rpy="0 0 0"/>
+                    		<origin xyz="0 -${CM_XY_PRE_WHEEL} ${CM_Z_PRE_WHEEL}" rpy="0 0 0"/>
                     		<mass value="0.66"/>
                     		<inertia ixx="0.00024" ixy="0" ixz="0" iyy="0.00016" iyz="0" izz="0.00024"/>
@@ -575,4 +557,5 @@
                     <!-- LF_WHEEL_JOINT -->
                     <axis xyz="1 0 0"/>
+                    <limit effort="${MAX_TORQUE_WHEEL}" velocity="${VELOCITY}"/>
                     <origin xyz="0 ${WHEEL_pos} 0" rpy="0 0 0" />
                 </xacro:unless>
@@ -580,4 +563,5 @@
                     <axis xyz="0 1 0"/>
                     <!-- RF_WHEEL_JOINT -->
+                    <limit effort="${MAX_TORQUE_WHEEL}" velocity="${VELOCITY}"/>
                     <origin xyz="${WHEEL_pos} 0 0" rpy="0 0 0" />
                 </xacro:if>
@@ -587,4 +571,5 @@
                     <axis xyz="0 -1 0"/>
                     <!-- LH_WHEEL_JOINT -->
+                    <limit effort="${MAX_TORQUE_WHEEL}" velocity="${VELOCITY}"/>
                     <origin xyz="-${WHEEL_pos} 0 0" rpy="0 0 0" />
                 </xacro:unless>
@@ -592,4 +577,5 @@
                     <!-- RF_WHEEL_JOINT -->
                     <axis xyz="-1 0 0"/>
+                    <limit effort="${MAX_TORQUE_WHEEL}" velocity="${VELOCITY}"/>
                     <origin xyz="0 -${WHEEL_pos} 0" rpy="0 0 0" />
                 </xacro:if>
@@ -672,5 +658,5 @@
                         <!-- PRE_WHEEL_LEG -->
                         <inertial>
-                    		<origin xyz="0 ${WHEEL_pos} 0" rpy="0 0 0"/>
+                    		<origin xyz="0 ${CM_XY_WHEEL} ${CM_Z_WHEEL}" rpy="0 0 0"/>
                     		<mass value="1.0"/>
                     		<inertia ixx="0.00224" ixy="0" ixz="0" iyy="0.00121" iyz="0" izz="0.00224"/>
@@ -680,5 +666,5 @@
                         <!-- PRE_WHEEL_LEG -->
                         <inertial>
-                    		<origin xyz="${WHEEL_pos} 0 0" rpy="0 0 0"/>
+                    		<origin xyz="${CM_XY_WHEEL} 0 ${CM_Z_WHEEL}" rpy="0 0 0"/>
                     		<mass value="1.0"/>
                     		<inertia ixx="0.00121" ixy="0" ixz="0" iyy="0.00224" iyz="0" izz="0.00121"/>
@@ -690,5 +676,5 @@
                         <!-- PRE_WHEEL_LEG -->
                         <inertial>
-                    		<origin xyz="-${WHEEL_pos}  0 0" rpy="0 0 0"/>
+                    		<origin xyz="-${CM_XY_WHEEL}  0 ${CM_Z_WHEEL}" rpy="0 0 0"/>
                     		<mass value="1.0"/>
                     		<inertia ixx="0.00121" ixy="0" ixz="0" iyy="0.00224" iyz="0" izz="0.00121"/>
@@ -698,5 +684,5 @@
                         <!-- PRE_WHEEL_LEG-->
                         <inertial>
-                    		<origin xyz="0 -${WHEEL_pos} 0" rpy="0 0 0"/>
+                    		<origin xyz="0 -${CM_XY_WHEEL} ${CM_Z_WHEEL}" rpy="0 0 0"/>
                     		<mass value="1.0"/>
                     		<inertia ixx="0.00224" ixy="0" ixz="0" iyy="0.00121" iyz="0" izz="0.00224"/>
