Commit message: correcting leg

File: urdfs/leg.xacro (robot description, xacro)
@@ -130,5 +130,5 @@
                     <axis xyz="0 0 1"/>
                     <limit effort="${MAX_TORQUE_UPPER}" lower="-${REV_LIMIT}" upper="${REV_LIMIT}" velocity="${VELOCITY}"/>
-                    <origin xyz="0 ${UPPER_LEG_pos} 0" rpy="0 0 0" />
+                    <origin xyz="0 0 0" rpy="0 0 0" />
                 </xacro:unless>
                 <xacro:if value="${is_right}">
@@ -136,5 +136,5 @@
                     <axis xyz="0 0 1"/>
                     <limit effort="${MAX_TORQUE_UPPER}" lower="-${REV_LIMIT}" upper="${REV_LIMIT}" velocity="${VELOCITY}"/>
-                    <origin xyz="${UPPER_LEG_pos} 0 0" rpy="0 0 0" />
+                    <origin xyz="0 0 0" rpy="0 0 0" />
                 </xacro:if>
             </xacro:if>
@@ -144,5 +144,5 @@
                     <axis xyz="0 0 1"/>
                     <limit effort="${MAX_TORQUE_UPPER}" lower="-${REV_LIMIT}" upper="${REV_LIMIT}" velocity="${VELOCITY}"/>
-                    <origin xyz="-${UPPER_LEG_pos} 0 0" rpy="0 0 0" />
+                    <origin xyz="0 0 0" rpy="0 0 0" />
                 </xacro:unless>
                 <xacro:if value="${is_right}">
@@ -150,5 +150,5 @@
                     <axis xyz="0 0 1"/>
                     <limit effort="${MAX_TORQUE_UPPER}" lower="-${REV_LIMIT}" upper="${REV_LIMIT}" velocity="${VELOCITY}"/>
-                    <origin xyz="0 -${UPPER_LEG_pos} 0" rpy="0 0 0" />
+                    <origin xyz="0 0 0" rpy="0 0 0" />
                 </xacro:if>
             </xacro:unless>
@@ -160,8 +160,8 @@
             <!--VISUAL-->
             <visual>
-                <origin xyz="0 0 0" rpy="0 0 0" />
                 <xacro:if value="${is_front}">
                     <xacro:unless value="${is_right}">
 			<!-- LF UPPER_LEG -->
+                        <origin xyz="0 ${UPPER_LEG_pos} 0" rpy="0 0 0" />
                         <geometry>
                             <mesh filename="package://starbot_description/meshes/stl/upper_leg_y.stl"/>
@@ -170,4 +170,5 @@
                     <xacro:if value="${is_right}">
 			<!-- RF UPPER_LEG-->
+                        <origin xyz="${UPPER_LEG_pos} 0 0" rpy="0 0 0" />
                         <geometry>
                             <mesh filename="package://starbot_description/meshes/stl/upper_leg_x.stl"/>
@@ -178,4 +179,5 @@
                     <xacro:unless value="${is_right}">
 			<!-- LH UPPER_LEG -->
+                        <origin xyz="-${UPPER_LEG_pos} 0 0" rpy="0 0 0" />
                         <geometry>
                             <mesh filename="package://starbot_description/meshes/stl/upper_leg_nx.stl"/>
@@ -184,4 +186,5 @@
                     <xacro:if value="${is_right}">
 		        <!-- RH UPPER_LEG -->
+                        <origin xyz="0 -${UPPER_LEG_pos} 0" rpy="0 0 0" />
                         <geometry>
                             <mesh filename="package://starbot_description/meshes/stl/upper_leg_ny.stl"/>
@@ -196,5 +199,5 @@
                     <xacro:unless value="${is_right}">
                         <!-- LF UPPER_LEG -->
-			<origin xyz="0 0 0" rpy="0 0 0" />
+			            <origin xyz="0 ${UPPER_LEG_pos} 0" rpy="0 0 0" />
                         <geometry>
                             <mesh filename="package://starbot_description/meshes/stl/upper_leg_y.stl"/>
@@ -203,5 +206,5 @@
                     <xacro:if value="${is_right}">
                         <!-- RF UPPER_LEG -->
-       			<origin xyz="0 0 0" rpy="0 0 0" />
+       			        <origin xyz="${UPPER_LEG_pos} 0 0" rpy="0 0 0" />
                         <geometry>
                             <mesh filename="package://starbot_description/meshes/stl/upper_leg_x.stl"/>
@@ -212,5 +215,5 @@
                     <xacro:unless value="${is_right}">
                         <!-- LH UPPER_LEG -->
-			<origin xyz="0 0  0" rpy="0 0 0" />
+			            <origin xyz="-${UPPER_LEG_pos} 0 0" rpy="0 0 0" />
                         <geometry>
                             <mesh filename="package://starbot_description/meshes/stl/upper_leg_nx.stl"/>
@@ -219,5 +222,5 @@
                     <xacro:if value="${is_right}">
                         <!-- RH UPPER_LEG-->
-			<origin xyz=" 0 0 0" rpy="0 0 0" />
+			            <origin xyz=" 0 -${UPPER_LEG_pos} 0" rpy="0 0 0" />
                         <geometry>
                             <mesh filename="package://starbot_description/meshes/stl/upper_leg_ny.stl"/>
@@ -274,5 +277,5 @@
                     <axis xyz="0 1 0"/>
                     <limit effort="${MAX_FORCE_LOWERLEG}" lower="${LOWER_LIMIT_PRI}" upper="${UPPER_LIMIT_PRI}" velocity="${VELOCITY}"/>
-                    <origin xyz="0 ${LOWER_LEG_pos} 0" rpy="0 0 0" />
+                    <origin xyz="0 0 0" rpy="0 0 0" />
                 </xacro:unless>
                 <xacro:if value="${is_right}">
@@ -280,5 +283,5 @@
                     <!-- RF_LOWER_LEG_JOINT -->
                     <limit effort="${MAX_FORCE_LOWERLEG}" lower="${LOWER_LIMIT_PRI}" upper="${UPPER_LIMIT_PRI}" velocity="${VELOCITY}"/>
-                    <origin xyz="${LOWER_LEG_pos} 0 0" rpy="0 0 0" />
+                    <origin xyz="0 0 0" rpy="0 0 0" />
                 </xacro:if>
             </xacro:if>
@@ -288,5 +291,5 @@
                     <!-- LH_LOWER_LEG_JOINT -->
                     <limit effort="${MAX_FORCE_LOWERLEG}" lower="${LOWER_LIMIT_PRI}" upper="${UPPER_LIMIT_PRI}" velocity="${VELOCITY}"/>
-                    <origin xyz="-${LOWER_LEG_pos} 0 0" rpy="0 0 0" />
+                    <origin xyz="0 0 0" rpy="0 0 0" />
                 </xacro:unless>
                 <xacro:if value="${is_right}">
@@ -294,5 +297,5 @@
                     <axis xyz="0 -1 0"/>
                     <limit effort="${MAX_FORCE_LOWERLEG}" lower="${LOWER_LIMIT_PRI}" upper="${UPPER_LIMIT_PRI}" velocity="${VELOCITY}"/>
-                    <origin xyz="0 -${LOWER_LEG_pos} 0" rpy="0 0 0" />
+                    <origin xyz="0 0 0" rpy="0 0 0" />
                 </xacro:if>
             </xacro:unless>
@@ -304,8 +307,8 @@
             <!--VISUAL-->
             <visual>
-		<origin xyz="0 0 0" rpy="0 0 0" />
                 <xacro:if value="${is_front}">
                     <xacro:unless value="${is_right}">
                         <!-- LF LOWER_LEG -->
+		                <origin xyz="0 ${LOWER_LEG_pos} 0" rpy="0 0 0" />
                         <geometry>
                             <mesh filename="package://starbot_description/meshes/stl/lower_leg_y.stl"/>
@@ -314,4 +317,5 @@
                     <xacro:if value="${is_right}">
                         <!-- RF LOWER_LEG-->
+                        <origin xyz="${LOWER_LEG_pos} 0 0" rpy="0 0 0" />
                         <geometry>
                             <mesh filename="package://starbot_description/meshes/stl/lower_leg_x.stl"/>
@@ -322,4 +326,5 @@
                     <xacro:unless value="${is_right}">
                         <!-- LH LOWER_LEG -->
+                        <origin xyz="-${LOWER_LEG_pos} 0 0" rpy="0 0 0" />
                         <geometry>
                             <mesh filename="package://starbot_description/meshes/stl/lower_leg_nx.stl"/>
@@ -328,4 +333,5 @@
                     <xacro:if value="${is_right}">
                         <!-- RH LOWER_LEG -->
+                        <origin xyz="0 -${LOWER_LEG_pos} 0" rpy="0 0 0" />
                         <geometry>
                             <mesh filename="package://starbot_description/meshes/stl/lower_leg_ny.stl"/>
@@ -337,8 +343,8 @@
             <!--COLLISION-->
             <collision>
-                <origin xyz="0 0 0" rpy="0 0 0" />
                 <xacro:if value="${is_front}">
                     <xacro:unless value="${is_right}">
                         <!-- LF LOWER_LEG -->
+                        <origin xyz="0 ${LOWER_LEG_pos} 0" rpy="0 0 0" />
                         <geometry>
                             <mesh filename="package://starbot_description/meshes/stl/lower_leg_y.stl"/>
@@ -347,4 +353,5 @@
                     <xacro:if value="${is_right}">
                         <!-- RF LOWER_LEG -->
+                        <origin xyz="${LOWER_LEG_pos} 0 0" rpy="0 0 0" />
                         <geometry>
                             <mesh filename="package://starbot_description/meshes/stl/lower_leg_x.stl"/>
@@ -355,4 +362,5 @@
                     <xacro:unless value="${is_right}">
                         <!-- LH LOWER_LEG -->
+                        <origin xyz="-${LOWER_LEG_pos} 0 0" rpy="0 0 0" />
                         <geometry>
                             <mesh filename="package://starbot_description/meshes/stl/lower_leg_nx.stl"/>
@@ -361,4 +369,5 @@
                     <xacro:if value="${is_right}">
                         <!-- RH LOWER_LEG-->
+                        <origin xyz="0 -${LOWER_LEG_pos} 0" rpy="0 0 0" />
                         <geometry>
                             <mesh filename="package://starbot_description/meshes/stl/lower_leg_ny.stl"/>

Commit message: fixes to frames after meeting with prof.

File: urdfs/leg.xacro (robot description, xacro)
@@ -10,6 +10,7 @@
     <xacro:property name="VELOCITY" value="0" />
     <xacro:property name="UPPER_LEG" value="0.15312" />
-    <xacro:property name="LOWER_LEG_pos" value="0.02546" />
-    <xacro:property name="PRE_WHEEL_pos" value="0.16173" />
+    <xacro:property name="LOWER_LEG_pos" value="0.125" />
+     <xacro:property name="LOWER_LEG_joint_pos" value="0.05" />
+    <xacro:property name="PRE_WHEEL_pos" value="0.285" />
     <xacro:property name="WHEEL_pos" value="0.10183" />
     <material name="orange">
@@ -147,5 +148,5 @@
                     <axis xyz="0 0 1"/>
                     <limit effort="${MAX_TORQUE}" lower="-0.785" upper="0.785" velocity="${VELOCITY}"/>
-                    <origin xyz="0 ${UPPER_LEG} 0" rpy="0 0 0" />
+                    <origin xyz="0 0 0" rpy="0 0 0" />
                 </xacro:unless>
                 <xacro:if value="${is_right}">
@@ -153,5 +154,5 @@
                     <axis xyz="0 0 1"/>
                     <limit effort="${MAX_TORQUE}" lower="-0.785" upper="0.785" velocity="${VELOCITY}"/>
-                    <origin xyz="${UPPER_LEG} 0 0" rpy="0 0 0" />
+                    <origin xyz="0 0 0" rpy="0 0 0" />
                 </xacro:if>
             </xacro:if>
@@ -161,5 +162,5 @@
                     <axis xyz="0 0 1"/>
                     <limit effort="${MAX_TORQUE}" lower="-0.785" upper="0.785" velocity="${VELOCITY}"/>
-                    <origin xyz="-${UPPER_LEG} 0 0" rpy="0 0 0" />
+                    <origin xyz="0 0 0" rpy="0 0 0" />
                 </xacro:unless>
                 <xacro:if value="${is_right}">
@@ -167,5 +168,5 @@
                     <axis xyz="0 0 1"/>
                     <limit effort="${MAX_TORQUE}" lower="-0.785" upper="0.785" velocity="${VELOCITY}"/>
-                    <origin xyz="0 -${UPPER_LEG} 0" rpy="0 0 0" />
+                    <origin xyz="0 0 0" rpy="0 0 0" />
                 </xacro:if>
             </xacro:unless>
@@ -177,8 +178,8 @@
             <!--VISUAL-->
             <visual>
-                <origin xyz="0 0 0" rpy="0 0 0" />
                 <xacro:if value="${is_front}">
                     <xacro:unless value="${is_right}">
 			<!-- LF UPPER_LEG -->
+			<origin xyz="0 ${UPPER_LEG} 0" rpy="0 0 0" />
                         <geometry>
                             <mesh filename="package://starbot_description/meshes/stl/upper_leg_y.stl"/>
@@ -187,4 +188,5 @@
                     <xacro:if value="${is_right}">
 			<!-- RF UPPER_LEG-->
+			<origin xyz="${UPPER_LEG} 0 0" rpy="0 0 0" />
                         <geometry>
                             <mesh filename="package://starbot_description/meshes/stl/upper_leg_x.stl"/>
@@ -195,4 +197,5 @@
                     <xacro:unless value="${is_right}">
 			<!-- LH UPPER_LEG -->
+			<origin xyz="-${UPPER_LEG} 0 0" rpy="0 0 0" />
                         <geometry>
                             <mesh filename="package://starbot_description/meshes/stl/upper_leg_nx.stl"/>
@@ -201,4 +204,5 @@
                     <xacro:if value="${is_right}">
 		        <!-- RH UPPER_LEG -->
+		        <origin xyz="0 -${UPPER_LEG} 0" rpy="0 0 0" />
                         <geometry>
                             <mesh filename="package://starbot_description/meshes/stl/upper_leg_ny.stl"/>
@@ -213,5 +217,5 @@
                     <xacro:unless value="${is_right}">
                         <!-- LF UPPER_LEG -->
-			<origin xyz="0 0 0" rpy="0 0 0" />
+			<origin xyz="0 ${UPPER_LEG} 0" rpy="0 0 0" />
                         <geometry>
                             <mesh filename="package://starbot_description/meshes/stl/upper_leg_y.stl"/>
@@ -220,5 +224,5 @@
                     <xacro:if value="${is_right}">
                         <!-- RF UPPER_LEG -->
-       			<origin xyz="0 0 0" rpy="0 0 0" />
+       			<origin xyz="${UPPER_LEG} 0 0" rpy="0 0 0" />
                         <geometry>
                             <mesh filename="package://starbot_description/meshes/stl/upper_leg_x.stl"/>
@@ -229,5 +233,5 @@
                     <xacro:unless value="${is_right}">
                         <!-- LH UPPER_LEG -->
-			<origin xyz="0 0  0" rpy="0 0 0" />
+			<origin xyz="-${UPPER_LEG} 0 0" rpy="0 0 0" />
                         <geometry>
                             <mesh filename="package://starbot_description/meshes/stl/upper_leg_nx.stl"/>
@@ -236,5 +240,5 @@
                     <xacro:if value="${is_right}">
                         <!-- RH UPPER_LEG-->
-			<origin xyz=" 0 0 0" rpy="0 0 0" />
+			<origin xyz="0 -${UPPER_LEG} 0" rpy="0 0 0" />
                         <geometry>
                             <mesh filename="package://starbot_description/meshes/stl/upper_leg_ny.stl"/>
@@ -291,5 +295,5 @@
                     <axis xyz="0 1 0"/>
                     <limit effort="${MAX_FORCE_LOWERLEG}" lower="0.02" upper="0.20" velocity="${VELOCITY}"/>
-                    <origin xyz="0 ${LOWER_LEG_pos} 0" rpy="0 0 0" />
+                    <origin xyz="0 ${LOWER_LEG_joint_pos} 0" rpy="0 0 0" />
                 </xacro:unless>
                 <xacro:if value="${is_right}">
@@ -297,5 +301,5 @@
                     <!-- RF_LOWER_LEG_JOINT -->
                     <limit effort="${MAX_FORCE_LOWERLEG}" lower="0.02" upper="0.20" velocity="${VELOCITY}"/>
-                    <origin xyz="${LOWER_LEG_pos} 0 0" rpy="0 0 0" />
+                    <origin xyz="${LOWER_LEG_joint_pos} 0 0" rpy="0 0 0" />
                 </xacro:if>
             </xacro:if>
@@ -305,5 +309,5 @@
                     <!-- LH_LOWER_LEG_JOINT -->
                     <limit effort="${MAX_FORCE_LOWERLEG}" lower="0.02" upper="0.20" velocity="${VELOCITY}"/>
-                    <origin xyz="-${LOWER_LEG_pos} 0 0" rpy="0 0 0" />
+                    <origin xyz="-${LOWER_LEG_joint_pos} 0 0" rpy="0 0 0" />
                 </xacro:unless>
                 <xacro:if value="${is_right}">
@@ -311,5 +315,5 @@
                     <axis xyz="0 -1 0"/>
                     <limit effort="${MAX_FORCE_LOWERLEG}" lower="0.02" upper="0.20" velocity="${VELOCITY}"/>
-                    <origin xyz="0 -${LOWER_LEG_pos} 0" rpy="0 0 0" />
+                    <origin xyz="0 -${LOWER_LEG_joint_pos} 0" rpy="0 0 0" />
                 </xacro:if>
             </xacro:unless>
@@ -321,8 +325,8 @@
             <!--VISUAL-->
             <visual>
-		<origin xyz="0 0 0" rpy="0 0 0" />
                 <xacro:if value="${is_front}">
                     <xacro:unless value="${is_right}">
                         <!-- LF LOWER_LEG -->
+                        <origin xyz="0 ${LOWER_LEG_pos} 0" rpy="0 0 0" />
                         <geometry>
                             <mesh filename="package://starbot_description/meshes/stl/lower_leg_y.stl"/>
@@ -331,4 +335,5 @@
                     <xacro:if value="${is_right}">
                         <!-- RF LOWER_LEG-->
+                        <origin xyz="${LOWER_LEG_pos} 0 0" rpy="0 0 0" />
                         <geometry>
                             <mesh filename="package://starbot_description/meshes/stl/lower_leg_x.stl"/>
@@ -339,4 +344,5 @@
                     <xacro:unless value="${is_right}">
                         <!-- LH LOWER_LEG -->
+                        <origin xyz="-${LOWER_LEG_pos} 0 0" rpy="0 0 0" />
                         <geometry>
                             <mesh filename="package://starbot_description/meshes/stl/lower_leg_nx.stl"/>
@@ -345,4 +351,5 @@
                     <xacro:if value="${is_right}">
                         <!-- RH LOWER_LEG -->
+                        <origin xyz="0 -${LOWER_LEG_pos} 0" rpy="0 0 0" />
                         <geometry>
                             <mesh filename="package://starbot_description/meshes/stl/lower_leg_ny.stl"/>
@@ -354,8 +361,8 @@
             <!--COLLISION-->
             <collision>
-                <origin xyz="0 0 0" rpy="0 0 0" />
                 <xacro:if value="${is_front}">
                     <xacro:unless value="${is_right}">
                         <!-- LF LOWER_LEG -->
+                         <origin xyz="0 ${LOWER_LEG_pos} 0" rpy="0 0 0" />
                         <geometry>
                             <mesh filename="package://starbot_description/meshes/stl/lower_leg_y.stl"/>
@@ -364,4 +371,5 @@
                     <xacro:if value="${is_right}">
                         <!-- RF LOWER_LEG -->
+                        <origin xyz="${LOWER_LEG_pos} 0 0" rpy="0 0 0" />
                         <geometry>
                             <mesh filename="package://starbot_description/meshes/stl/lower_leg_x.stl"/>
@@ -372,4 +380,5 @@
                     <xacro:unless value="${is_right}">
                         <!-- LH LOWER_LEG -->
+                        <origin xyz="-${LOWER_LEG_pos} 0 0" rpy="0 0 0" />
                         <geometry>
                             <mesh filename="package://starbot_description/meshes/stl/lower_leg_nx.stl"/>
@@ -378,4 +387,5 @@
                     <xacro:if value="${is_right}">
                         <!-- RH LOWER_LEG-->
+                         <origin xyz="0 -${LOWER_LEG_pos} 0" rpy="0 0 0" />
                         <geometry>
                             <mesh filename="package://starbot_description/meshes/stl/lower_leg_ny.stl"/>
