Commit message: adjusted joint limits

File: urdfs/common.xacro (robot description, xacro)
@@ -3,7 +3,7 @@
     <!-- revolute prismatic limits -->
     <xacro:property name="REV_LIMIT" value="0.785" />
-    <xacro:property name="REV_LIMIT_PRE_WHEEL" value="1.57" />
-    <xacro:property name="LOWER_LIMIT_PRI" value="0.01" />
-    <xacro:property name="UPPER_LIMIT_PRI" value="0.20" />
+    <xacro:property name="REV_LIMIT_PRE_WHEEL" value="3.14" />
+    <xacro:property name="LOWER_LIMIT_PRI" value="0" />
+    <xacro:property name="UPPER_LIMIT_PRI" value="0.2" />
     <!-- center of mass of each part besides shoulder (for inertia) -->
     <xacro:property name="CM_XY_UPPER" value="0.076" />
@@ -18,6 +18,7 @@
     <xacro:property name="SHOULDER_pos" value="0.14142" />
     <xacro:property name="UPPER_LEG_pos" value="0.15312" />
-    <xacro:property name="LOWER_LEG_pos" value="0.02546" />
-    <xacro:property name="PRE_WHEEL_pos" value="0.16173" />
+    <xacro:property name="LOWER_LEG_pos" value="0.12546" />
+    <xacro:property name="LOWER_LEG_JOINT_pos" value="0.05" />
+    <xacro:property name="PRE_WHEEL_pos" value="0.285" />
     <xacro:property name="WHEEL_pos" value="0.10183" />
     <xacro:property name="VELOCITY" value="58.17764173" />

File: urdfs/leg.xacro (robot description, xacro)
@@ -277,5 +277,5 @@
                     <axis xyz="0 1 0"/>
                     <limit effort="${MAX_FORCE_LOWERLEG}" lower="${LOWER_LIMIT_PRI}" upper="${UPPER_LIMIT_PRI}" velocity="${VELOCITY}"/>
-                    <origin xyz="0 0 0" rpy="0 0 0" />
+                    <origin xyz="0 ${LOWER_LEG_JOINT_pos} 0" rpy="0 0 0" />
                 </xacro:unless>
                 <xacro:if value="${is_right}">
@@ -283,5 +283,5 @@
                     <!-- RF_LOWER_LEG_JOINT -->
                     <limit effort="${MAX_FORCE_LOWERLEG}" lower="${LOWER_LIMIT_PRI}" upper="${UPPER_LIMIT_PRI}" velocity="${VELOCITY}"/>
-                    <origin xyz="0 0 0" rpy="0 0 0" />
+                    <origin xyz="${LOWER_LEG_JOINT_pos} 0 0" rpy="0 0 0" />
                 </xacro:if>
             </xacro:if>
@@ -291,5 +291,5 @@
                     <!-- LH_LOWER_LEG_JOINT -->
                     <limit effort="${MAX_FORCE_LOWERLEG}" lower="${LOWER_LIMIT_PRI}" upper="${UPPER_LIMIT_PRI}" velocity="${VELOCITY}"/>
-                    <origin xyz="0 0 0" rpy="0 0 0" />
+                    <origin xyz="-${LOWER_LEG_JOINT_pos} 0 0" rpy="0 0 0" />
                 </xacro:unless>
                 <xacro:if value="${is_right}">
@@ -297,5 +297,5 @@
                     <axis xyz="0 -1 0"/>
                     <limit effort="${MAX_FORCE_LOWERLEG}" lower="${LOWER_LIMIT_PRI}" upper="${UPPER_LIMIT_PRI}" velocity="${VELOCITY}"/>
-                    <origin xyz="0 0 0" rpy="0 0 0" />
+                    <origin xyz="0 -${LOWER_LEG_JOINT_pos} 0" rpy="0 0 0" />
                 </xacro:if>
             </xacro:unless>
@@ -424,5 +424,5 @@
                     <!-- LF_PRE_WHEEL_JOINT -->
                     <axis xyz="0 1 0"/>
-                    <limit effort="${MAX_TORQUE_PRE_WHEEL}" lower="-${REV_LIMIT_PRE_WHEEL}" upper="${REV_LIMIT_PRE_WHEEL}" velocity="${VELOCITY}"/>
+                    <limit effort="${MAX_TORQUE_PRE_WHEEL}" lower="0" upper="${REV_LIMIT_PRE_WHEEL}" velocity="${VELOCITY}"/>
                     <origin xyz="0 ${PRE_WHEEL_pos} 0" rpy="0 0 0" />
                 </xacro:unless>
@@ -430,5 +430,5 @@
                     <axis xyz="1 0 0"/>
                     <!-- RF_PRE_WHEEL_JOINT -->
-                    <limit effort="${MAX_TORQUE_PRE_WHEEL}" lower="-${REV_LIMIT_PRE_WHEEL}" upper="${REV_LIMIT_PRE_WHEEL}" velocity="${VELOCITY}"/>
+                    <limit effort="${MAX_TORQUE_PRE_WHEEL}" lower="0" upper="${REV_LIMIT_PRE_WHEEL}" velocity="${VELOCITY}"/>
                     <origin xyz="${PRE_WHEEL_pos} 0 0" rpy="0 0 0" />
                 </xacro:if>
@@ -438,5 +438,5 @@
                     <axis xyz="-1 0  0"/>
                     <!-- LH_PRE_WHEEL_JOINT -->
-                    <limit effort="${MAX_TORQUE_PRE_WHEEL}" lower="-${REV_LIMIT_PRE_WHEEL}" upper="${REV_LIMIT_PRE_WHEEL}" velocity="${VELOCITY}"/>
+                    <limit effort="${MAX_TORQUE_PRE_WHEEL}" lower="0" upper="${REV_LIMIT_PRE_WHEEL}" velocity="${VELOCITY}"/>
                     <origin xyz="-${PRE_WHEEL_pos} 0 0" rpy="0 0 0" />
                 </xacro:unless>
@@ -444,5 +444,5 @@
                     <!-- RF_PRE_WHEEL_JOINT -->
                     <axis xyz="0  -1 0"/>
-                    <limit effort="${MAX_TORQUE_PRE_WHEEL}" lower="-${REV_LIMIT_PRE_WHEEL}" upper="${REV_LIMIT_PRE_WHEEL}" velocity="${VELOCITY}"/>
+                    <limit effort="${MAX_TORQUE_PRE_WHEEL}" lower="0" upper="${REV_LIMIT_PRE_WHEEL}" velocity="${VELOCITY}"/>
                     <origin xyz="0 -${PRE_WHEEL_pos} 0" rpy="0 0 0" />
                 </xacro:if>
