Commit message: final correction of limits and positions

File: urdfs/common.xacro (robot description, xacro)
@@ -3,6 +3,6 @@
     <!-- revolute prismatic limits -->
     <xacro:property name="REV_LIMIT" value="0.785" />
-    <xacro:property name="REV_LIMIT_PRE_WHEEL" value="3.14" />
-    <xacro:property name="LOWER_LIMIT_PRI" value="0" />
+    <xacro:property name="REV_LIMIT_PRE_WHEEL" value="1.57" />
+    <xacro:property name="LOWER_LIMIT_PRI" value="0." />
     <xacro:property name="UPPER_LIMIT_PRI" value="0.2" />
     <!-- center of mass of each part besides shoulder (for inertia) -->
@@ -15,17 +15,14 @@
     <xacro:property name="CM_XY_WHEEL" value="0.051" />
     <xacro:property name="CM_Z_WHEEL" value="0.0" />
-    <!-- These are absoulte distance value, the sign are decided in leg.xacro -->
+    <!-- These are absolute distance value, the sign are decided in leg.xacro -->
     <xacro:property name="SHOULDER_pos" value="0.14142" />
     <xacro:property name="UPPER_LEG_pos" value="0.15312" />
     <xacro:property name="LOWER_LEG_pos" value="0.12546" />
-    <xacro:property name="LOWER_LEG_JOINT_pos" value="0.05" />
+    <xacro:property name="LOWER_LEG_joint_pos" value="0.05" />
     <xacro:property name="PRE_WHEEL_pos" value="0.285" />
     <xacro:property name="WHEEL_pos" value="0.10183" />
     <xacro:property name="VELOCITY" value="58.17764173" />
     <!-- torque limits -->
-    <xacro:property name="MAX_TORQUE_SHOULDER" value="300" />
-    <xacro:property name="MAX_TORQUE_UPPER" value="300" />
-    <xacro:property name="MAX_TORQUE_PRE_WHEEL" value="300" />
-    <xacro:property name="MAX_TORQUE_WHEEL" value="300" />
+    <xacro:property name="MAX_TORQUE" value="300" />
     <xacro:property name="MAX_FORCE_LOWERLEG" value="10000" />
     <!-- material colors -->

File: urdfs/leg.xacro (robot description, xacro)
@@ -15,13 +15,13 @@
             <xacro:if value="${is_front}">
                 <xacro:unless value="${is_right}">
-                    <!-- LF_UPPER_LEG_JOINT -->
+                    <!-- LF_SHOULDER_JOINT -->
                     <axis xyz="1 0 0"/>
-                    <limit effort="${MAX_TORQUE_SHOULDER}" lower="-${REV_LIMIT}" upper="${REV_LIMIT}" velocity="${VELOCITY}"/>
+                    <limit effort="${MAX_TORQUE}" lower="-${REV_LIMIT}" upper="${REV_LIMIT}" velocity="${VELOCITY}"/>
                     <origin xyz="0 ${SHOULDER_pos}  0" rpy="0 0 0" />
                 </xacro:unless>
                 <xacro:if value="${is_right}">
-                    <!-- RF_UPPER_LEG_JOINT -->
+                    <!-- RF_SHOULDER_JOINT -->
                     <axis xyz="0 1 0"/>
-                    <limit effort="${MAX_TORQUE_SHOULDER}" lower="-${REV_LIMIT}" upper="${REV_LIMIT}" velocity="${VELOCITY}"/>
+                    <limit effort="${MAX_TORQUE}" lower="-${REV_LIMIT}" upper="${REV_LIMIT}" velocity="${VELOCITY}"/>
                     <origin xyz="${SHOULDER_pos} 0 0" rpy="0 0 0" />
                 </xacro:if>
@@ -29,7 +29,7 @@
             <xacro:unless value="${is_front}">
                 <xacro:unless value="${is_right}">
-                    <!-- LH_UPPER_LEG_JOINT -->
+                    <!-- LH_SHOULDER_JOINT -->
                     <axis xyz="0 -1 0"/>
-                    <limit effort="${MAX_TORQUE_SHOULDER}" lower="-${REV_LIMIT}" upper="${REV_LIMIT}" velocity="${VELOCITY}"/>
+                    <limit effort="${MAX_TORQUE}" lower="-${REV_LIMIT}" upper="${REV_LIMIT}" velocity="${VELOCITY}"/>
                     <origin xyz="-${SHOULDER_pos} 0 0" rpy="0 0 0" />
                 </xacro:unless>
@@ -37,5 +37,5 @@
                     <!-- RH_UPPER_LEG_JOINT -->
                     <axis xyz="-1 0 0"/>
-                    <limit effort="${MAX_TORQUE_SHOULDER}" lower="-${REV_LIMIT}" upper="${REV_LIMIT}" velocity="${VELOCITY}"/>
+                    <limit effort="${MAX_TORQUE}" lower="-${REV_LIMIT}" upper="${REV_LIMIT}" velocity="${VELOCITY}"/>
                     <origin xyz="0 -${SHOULDER_pos} 0" rpy="0 0 0" />
                 </xacro:if>
@@ -129,5 +129,5 @@
                     <!-- LF_UPPER_LEG_JOINT -->
                     <axis xyz="0 0 1"/>
-                    <limit effort="${MAX_TORQUE_UPPER}" lower="-${REV_LIMIT}" upper="${REV_LIMIT}" velocity="${VELOCITY}"/>
+                    <limit effort="${MAX_TORQUE}" lower="-${REV_LIMIT}" upper="${REV_LIMIT}" velocity="${VELOCITY}"/>
                     <origin xyz="0 0 0" rpy="0 0 0" />
                 </xacro:unless>
@@ -135,5 +135,5 @@
                     <!-- RF_UPPER_LEG_JOINT -->
                     <axis xyz="0 0 1"/>
-                    <limit effort="${MAX_TORQUE_UPPER}" lower="-${REV_LIMIT}" upper="${REV_LIMIT}" velocity="${VELOCITY}"/>
+                    <limit effort="${MAX_TORQUE}" lower="-${REV_LIMIT}" upper="${REV_LIMIT}" velocity="${VELOCITY}"/>
                     <origin xyz="0 0 0" rpy="0 0 0" />
                 </xacro:if>
@@ -143,5 +143,5 @@
                     <!-- LH_UPPER_LEG_JOINT -->
                     <axis xyz="0 0 1"/>
-                    <limit effort="${MAX_TORQUE_UPPER}" lower="-${REV_LIMIT}" upper="${REV_LIMIT}" velocity="${VELOCITY}"/>
+                    <limit effort="${MAX_TORQUE}" lower="-${REV_LIMIT}" upper="${REV_LIMIT}" velocity="${VELOCITY}"/>
                     <origin xyz="0 0 0" rpy="0 0 0" />
                 </xacro:unless>
@@ -149,5 +149,5 @@
                     <!-- RH_UPPER_LEG_JOINT -->
                     <axis xyz="0 0 1"/>
-                    <limit effort="${MAX_TORQUE_UPPER}" lower="-${REV_LIMIT}" upper="${REV_LIMIT}" velocity="${VELOCITY}"/>
+                    <limit effort="${MAX_TORQUE}" lower="-${REV_LIMIT}" upper="${REV_LIMIT}" velocity="${VELOCITY}"/>
                     <origin xyz="0 0 0" rpy="0 0 0" />
                 </xacro:if>
@@ -163,5 +163,5 @@
                     <xacro:unless value="${is_right}">
 			<!-- LF UPPER_LEG -->
-                        <origin xyz="0 ${UPPER_LEG_pos} 0" rpy="0 0 0" />
+			<origin xyz="0 ${UPPER_LEG_pos} 0" rpy="0 0 0" />
                         <geometry>
                             <mesh filename="package://starbot_description/meshes/stl/upper_leg_y.stl"/>
@@ -170,5 +170,5 @@
                     <xacro:if value="${is_right}">
 			<!-- RF UPPER_LEG-->
-                        <origin xyz="${UPPER_LEG_pos} 0 0" rpy="0 0 0" />
+			<origin xyz="${UPPER_LEG_pos} 0 0" rpy="0 0 0" />
                         <geometry>
                             <mesh filename="package://starbot_description/meshes/stl/upper_leg_x.stl"/>
@@ -179,5 +179,5 @@
                     <xacro:unless value="${is_right}">
 			<!-- LH UPPER_LEG -->
-                        <origin xyz="-${UPPER_LEG_pos} 0 0" rpy="0 0 0" />
+			<origin xyz="-${UPPER_LEG_pos} 0 0" rpy="0 0 0" />
                         <geometry>
                             <mesh filename="package://starbot_description/meshes/stl/upper_leg_nx.stl"/>
@@ -186,5 +186,5 @@
                     <xacro:if value="${is_right}">
 		        <!-- RH UPPER_LEG -->
-                        <origin xyz="0 -${UPPER_LEG_pos} 0" rpy="0 0 0" />
+		        <origin xyz="0 -${UPPER_LEG_pos} 0" rpy="0 0 0" />
                         <geometry>
                             <mesh filename="package://starbot_description/meshes/stl/upper_leg_ny.stl"/>
@@ -199,5 +199,5 @@
                     <xacro:unless value="${is_right}">
                         <!-- LF UPPER_LEG -->
-			            <origin xyz="0 ${UPPER_LEG_pos} 0" rpy="0 0 0" />
+			<origin xyz="0 ${UPPER_LEG_pos} 0" rpy="0 0 0" />
                         <geometry>
                             <mesh filename="package://starbot_description/meshes/stl/upper_leg_y.stl"/>
@@ -206,5 +206,5 @@
                     <xacro:if value="${is_right}">
                         <!-- RF UPPER_LEG -->
-       			        <origin xyz="${UPPER_LEG_pos} 0 0" rpy="0 0 0" />
+       			<origin xyz="${UPPER_LEG_pos} 0 0" rpy="0 0 0" />
                         <geometry>
                             <mesh filename="package://starbot_description/meshes/stl/upper_leg_x.stl"/>
@@ -215,5 +215,5 @@
                     <xacro:unless value="${is_right}">
                         <!-- LH UPPER_LEG -->
-			            <origin xyz="-${UPPER_LEG_pos} 0 0" rpy="0 0 0" />
+			<origin xyz="-${UPPER_LEG_pos} 0 0" rpy="0 0 0" />
                         <geometry>
                             <mesh filename="package://starbot_description/meshes/stl/upper_leg_nx.stl"/>
@@ -222,5 +222,5 @@
                     <xacro:if value="${is_right}">
                         <!-- RH UPPER_LEG-->
-			            <origin xyz=" 0 -${UPPER_LEG_pos} 0" rpy="0 0 0" />
+			<origin xyz="0 -${UPPER_LEG_pos} 0" rpy="0 0 0" />
                         <geometry>
                             <mesh filename="package://starbot_description/meshes/stl/upper_leg_ny.stl"/>
@@ -234,5 +234,5 @@
                         <!-- LF UPPER_LEG -->
                         <inertial>
-                    		<origin xyz="0 ${CM_XY_UPPER} ${CM_Z_UPPER}" rpy="0 0 0"/>
+                    		<origin xyz="0 ${UPPER_LEG_pos} 0" rpy="0 0 0"/>
                     		<mass value="2.3"/>
                     		<inertia ixx="0.01246" ixy="0" ixz="0" iyy="0.00148" iyz="0" izz="0.01246"/>
@@ -242,5 +242,5 @@
                         <!-- RF UPPER_LEG -->
                         <inertial>
-                    		<origin xyz="${CM_XY_UPPER} 0 ${CM_Z_UPPER}" rpy="0 0 0"/>
+                    		<origin xyz="${UPPER_LEG_pos} 0 0" rpy="0 0 0"/>
                     		<mass value="2.3"/>
                     		<inertia ixx="0.00148" ixy="0" ixz="0" iyy="0.01246" iyz="0" izz="0.00148"/>
@@ -252,5 +252,5 @@
                         <!-- LH UPPER_LEG -->
                         <inertial>
-                    		<origin xyz="-${CM_XY_UPPER} 0 ${CM_Z_UPPER}" rpy="0 0 0"/>
+                    		<origin xyz="-${UPPER_LEG_pos} 0 0" rpy="0 0 0"/>
                     		<mass value="2.3"/>
                     		<inertia ixx="0.00148" ixy="0" ixz="0" iyy="0.01246" iyz="0" izz="0.00148"/>
@@ -260,5 +260,5 @@
                         <!-- RH UPPER_LEG-->
                         <inertial>
-                    		<origin xyz="0 -${CM_XY_UPPER} ${CM_Z_UPPER}" rpy="0 0 0"/>
+                    		<origin xyz="0 -${UPPER_LEG_pos} 0" rpy="0 0 0"/>
                     		<mass value="2.3"/>
                     		<inertia ixx="0.01246" ixy="0" ixz="0" iyy="0.00148" iyz="0" izz="0.01246"/>
@@ -277,5 +277,5 @@
                     <axis xyz="0 1 0"/>
                     <limit effort="${MAX_FORCE_LOWERLEG}" lower="${LOWER_LIMIT_PRI}" upper="${UPPER_LIMIT_PRI}" velocity="${VELOCITY}"/>
-                    <origin xyz="0 ${LOWER_LEG_JOINT_pos} 0" rpy="0 0 0" />
+                    <origin xyz="0 ${LOWER_LEG_joint_pos} 0" rpy="0 0 0" />
                 </xacro:unless>
                 <xacro:if value="${is_right}">
@@ -283,5 +283,5 @@
                     <!-- RF_LOWER_LEG_JOINT -->
                     <limit effort="${MAX_FORCE_LOWERLEG}" lower="${LOWER_LIMIT_PRI}" upper="${UPPER_LIMIT_PRI}" velocity="${VELOCITY}"/>
-                    <origin xyz="${LOWER_LEG_JOINT_pos} 0 0" rpy="0 0 0" />
+                    <origin xyz="${LOWER_LEG_joint_pos} 0 0" rpy="0 0 0" />
                 </xacro:if>
             </xacro:if>
@@ -291,5 +291,5 @@
                     <!-- LH_LOWER_LEG_JOINT -->
                     <limit effort="${MAX_FORCE_LOWERLEG}" lower="${LOWER_LIMIT_PRI}" upper="${UPPER_LIMIT_PRI}" velocity="${VELOCITY}"/>
-                    <origin xyz="-${LOWER_LEG_JOINT_pos} 0 0" rpy="0 0 0" />
+                    <origin xyz="-${LOWER_LEG_joint_pos} 0 0" rpy="0 0 0" />
                 </xacro:unless>
                 <xacro:if value="${is_right}">
@@ -297,5 +297,5 @@
                     <axis xyz="0 -1 0"/>
                     <limit effort="${MAX_FORCE_LOWERLEG}" lower="${LOWER_LIMIT_PRI}" upper="${UPPER_LIMIT_PRI}" velocity="${VELOCITY}"/>
-                    <origin xyz="0 -${LOWER_LEG_JOINT_pos} 0" rpy="0 0 0" />
+                    <origin xyz="0 -${LOWER_LEG_joint_pos} 0" rpy="0 0 0" />
                 </xacro:if>
             </xacro:unless>
@@ -310,5 +310,5 @@
                     <xacro:unless value="${is_right}">
                         <!-- LF LOWER_LEG -->
-		                <origin xyz="0 ${LOWER_LEG_pos} 0" rpy="0 0 0" />
+                        <origin xyz="0 ${LOWER_LEG_pos} 0" rpy="0 0 0" />
                         <geometry>
                             <mesh filename="package://starbot_description/meshes/stl/lower_leg_y.stl"/>
@@ -346,5 +346,5 @@
                     <xacro:unless value="${is_right}">
                         <!-- LF LOWER_LEG -->
-                        <origin xyz="0 ${LOWER_LEG_pos} 0" rpy="0 0 0" />
+                         <origin xyz="0 ${LOWER_LEG_pos} 0" rpy="0 0 0" />
                         <geometry>
                             <mesh filename="package://starbot_description/meshes/stl/lower_leg_y.stl"/>
@@ -369,5 +369,5 @@
                     <xacro:if value="${is_right}">
                         <!-- RH LOWER_LEG-->
-                        <origin xyz="0 -${LOWER_LEG_pos} 0" rpy="0 0 0" />
+                         <origin xyz="0 -${LOWER_LEG_pos} 0" rpy="0 0 0" />
                         <geometry>
                             <mesh filename="package://starbot_description/meshes/stl/lower_leg_ny.stl"/>
@@ -381,5 +381,5 @@
                         <!-- LF LOWER_LEG -->
                         <inertial>
-                    		<origin xyz="0 ${CM_XY_LOWER} ${CM_Z_LOWER}" rpy="0 0 0"/>
+                    		<origin xyz="0 ${LOWER_LEG_pos} 0" rpy="0 0 0"/>
                     		<mass value="2.36"/>
                     		<inertia ixx="0.00767" ixy="0" ixz="0" iyy="0.00056" iyz="0" izz="0.00767"/>
@@ -389,5 +389,5 @@
                         <!-- RF LOWER_LEG -->
                         <inertial>
-                    		<origin xyz="${CM_XY_LOWER} 0 ${CM_Z_LOWER}" rpy="0 0 0"/>
+                    		<origin xyz="${LOWER_LEG_pos} 0 0" rpy="0 0 0"/>
                     		<mass value="2.36"/>
                     		<inertia ixx="0.00056" ixy="0" ixz="0" iyy="0.00767" iyz="0" izz="0.00056"/>
@@ -399,5 +399,5 @@
                         <!-- LH LOWER_LEG -->
                         <inertial>
-                    		<origin xyz="-${CM_XY_LOWER} 0 ${CM_Z_LOWER}" rpy="0 0 0"/>
+                    		<origin xyz="-${LOWER_LEG_pos} 0 0" rpy="0 0 0"/>
                     		<mass value="2.36"/>
                     		<inertia ixx="0.00056" ixy="0" ixz="0" iyy="0.00767" iyz="0" izz="0.00056"/>
@@ -407,5 +407,5 @@
                         <!-- RH LOWER_LEG-->
                         <inertial>
-                    		<origin xyz="0 -${CM_XY_LOWER} ${CM_Z_LOWER}" rpy="0 0 0"/>
+                    		<origin xyz="0 -${LOWER_LEG_pos} 0" rpy="0 0 0"/>
                     		<mass value="2.36"/>
                     		<inertia ixx="0.00767" ixy="0" ixz="0" iyy="0.00056" iyz="0" izz="0.00767"/>
@@ -424,5 +424,5 @@
                     <!-- LF_PRE_WHEEL_JOINT -->
                     <axis xyz="0 1 0"/>
-                    <limit effort="${MAX_TORQUE_PRE_WHEEL}" lower="0" upper="${REV_LIMIT_PRE_WHEEL}" velocity="${VELOCITY}"/>
+                    <limit effort="${MAX_TORQUE}" lower="-${REV_LIMIT_PRE_WHEEL}" upper="${REV_LIMIT_PRE_WHEEL}" velocity="${VELOCITY}"/>
                     <origin xyz="0 ${PRE_WHEEL_pos} 0" rpy="0 0 0" />
                 </xacro:unless>
@@ -430,5 +430,5 @@
                     <axis xyz="1 0 0"/>
                     <!-- RF_PRE_WHEEL_JOINT -->
-                    <limit effort="${MAX_TORQUE_PRE_WHEEL}" lower="0" upper="${REV_LIMIT_PRE_WHEEL}" velocity="${VELOCITY}"/>
+                    <limit effort="${MAX_TORQUE}" lower="-${REV_LIMIT_PRE_WHEEL}" upper="${REV_LIMIT_PRE_WHEEL}" velocity="${VELOCITY}"/>
                     <origin xyz="${PRE_WHEEL_pos} 0 0" rpy="0 0 0" />
                 </xacro:if>
@@ -438,5 +438,5 @@
                     <axis xyz="-1 0  0"/>
                     <!-- LH_PRE_WHEEL_JOINT -->
-                    <limit effort="${MAX_TORQUE_PRE_WHEEL}" lower="0" upper="${REV_LIMIT_PRE_WHEEL}" velocity="${VELOCITY}"/>
+                    <limit effort="${MAX_TORQUE}" lower="-${REV_LIMIT_PRE_WHEEL}" upper="${REV_LIMIT_PRE_WHEEL}" velocity="${VELOCITY}"/>
                     <origin xyz="-${PRE_WHEEL_pos} 0 0" rpy="0 0 0" />
                 </xacro:unless>
@@ -444,5 +444,5 @@
                     <!-- RF_PRE_WHEEL_JOINT -->
                     <axis xyz="0  -1 0"/>
-                    <limit effort="${MAX_TORQUE_PRE_WHEEL}" lower="0" upper="${REV_LIMIT_PRE_WHEEL}" velocity="${VELOCITY}"/>
+                    <limit effort="${MAX_TORQUE}" lower="-${REV_LIMIT_PRE_WHEEL}" upper="${REV_LIMIT_PRE_WHEEL}" velocity="${VELOCITY}"/>
                     <origin xyz="0 -${PRE_WHEEL_pos} 0" rpy="0 0 0" />
                 </xacro:if>
@@ -459,4 +459,5 @@
                     <xacro:unless value="${is_right}">
                         <!-- LF PRE_WHEEL -->
+                        <!--we need mesh geometry otherwise strange behaviour happens-->
                         <geometry>
                             <mesh filename="package://starbot_description/meshes/stl/joint_wheel_y.stl"/>
@@ -523,5 +524,5 @@
                         <!-- PRE_WHEEL_LEG -->
                         <inertial>
-                    		<origin xyz="0 ${CM_XY_PRE_WHEEL} ${CM_Z_PRE_WHEEL}" rpy="0 0 0"/>
+                    		<origin xyz="0 ${PRE_WHEEL_pos} 0" rpy="0 0 0"/>
                     		<mass value="0.66"/>
                     		<inertia ixx="0.00024" ixy="0" ixz="0" iyy="0.00016" iyz="0" izz="0.00024"/>
@@ -531,5 +532,5 @@
                         <!-- PRE_WHEEL_LEG -->
                         <inertial>
-                    		<origin xyz="${CM_XY_PRE_WHEEL} 0 ${CM_Z_PRE_WHEEL}" rpy="0 0 0"/>
+                    		<origin xyz="${PRE_WHEEL_pos} 0 0" rpy="0 0 0"/>
                     		<mass value="0.66"/>
                     		<inertia ixx="0.00016" ixy="0" ixz="0" iyy="0.00024" iyz="0" izz="0.00016"/>
@@ -541,5 +542,5 @@
                         <!-- PRE_WHEEL_LEG -->
                         <inertial>
-                    		<origin xyz="-${CM_XY_PRE_WHEEL} 0 ${CM_Z_PRE_WHEEL}" rpy="0 0 0"/>
+                    		<origin xyz="-${PRE_WHEEL_pos} 0 0" rpy="0 0 0"/>
                     		<mass value="0.66"/>
                     		<inertia ixx="0.00016" ixy="0" ixz="0" iyy="0.00024" iyz="0" izz="0.00016"/>
@@ -549,5 +550,5 @@
                         <!-- PRE_WHEEL_LEG-->
                         <inertial>
-                    		<origin xyz="0 -${CM_XY_PRE_WHEEL} ${CM_Z_PRE_WHEEL}" rpy="0 0 0"/>
+                    		<origin xyz="0 -${PRE_WHEEL_pos} 0" rpy="0 0 0"/>
                     		<mass value="0.66"/>
                     		<inertia ixx="0.00024" ixy="0" ixz="0" iyy="0.00016" iyz="0" izz="0.00024"/>
@@ -566,5 +567,4 @@
                     <!-- LF_WHEEL_JOINT -->
                     <axis xyz="1 0 0"/>
-                    <limit effort="${MAX_TORQUE_WHEEL}" velocity="${VELOCITY}"/>
                     <origin xyz="0 ${WHEEL_pos} 0" rpy="0 0 0" />
                 </xacro:unless>
@@ -572,5 +572,4 @@
                     <axis xyz="0 1 0"/>
                     <!-- RF_WHEEL_JOINT -->
-                    <limit effort="${MAX_TORQUE_WHEEL}" velocity="${VELOCITY}"/>
                     <origin xyz="${WHEEL_pos} 0 0" rpy="0 0 0" />
                 </xacro:if>
@@ -580,5 +579,4 @@
                     <axis xyz="0 -1 0"/>
                     <!-- LH_WHEEL_JOINT -->
-                    <limit effort="${MAX_TORQUE_WHEEL}" velocity="${VELOCITY}"/>
                     <origin xyz="-${WHEEL_pos} 0 0" rpy="0 0 0" />
                 </xacro:unless>
@@ -586,5 +584,4 @@
                     <!-- RF_WHEEL_JOINT -->
                     <axis xyz="-1 0 0"/>
-                    <limit effort="${MAX_TORQUE_WHEEL}" velocity="${VELOCITY}"/>
                     <origin xyz="0 -${WHEEL_pos} 0" rpy="0 0 0" />
                 </xacro:if>
@@ -667,5 +664,5 @@
                         <!-- PRE_WHEEL_LEG -->
                         <inertial>
-                    		<origin xyz="0 ${CM_XY_WHEEL} ${CM_Z_WHEEL}" rpy="0 0 0"/>
+                    		<origin xyz="0 ${WHEEL_pos} 0" rpy="0 0 0"/>
                     		<mass value="1.0"/>
                     		<inertia ixx="0.00224" ixy="0" ixz="0" iyy="0.00121" iyz="0" izz="0.00224"/>
@@ -675,5 +672,5 @@
                         <!-- PRE_WHEEL_LEG -->
                         <inertial>
-                    		<origin xyz="${CM_XY_WHEEL} 0 ${CM_Z_WHEEL}" rpy="0 0 0"/>
+                    		<origin xyz="${WHEEL_pos} 0 0" rpy="0 0 0"/>
                     		<mass value="1.0"/>
                     		<inertia ixx="0.00121" ixy="0" ixz="0" iyy="0.00224" iyz="0" izz="0.00121"/>
@@ -685,5 +682,5 @@
                         <!-- PRE_WHEEL_LEG -->
                         <inertial>
-                    		<origin xyz="-${CM_XY_WHEEL}  0 ${CM_Z_WHEEL}" rpy="0 0 0"/>
+                    		<origin xyz="-${WHEEL_pos}  0 0" rpy="0 0 0"/>
                     		<mass value="1.0"/>
                     		<inertia ixx="0.00121" ixy="0" ixz="0" iyy="0.00224" iyz="0" izz="0.00121"/>
@@ -693,5 +690,5 @@
                         <!-- PRE_WHEEL_LEG-->
                         <inertial>
-                    		<origin xyz="0 -${CM_XY_WHEEL} ${CM_Z_WHEEL}" rpy="0 0 0"/>
+                    		<origin xyz="0 -${WHEEL_pos} 0" rpy="0 0 0"/>
                     		<mass value="1.0"/>
                     		<inertia ixx="0.00224" ixy="0" ixz="0" iyy="0.00121" iyz="0" izz="0.00224"/>
