Commit message: temporarly commented collision for lower leg and setting lower values for the prismatic joints cause pipe diameter is too small

File: urdfs/common.xacro (robot description, xacro)
@@ -4,5 +4,5 @@
     <xacro:property name="REV_LIMIT" value="0.785" />
     <xacro:property name="REV_LIMIT_PRE_WHEEL" value="1.57" />
-    <xacro:property name="LOWER_LIMIT_PRI" value="0." />
+    <xacro:property name="LOWER_LIMIT_PRI" value="-0.15" />
     <xacro:property name="UPPER_LIMIT_PRI" value="0.2" />
     <!-- center of mass of each part besides shoulder (for inertia) -->

File: urdfs/leg.xacro (robot description, xacro)
@@ -310,38 +310,4 @@
             </visual>
             <!--COLLISION-->
-            <collision>
-                <xacro:if value="${is_front}">
-                    <xacro:unless value="${is_right}">
-                        <!-- LF LOWER_LEG -->
-                         <origin xyz="0 ${LOWER_LEG_pos} 0" rpy="0 0 0" />
-                        <geometry>
-                            <mesh filename="package://starbot_description/meshes/stl/lower_leg_y.stl" />
-                        </geometry>
-                    </xacro:unless>
-                    <xacro:if value="${is_right}">
-                        <!-- RF LOWER_LEG -->
-                        <origin xyz="${LOWER_LEG_pos} 0 0" rpy="0 0 0" />
-                        <geometry>
-                            <mesh filename="package://starbot_description/meshes/stl/lower_leg_x.stl"/>
-                        </geometry>
-                    </xacro:if>
-                </xacro:if>
-                <xacro:unless value="${is_front}">
-                    <xacro:unless value="${is_right}">
-                        <!-- LH LOWER_LEG -->
-                        <origin xyz="-${LOWER_LEG_pos} 0 0" rpy="0 0 0" />
-                        <geometry>
-                            <mesh filename="package://starbot_description/meshes/stl/lower_leg_nx.stl" />
-                        </geometry>
-                    </xacro:unless>
-                    <xacro:if value="${is_right}">
-                        <!-- RH LOWER_LEG-->
-                         <origin xyz="0 -${LOWER_LEG_pos} 0" rpy="0 0 0" />
-                        <geometry>
-                            <mesh filename="package://starbot_description/meshes/stl/lower_leg_ny.stl"/>
-                        </geometry>
-                    </xacro:if>
-                </xacro:unless>
-            </collision>
             <!-- LOWER LEG LINK INERTIAL -->
             <xacro:if value="${is_front}">

Commit message: parameters correction to stardard values

File: urdfs/common.xacro (robot description, xacro)
@@ -4,5 +4,5 @@
     <xacro:property name="REV_LIMIT" value="0.785" />
     <xacro:property name="REV_LIMIT_PRE_WHEEL" value="1.57" />
-    <xacro:property name="LOWER_LIMIT_PRI" value="-0.15" />
+    <xacro:property name="LOWER_LIMIT_PRI" value="0." />
     <xacro:property name="UPPER_LIMIT_PRI" value="0.2" />
     <!-- center of mass of each part besides shoulder (for inertia) -->
