Commit message: fixed inertia and color application

File: robots/starbot.srdf.xacro (robot description, xacro)
@@ -1,31 +1,39 @@
 <?xml version="1.0" ?>
-<robot name="solo" xmlns:xacro="http://ros.org/wiki/xacro">
-	<xacro:arg name="flywheel" default="false"/>
+<robot name="starbot" xmlns:xacro="http://ros.org/wiki/xacro">
+	<xacro:arg name="new_gazebo_version" default="false"/>
     <!-- left front leg -->
     <group name="lf_leg">
-        <joint name="lf_haa_joint" />
-        <joint name="lf_hfe_joint" />
-        <joint name="lf_kfe_joint" />
+        <joint name="lf_bs_joint" />
+        <joint name="lf_upper_leg_joint" />
+        <joint name="lf_lower_leg_joint" />
+        <joint name="lf_pre_wheel_joint" />
+        <joint name="lf_wheel_joint" />
         <chain base_link="base_link" tip_link="lf_foot" />
     </group>
     <!-- right front leg -->
     <group name="rf_leg">
-        <joint name="rf_haa_joint" />
-        <joint name="rf_hfe_joint" />
-        <joint name="rf_kfe_joint" />
+        <joint name="rf_bs_joint" />
+        <joint name="rf_upper_leg_joint" />
+        <joint name="rf_lower_leg_joint" />
+        <joint name="rf_pre_wheel_joint" />
+        <joint name="rf_wheel_joint" />
         <chain base_link="base_link" tip_link="rf_foot" />
     </group>
     <!-- left hind leg -->
     <group name="lh_leg">
-        <joint name="lh_haa_joint" />
-        <joint name="lh_hfe_joint" />
-        <joint name="lh_kfe_joint" />
+        <joint name="lh_bs_joint" />
+        <joint name="lh_upper_leg_joint" />
+        <joint name="lh_lower_leg_joint" />
+        <joint name="lh_pre_wheel_joint" />
+        <joint name="lh_wheel_joint" />
         <chain base_link="base_link" tip_link="lh_foot" />
     </group>
     <!-- right hind leg -->
     <group name="rh_leg">
-        <joint name="rh_haa_joint" />
-        <joint name="rh_hfe_joint" />
-        <joint name="rh_kfe_joint" />
+        <joint name="rh_bs_joint" />
+        <joint name="rh_upper_leg_joint" />
+        <joint name="rh_lower_leg_joint" />
+        <joint name="rh_pre_wheel_joint" />
+        <joint name="rh_wheel_joint" />
         <chain base_link="base_link" tip_link="rh_foot" />
     </group>
@@ -42,16 +50,24 @@
      <group_state name="home" group="all_legs">
 		    <joint name="floating_base_joint" value="0. 0. 0.223 0. 0. 0. 1." />
-                    <joint name="lf_haa_joint" value="0.0" />
-                    <joint name="lf_hfe_joint" value="0.75" />
-                    <joint name="lf_kfe_joint" value="-1.5" />
-                    <joint name="lh_haa_joint" value="0.0" />
-                    <joint name="lh_hfe_joint" value="-0.75" />
-                    <joint name="lh_kfe_joint" value="1.5" />
-                    <joint name="rf_haa_joint" value="-0.0" />
-                    <joint name="rf_hfe_joint" value="0.75" />
-                    <joint name="rf_kfe_joint" value="-1.5" />
-                    <joint name="rh_haa_joint" value="-0.0" />
-                    <joint name="rh_hfe_joint" value="-0.75" />
-                    <joint name="rh_kfe_joint" value="1.5" />
+		    <joint name="lf_bs_joint" value="0.0"  />
+		    <joint name="lf_upper_leg_joint" value="0.0"  />
+		    <joint name="lf_lower_leg_joint" value="0.0"  />
+		    <joint name="lf_pre_wheel_joint" value="0.0"  />
+		    <joint name="lf_wheel_joint" value="0.0"  />
+		    <joint name="rf_bs_joint" value="0.0"  />
+		    <joint name="rf_upper_leg_joint" value="0.0"  />
+		    <joint name="rf_lower_leg_joint" value="0.0"  />
+		    <joint name="rf_pre_wheel_joint" value="0.0"  />
+		    <joint name="rf_wheel_joint" value="0.0"  />
+		    <joint name="lh_bs_joint" value="0.0"  />
+		    <joint name="lh_upper_leg_joint" value="0.0"  />
+		    <joint name="lh_lower_leg_joint" value="0.0"  />
+		    <joint name="lh_pre_wheel_joint" value="0.0"  />
+		    <joint name="lh_wheel_joint" value="0.0"  />
+		    <joint name="rh_bs_joint" value="0.0"  />
+		    <joint name="rh_upper_leg_joint" value="0.0"  />
+		    <joint name="rh_lower_leg_joint" value="0.0"  />
+		    <joint name="rh_pre_wheel_joint" value="0.0"  />
+		    <joint name="rh_wheel_joint" value="0.0"  />
      </group_state>
 </robot>

File: robots/starbot.urdf.xacro (robot description, xacro)
@@ -37,6 +37,6 @@
            <mesh filename="package://starbot_description/meshes/stl/octagon.stl"/>
         </geometry>
-        <material name="body_color">
-        	<color rgba="0.8 0.8 0.8 1.0"/>
+        <material name="yellow">
+        	<color rgba="0.8 0.6 0.0 1.0"/>
         </material>
       </visual>

File: urdfs/leg.xacro (robot description, xacro)
@@ -12,4 +12,13 @@
     <xacro:property name="PRE_WHEEL_pos" value="0.16173" />
     <xacro:property name="WHEEL_pos" value="0.10183" />
+    <material name="orange">
+     <color rgba="0.800 0.331 0.183 1.0"/>
+    </material>
+    <material name="blue">
+     <color rgba="0.051 0.144 0.800 1.0"/>
+    </material>
+    <material name="gray">
+     <color rgba="0.638 0.779 0.819 1.0"/>
+    </material>
     <!-- This macro has for purpose to define a leg -->
     <xacro:macro name="leg" params="name parent is_front is_right robot_name">
@@ -84,7 +93,5 @@
                     </xacro:if>
                 </xacro:unless>
-                <material name="shoulder_color">
-                    <color rgba="0.8 0.8 0.8 1.0"/>
-                </material>
+                <material name="orange"/>
             </visual>
             <!--COLLISION-->
@@ -119,7 +126,4 @@
                     </xacro:if>
                 </xacro:unless>
-                <material name="collision_color">
-                    <color rgba="0.8 0.8 0.8 1.0"/>
-                </material>
             </collision>
             <!--INERTIAL -->
@@ -200,7 +204,5 @@
                     </xacro:if>
                 </xacro:unless>
-                <material name="upper_leg_color">
-                <color rgba="0.8 0.8 0.8 1.0"/>
-                </material>
+                <material name="orange"/>
             </visual>
             <!--COLLISION-->
@@ -235,25 +237,42 @@
                     </xacro:if>
                 </xacro:unless>
-                <material name="collision_color">
-                    <color rgba="0.8 0.8 0.8 1.0"/>
-                </material>
             </collision>
             <!-- UPPER LEG LINK INERTIAL -->
-            <xacro:unless value="${is_right}">
-                <!-- Left upper leg inertia -->
-                <inertial>
-                    <origin xyz="0 0 0" rpy="0 0 0"/>
-                    <mass value="2.3"/>
-                    <inertia ixx="0.01259" ixy="0" ixz="0" iyy="0.00147" iyz="0" izz="0.01259"/>
-                </inertial>
-            </xacro:unless>
-            <xacro:if value="${is_right}">
-                <!-- Right upper leg inertia -->
-                <inertial>
-                    <origin xyz="0 0 0" rpy="0 0 0"/>
-                    <mass value="2.3"/>
-                    <inertia ixx="0.00147" ixy="0" ixz="0" iyy="0.01259" iyz="0" izz="0.01259"/>
-                </inertial>
-            </xacro:if>
+            <xacro:if value="${is_front}">
+                    <xacro:unless value="${is_right}">
+                        <!-- LF UPPER_LEG -->
+                        <inertial>
+                    		<origin xyz="0 0 0" rpy="0 0 0"/>
+                    		<mass value="2.3"/>
+                    		<inertia ixx="0.01246" ixy="0" ixz="0" iyy="0.00148" iyz="0" izz="0.01246"/>
+                	</inertial>
+                    </xacro:unless>
+                    <xacro:if value="${is_right}">
+                        <!-- RF UPPER_LEG -->
+                        <inertial>
+                    		<origin xyz="0 0 0" rpy="0 0 0"/>
+                    		<mass value="2.3"/>
+                    		<inertia ixx="0.00148" ixy="0" ixz="0" iyy="0.01246" iyz="0" izz="0.00148"/>
+                	</inertial>
+                    </xacro:if>
+                </xacro:if>
+                <xacro:unless value="${is_front}">
+                    <xacro:unless value="${is_right}">
+                        <!-- LH UPPER_LEG -->
+                        <inertial>
+                    		<origin xyz="0 0 0" rpy="0 0 0"/>
+                    		<mass value="2.3"/>
+                    		<inertia ixx="0.00148" ixy="0" ixz="0" iyy="0.01246" iyz="0" izz="0.00148"/>
+                	</inertial>
+                    </xacro:unless>
+                    <xacro:if value="${is_right}">
+                        <!-- RH UPPER_LEG-->
+                        <inertial>
+                    		<origin xyz="0 0 0" rpy="0 0 0"/>
+                    		<mass value="2.3"/>
+                    		<inertia ixx="0.01246" ixy="0" ixz="0" iyy="0.00148" iyz="0" izz="0.01246"/>
+                	</inertial>
+                    </xacro:if>
+                </xacro:unless>
         </link>
         <!--LOWER LEG JOINT-->
@@ -328,7 +347,5 @@
                     </xacro:if>
                 </xacro:unless>
-                <material name="upper_leg_color">
-                    <color rgba="0.3 0.3 0.6 1.0"/>
-                </material>
+                <material name="orange"/>
             </visual>
             <!--COLLISION-->
@@ -363,25 +380,42 @@
                     </xacro:if>
                 </xacro:unless>
-                <material name="collision_color">
-                    <color rgba="0.8 0.8 0.8 1.0"/>
-                </material>
             </collision>
             <!-- LOWER LEG LINK INERTIAL -->
-            <xacro:unless value="${is_right}">
-                <!-- Left lower leg inertia -->
-                <inertial>
-                    <origin xyz="0 0 0" rpy="0 0 0"/>
-                    <mass value="2.36"/>
-                    <inertia ixx="0.00056" ixy="0" ixz="0" iyy="0.00056" iyz="0" izz="0.00049"/>
-                </inertial>
-            </xacro:unless>
-            <xacro:if value="${is_right}">
-                <!-- Right lower leg inertia -->
-                <inertial>
-                    <origin xyz="0 0 0" rpy="0 0 0"/>
-                    <mass value="2.36"/>
-                    <inertia ixx="0.00954" ixy="0" ixz="0" iyy="0.00954" iyz="0" izz="0.01845"/>
-                </inertial>
-            </xacro:if>
+            <xacro:if value="${is_front}">
+                    <xacro:unless value="${is_right}">
+                        <!-- LF LOWER_LEG -->
+                        <inertial>
+                    		<origin xyz="0 0 0" rpy="0 0 0"/>
+                    		<mass value="2.36"/>
+                    		<inertia ixx="0.00767" ixy="0" ixz="0" iyy="0.00056" iyz="0" izz="0.00767"/>
+                	</inertial>
+                    </xacro:unless>
+                    <xacro:if value="${is_right}">
+                        <!-- RF LOWER_LEG -->
+                        <inertial>
+                    		<origin xyz="0 0 0" rpy="0 0 0"/>
+                    		<mass value="2.36"/>
+                    		<inertia ixx="0.00056" ixy="0" ixz="0" iyy="0.00767" iyz="0" izz="0.00056"/>
+                	</inertial>
+                    </xacro:if>
+                </xacro:if>
+                <xacro:unless value="${is_front}">
+                    <xacro:unless value="${is_right}">
+                        <!-- LH LOWER_LEG -->
+                        <inertial>
+                    		<origin xyz="0 0 0" rpy="0 0 0"/>
+                    		<mass value="2.36"/>
+                    		<inertia ixx="0.00056" ixy="0" ixz="0" iyy="0.00767" iyz="0" izz="0.00056"/>
+                	</inertial>
+                    </xacro:unless>
+                    <xacro:if value="${is_right}">
+                        <!-- RH LOWER_LEG-->
+                        <inertial>
+                    		<origin xyz="0 0 0" rpy="0 0 0"/>
+                    		<mass value="2.36"/>
+                    		<inertia ixx="0.00767" ixy="0" ixz="0" iyy="0.00056" iyz="0" izz="0.00767"/>
+                	</inertial>
+                    </xacro:if>
+                </xacro:unless>
         </link>
         <!--PRE WHEEL JOINT-->
@@ -456,7 +490,5 @@
                     </xacro:if>
                 </xacro:unless>
-                <material name="upper_leg_color">
-                    <color rgba="0.3 0.3 0.6 1.0"/>
-                </material>
+                <material name="gray"/>
             </visual>
             <!--COLLISION-->
@@ -491,25 +523,42 @@
                     </xacro:if>
                 </xacro:unless>
-                <material name="collision_color">
-                    <color rgba="0.8 0.8 0.8 1.0"/>
-                </material>
             </collision>
             <!-- PRE WHEEL LINK INERTIAL -->
-            <xacro:unless value="${is_right}">
-                <!-- Left pre_wheel inertia -->
-                <inertial>
-                    <origin xyz="0 0 0" rpy="0 0 0"/>
-                    <mass value="0.66"/>
-                    <inertia ixx="0.00015" ixy="0" ixz="0" iyy="0.00015" iyz="0" izz="0.00013"/>
-                </inertial>
-            </xacro:unless>
-            <xacro:if value="${is_right}">
-                <!-- Right pre_wheel inertia -->
-                <inertial>
-                    <origin xyz="0 0 0" rpy="0 0 0"/>
-                    <mass value="0.66"/>
-                    <inertia ixx="0.00029" ixy="0" ixz="0" iyy="0.00029" iyz="0" izz="0.00041"/>
-                </inertial>
-            </xacro:if>
+            <xacro:if value="${is_front}">
+                    <xacro:unless value="${is_right}">
+                        <!-- PRE_WHEEL_LEG -->
+                        <inertial>
+                    		<origin xyz="0 0 0" rpy="0 0 0"/>
+                    		<mass value="0.66"/>
+                    		<inertia ixx="0.00024" ixy="0" ixz="0" iyy="0.00016" iyz="0" izz="0.00024"/>
+                	</inertial>
+                    </xacro:unless>
+                    <xacro:if value="${is_right}">
+                        <!-- PRE_WHEEL_LEG -->
+                        <inertial>
+                    		<origin xyz="0 0 0" rpy="0 0 0"/>
+                    		<mass value="0.66"/>
+                    		<inertia ixx="0.00016" ixy="0" ixz="0" iyy="0.00024" iyz="0" izz="0.00016"/>
+                	</inertial>
+                    </xacro:if>
+                </xacro:if>
+                <xacro:unless value="${is_front}">
+                    <xacro:unless value="${is_right}">
+                        <!-- PRE_WHEEL_LEG -->
+                        <inertial>
+                    		<origin xyz="0 0 0" rpy="0 0 0"/>
+                    		<mass value="0.66"/>
+                    		<inertia ixx="0.00016" ixy="0" ixz="0" iyy="0.00024" iyz="0" izz="0.00016"/>
+                	</inertial>
+                    </xacro:unless>
+                    <xacro:if value="${is_right}">
+                        <!-- PRE_WHEEL_LEG-->
+                        <inertial>
+                    		<origin xyz="0 0 0" rpy="0 0 0"/>
+                    		<mass value="0.66"/>
+                    		<inertia ixx="0.00024" ixy="0" ixz="0" iyy="0.00016" iyz="0" izz="0.00024"/>
+                	</inertial>
+                    </xacro:if>
+                </xacro:unless>
         </link>
         <!--WHEEL JOINT-->
@@ -580,7 +629,5 @@
                     </xacro:if>
                 </xacro:unless>
-                <material name="upper_leg_color">
-                    <color rgba="0.3 0.3 0.6 1.0"/>
-                </material>
+                <material name="blue"/>
             </visual>
             <!--COLLISION-->
@@ -615,25 +662,42 @@
                     </xacro:if>
                 </xacro:unless>
-                <material name="collision_color">
-                    <color rgba="0.8 0.8 0.8 1.0"/>
-                </material>
             </collision>
             <!-- WHEEL LINK INERTIAL -->
-            <xacro:unless value="${is_right}">
-                <!-- Left pre_wheel inertia -->
-                <inertial>
-                    <origin xyz="0 0 0" rpy="0 0 0"/>
-                    <mass value="1.0"/>
-                    <inertia ixx="0.00224" ixy="0" ixz="0" iyy="0.00121" iyz="0" izz="0.00121"/>
-                </inertial>
-            </xacro:unless>
-            <xacro:if value="${is_right}">
-                <!-- Right pre_wheel inertia -->
-                <inertial>
-                    <origin xyz="0 0 0" rpy="0 0 0"/>
-                    <mass value="1.0"/>
-                    <inertia ixx="0.00121" ixy="0" ixz="0" iyy="0.00224" iyz="0" izz="0.00121"/>
-                </inertial>
-            </xacro:if>
+            <xacro:if value="${is_front}">
+                    <xacro:unless value="${is_right}">
+                        <!-- PRE_WHEEL_LEG -->
+                        <inertial>
+                    		<origin xyz="0 0 0" rpy="0 0 0"/>
+                    		<mass value="1.0"/>
+                    		<inertia ixx="0.00224" ixy="0" ixz="0" iyy="0.00121" iyz="0" izz="0.00224"/>
+                	</inertial>
+                    </xacro:unless>
+                    <xacro:if value="${is_right}">
+                        <!-- PRE_WHEEL_LEG -->
+                        <inertial>
+                    		<origin xyz="0 0 0" rpy="0 0 0"/>
+                    		<mass value="1.0"/>
+                    		<inertia ixx="0.00121" ixy="0" ixz="0" iyy="0.00224" iyz="0" izz="0.00121"/>
+                	</inertial>
+                    </xacro:if>
+                </xacro:if>
+                <xacro:unless value="${is_front}">
+                    <xacro:unless value="${is_right}">
+                        <!-- PRE_WHEEL_LEG -->
+                        <inertial>
+                    		<origin xyz="0 0 0" rpy="0 0 0"/>
+                    		<mass value="1.0"/>
+                    		<inertia ixx="0.00121" ixy="0" ixz="0" iyy="0.00224" iyz="0" izz="0.00121"/>
+                	</inertial>
+                    </xacro:unless>
+                    <xacro:if value="${is_right}">
+                        <!-- PRE_WHEEL_LEG-->
+                        <inertial>
+                    		<origin xyz="0 0 0" rpy="0 0 0"/>
+                    		<mass value="1.0"/>
+                    		<inertia ixx="0.00224" ixy="0" ixz="0" iyy="0.00121" iyz="0" izz="0.00224"/>
+                	</inertial>
+                    </xacro:if>
+                </xacro:unless>
         </link>
         <!-- Extensions -->
