Commit message: now rviz starts

File: robots/starbot.urdf.xacro (robot description, xacro)
@@ -31,18 +31,30 @@
     <!-- TODO Include the legs (add parameters if necessary)-->
     <!-- LEFT FRONT LEG -->
-    <xacro:leg
-    prefix="lf"
-    robot_name="$(arg robot_name)"/>
+     <xacro:leg
+    	name="lf"
+    	parent="base_link"
+    	robot_name="$(arg robot_name)">
+    	<origin xyz="0.1 0.1 0.0" rpy="0 0 0"/>
+    </xacro:leg>
     <!-- RIGHT FRONT LEG -->
     <xacro:leg
-    prefix="rf"
-    robot_name="$(arg robot_name)"/>
+    	name="rf"
+    	parent="base_link"
+    	robot_name="$(arg robot_name)">
+    	<origin xyz="0.1 -0.1 0.0" rpy="0 0 0"/>
+    </xacro:leg>
     <!-- LEFT HIND LEG -->
-    <xacro:leg
-    prefix="lh"
-    robot_name="$(arg robot_name)"/>
+     <xacro:leg
+    	name="lh"
+    	parent="base_link"
+    	robot_name="$(arg robot_name)">
+    	<origin xyz="-0.1 0.1 0.0" rpy="0 0 0"/>
+    </xacro:leg>
     <!-- RIGHT HIND LEG -->
     <xacro:leg
-    prefix="rh"
-    robot_name="$(arg robot_name)"/>
+    	name="rh"
+    	parent="base_link"
+    	robot_name="$(arg robot_name)">
+    	<origin xyz="-0.1 -0.1 0.0" rpy="0 0 0"/>
+    </xacro:leg>
 </robot>

File: urdfs/leg.gazebo.xacro (robot description, xacro)
@@ -14,5 +14,5 @@
                                 <update_rate>1000.0</update_rate>
                                 <contact>
-                                        <collision>${name}_lowerleg_fixed_joint_lump__${name}_foot_collision_1</collision>
+                                        <collision>${name}_XXXX</collision>
                                 </contact>
                                 <!-- the sensor readings in terms of force torques are expressed in the lowerleg frame

File: urdfs/leg.xacro (robot description, xacro)
@@ -5,16 +5,16 @@
     <xacro:include filename="$(find starbot_description)/urdfs/leg.gazebo.xacro"/>
     <!-- This macro has for purpose to define a leg -->
-    <xacro:macro name="leg" params="prefix robot_name">
+    <xacro:macro name="leg" params="name parent robot_name *origin ">
            <!-- TODO ADD JOINTS AND LINKS -->
 	  <!-- TODO ADD JOINTS AND LINKS -->
         <!-- FOOT -->
-        <link name="${prefix}_foot">
+        <!--link name="${name}_foot"-->
             <!-- FOOT INERTIAL -->
             <!-- FOOT VISUAL -->
             <!-- FOOT COLLISION -->
-	</link> <!-- END FOOT LINK -->
+	<!--/link-->
         <!-- Extensions -->
-        <xacro:leg_transmission name="${prefix}"/>
-        <xacro:leg_gazebo name="${prefix}" robot_name="${robot_name}"/>
+        <xacro:leg_transmission name="${name}"/>
+        <xacro:leg_gazebo name="${name}" robot_name="${robot_name}"/>
     </xacro:macro>
 </robot>

Commit message: adding missing elements

File: robots/starbot.urdf.xacro (robot description, xacro)
@@ -28,4 +28,21 @@
     <link name="trunk">
         <!-- TODO the trunk (it will be fixed to base link but it has inertia) -->
+		<inertial>
+		  <origin xyz="0.0 0.0 0.0"/>
+		  <mass value="15" />
+		  <inertia  ixx="0.001" ixy="0.0"  ixz="0.0"  iyy="0.001"  iyz="0.0"  izz="0.001" />
+	       </inertial>
+	      <visual>
+		<origin xyz="0 0.0 0.0" rpy="0 0 0"/>
+		<geometry>
+		    <box size="0.1 0.1 0.1"/>
+		</geometry>
+	      </visual>
+	     <collision>
+		<origin  xyz="0 0.0 0.0 " rpy="0 0 0"/>
+		<geometry>
+		    <box size="0.1 0.1 0.1"/>
+		</geometry>
+	     </collision>
     </link>
     <!-- TODO Include the legs (add parameters if necessary)-->

File: urdfs/leg.transmission.xacro (robot description, xacro)
@@ -2,33 +2,11 @@
 <robot xmlns:xacro="http://ros.org/wiki/xacro">
         <xacro:macro name="leg_transmission" params="name">
-        <!-- 1st link -->
-                <transmission name="${name}_XXXXXX_trans">
+        	<!-- 1st joint -->
+                <transmission name="${name}_shoulder_pan_trans">
                         <type>transmission_interface/SimpleTransmission</type>
-                        <joint name="${name}_haa_joint">
+                        <joint name="${name}_shoulder_pan">
                                 <hardwareInterface>hardware_interface/EffortJointInterface</hardwareInterface>
                         </joint>
-                        <actuator name="${name}_XXXXXX_motor">
-                                <hardwareInterface>hardware_interface/EffortJointInterface</hardwareInterface>
-                                <mechanicalReduction>1</mechanicalReduction>
-                        </actuator>
-                </transmission>
-         <!-- 2nd link -->
-                <transmission name="${name}_XXXXXX_trans">
-                        <type>transmission_interface/SimpleTransmission</type>
-                        <joint name="${name}_XXXXXX_joint">
-                                <hardwareInterface>hardware_interface/EffortJointInterface</hardwareInterface>
-                        </joint>
-                        <actuator name="${name}_XXXXXX_motor">
-                                <hardwareInterface>hardware_interface/EffortJointInterface</hardwareInterface>
-                                <mechanicalReduction>1</mechanicalReduction>
-                        </actuator>
-                </transmission>
-        <!-- 3rd link ETC..... -->
-                <transmission name="${name}_XXXXXX_trans">
-                        <type>transmission_interface/SimpleTransmission</type>
-                        <joint name="${name}_XXXXXX_joint">
-                                <hardwareInterface>hardware_interface/EffortJointInterface</hardwareInterface>
-                        </joint>
-                        <actuator name="${name}_XXXXXX_motor">
+                        <actuator name="${name}_shoulder_pan_motor">
                                 <hardwareInterface>hardware_interface/EffortJointInterface</hardwareInterface>
                                 <mechanicalReduction>1</mechanicalReduction>

File: urdfs/leg.xacro (robot description, xacro)
@@ -7,11 +7,30 @@
     <xacro:macro name="leg" params="name parent robot_name *origin ">
            <!-- TODO ADD JOINTS AND LINKS -->
-	  <!-- TODO ADD JOINTS AND LINKS -->
-        <!-- FOOT -->
-        <!--link name="${name}_foot"-->
-            <!-- FOOT INERTIAL -->
-            <!-- FOOT VISUAL -->
-            <!-- FOOT COLLISION -->
-	<!--/link-->
+	 <joint name="${name}_shoulder_pan" type="revolute">
+	    <parent link="${parent}"/>
+	    <child link="${name}_shoulder"/>
+	    <axis xyz="0 0 1"/>
+	    <xacro:insert_block name="origin"/>
+	    <limit effort="50" velocity="10.0" lower="-3.14" upper="3.14" />
+	  </joint>
+	  <link name="${name}_shoulder">
+	      <inertial>
+		  <origin xyz="0.0 0.0 0.0"/>
+		  <mass value="0.05" />
+		  <inertia  ixx="0.001" ixy="0.0"  ixz="0.0"  iyy="0.001"  iyz="0.0"  izz="0.001" />
+	       </inertial>
+	      <visual>
+		<origin xyz="0 0.0 0.0" rpy="0 0 0"/>
+		<geometry>
+		    <box size="0.1 0.1 0.2"/>
+		</geometry>
+	      </visual>
+	     <collision>
+		<origin  xyz="0 0.0 0.0 " rpy="0 0 0"/>
+		<geometry>
+		    <box size="0.1 0.1 0.2"/>
+		</geometry>
+	     </collision>
+	  </link>
         <!-- Extensions -->
         <xacro:leg_transmission name="${name}"/>

Commit message: body and shouder joint added

File: robots/starbot.urdf.xacro (robot description, xacro)
@@ -27,30 +27,33 @@
     </joint>
     <link name="trunk">
-        <!-- TODO the trunk (it will be fixed to base link but it has inertia) -->
-		<inertial>
-		  <origin xyz="0.0 0.0 0.0"/>
-		  <mass value="15" />
-		  <inertia  ixx="0.001" ixy="0.0"  ixz="0.0"  iyy="0.001"  iyz="0.0"  izz="0.001" />
-	       </inertial>
-	      <visual>
-		<origin xyz="0 0.0 0.0" rpy="0 0 0"/>
-		<geometry>
-		    <box size="0.1 0.1 0.1"/>
-		</geometry>
-	      </visual>
-	     <collision>
-		<origin  xyz="0 0.0 0.0 " rpy="0 0 0"/>
-		<geometry>
-		    <box size="0.1 0.1 0.1"/>
-		</geometry>
-	     </collision>
+        <inertial>
+        <origin xyz="0 0 0" rpy="0 0 0"/>
+        <mass value="20.0"/>
+        <inertia ixx="0.16574" ixy="0" ixz="0" iyy="0.16574" iyz="0" izz="0.24057"/>
+      </inertial>
+      <visual>
+        <origin xyz="0 0 0" rpy="0 0 0"/>
+        <geometry>
+           <mesh filename="package://starbot_description/meshes/stl/octagon.stl"/>
+        </geometry>
+        <material name="body_color">
+        	<color rgba="0.8 0.8 0.8 1.0"/>
+        </material>
+      </visual>
+      <collision>
+        <origin xyz="0 0 0" rpy="0 0 0"/>
+        <geometry>
+          <box size="0.27816 0.27816 0.2"/>
+        </geometry>
+      </collision>
     </link>
-    <!-- TODO Include the legs (add parameters if necessary)-->
     <!-- LEFT FRONT LEG -->
      <xacro:leg
     	name="lf"
     	parent="base_link"
+    	is_front="true"
+    	is_right="false"
     	robot_name="$(arg robot_name)">
-    	<origin xyz="0.1 0.1 0.0" rpy="0 0 0"/>
+    	<origin xyz="0.14142 0.00035 2e-05" rpy="0 0 0"/>
     </xacro:leg>
     <!-- RIGHT FRONT LEG -->
@@ -58,6 +61,8 @@
     	name="rf"
     	parent="base_link"
+    	is_front="true"
+    	is_right="true"
     	robot_name="$(arg robot_name)">
-    	<origin xyz="0.1 -0.1 0.0" rpy="0 0 0"/>
+    	<origin xyz="-0.00035 0.14142 2e-05" rpy="0 0 0"/>
     </xacro:leg>
     <!-- LEFT HIND LEG -->
@@ -65,6 +70,8 @@
     	name="lh"
     	parent="base_link"
+    	is_front="false"
+    	is_right="false"
     	robot_name="$(arg robot_name)">
-    	<origin xyz="-0.1 0.1 0.0" rpy="0 0 0"/>
+    	<origin xyz="-0.00035 -0.14142 2e-05" rpy="0 0 0"/>
     </xacro:leg>
     <!-- RIGHT HIND LEG -->
@@ -72,6 +79,8 @@
     	name="rh"
     	parent="base_link"
+    	is_front="false"
+    	is_right="true"
     	robot_name="$(arg robot_name)">
-    	<origin xyz="-0.1 -0.1 0.0" rpy="0 0 0"/>
+    	<origin xyz="-0.14142 0.00035 2e-05" rpy="0 0 0"/>
     </xacro:leg>
 </robot>

File: urdfs/leg.gazebo.xacro (robot description, xacro)
@@ -2,4 +2,7 @@
 <robot xmlns:xacro="http://ros.org/wiki/xacro">
         <xacro:macro name="leg_gazebo" params="name robot_name">
+        	 <gazebo reference="${name}_bs_joint">
+                        <provideFeedback>true</provideFeedback>
+                 </gazebo>
 		 <!-- HERE WE HAVE FOOT SENSOR AND FRICTION PROPERTIES -->
                  <gazebo reference="${name}_foot">

File: urdfs/leg.transmission.xacro (robot description, xacro)
@@ -2,11 +2,11 @@
 <robot xmlns:xacro="http://ros.org/wiki/xacro">
         <xacro:macro name="leg_transmission" params="name">
-        	<!-- 1st joint -->
-                <transmission name="${name}_shoulder_pan_trans">
+        <!-- body_shoulder joint -->
+                <transmission name="${name}_bs_joint_trans">
                         <type>transmission_interface/SimpleTransmission</type>
-                        <joint name="${name}_shoulder_pan">
+                        <joint name="${name}_bs_joint">
                                 <hardwareInterface>hardware_interface/EffortJointInterface</hardwareInterface>
                         </joint>
-                        <actuator name="${name}_shoulder_pan_motor">
+                        <actuator name="${name}_bs_joint_motor">
                                 <hardwareInterface>hardware_interface/EffortJointInterface</hardwareInterface>
                                 <mechanicalReduction>1</mechanicalReduction>

File: urdfs/leg.xacro (robot description, xacro)
@@ -4,33 +4,99 @@
     <xacro:include filename="$(find starbot_description)/urdfs/leg.transmission.xacro"/>
     <xacro:include filename="$(find starbot_description)/urdfs/leg.gazebo.xacro"/>
+    <!-- These are absoulte distance value, the sign are decided below -->
+    <xacro:property name="MAX_TORQUE" value="0" />
+    <xacro:property name="VELOCITY" value="0" />
     <!-- This macro has for purpose to define a leg -->
-    <xacro:macro name="leg" params="name parent robot_name *origin ">
-           <!-- TODO ADD JOINTS AND LINKS -->
-	 <joint name="${name}_shoulder_pan" type="revolute">
-	    <parent link="${parent}"/>
-	    <child link="${name}_shoulder"/>
-	    <axis xyz="0 0 1"/>
-	    <xacro:insert_block name="origin"/>
-	    <limit effort="50" velocity="10.0" lower="-3.14" upper="3.14" />
-	  </joint>
-	  <link name="${name}_shoulder">
-	      <inertial>
-		  <origin xyz="0.0 0.0 0.0"/>
-		  <mass value="0.05" />
-		  <inertia  ixx="0.001" ixy="0.0"  ixz="0.0"  iyy="0.001"  iyz="0.0"  izz="0.001" />
-	       </inertial>
-	      <visual>
-		<origin xyz="0 0.0 0.0" rpy="0 0 0"/>
-		<geometry>
-		    <box size="0.1 0.1 0.2"/>
-		</geometry>
-	      </visual>
-	     <collision>
-		<origin  xyz="0 0.0 0.0 " rpy="0 0 0"/>
-		<geometry>
-		    <box size="0.1 0.1 0.2"/>
-		</geometry>
-	     </collision>
-	  </link>
+    <xacro:macro name="leg" params="name parent is_front is_right robot_name *origin">
+          <!-- Starbot 1.0 -->
+	  <!--BS_JOINT: Joint between the body and the shoulder -->
+            <joint name="${name}_bs_joint" type="revolute">
+                <parent link="${parent}"/>
+                <child link="${name}_shoulder"/>
+                <xacro:insert_block name="origin"/>
+                <!-- joints rotates around the z-axis -->
+                <axis xyz="0 0 1"/>
+                <!-- limit of the joint -->
+                <limit effort="${MAX_TORQUE}" lower="-3.14" upper="3.14" velocity="${VELOCITY}"/>
+            </joint>
+	  <!-- SHOULDER ASSEMBLY -->
+            <link name="${name}_shoulder">
+            	<!-- create a dummy shoulder_assembly link to join the two joints -->
+            	<!--VISUAL-->
+	        <visual>
+                    <xacro:if value="${is_front}">
+                        <xacro:unless value="${is_right}">
+                            <!-- LF SHOULDER -->
+                        	<geometry>
+                        	    <mesh filename="package://starbot_description/meshes/stl/shoulder.stl"/>
+                        	</geometry>
+                        </xacro:unless>
+                        <xacro:if value="${is_right}">
+                            <!-- RF SHOULDER-->
+                        	<geometry>
+                        	    <mesh filename="package://starbot_description/meshes/stl/shoulder.001.stl"/>
+                        	</geometry>
+                        </xacro:if>
+                    </xacro:if>
+                    <xacro:unless value="${is_front}">
+                        <xacro:unless value="${is_right}">
+                            <!-- LH SHOULDER -->
+                        	<geometry>
+                        	    <mesh filename="package://starbot_description/meshes/stl/shoulder.002.stl"/>
+                        	</geometry>
+                        </xacro:unless>
+                        <xacro:if value="${is_right}">
+                            <!-- RH SHOULDER -->
+                        	<geometry>
+                        	    <mesh filename="package://starbot_description/meshes/stl/shoulder.003.stl"/>
+                        	</geometry>
+                        </xacro:if>
+                    </xacro:unless>
+	                <material name="shoulder_color">
+                    		<color rgba="0.8 0.8 0.8 1.0"/>
+                	</material>
+	            </visual>
+	            <!--COLLISION-->
+	            <collision>
+	            <origin xyz="0 0 0" rpy="0 0 0" />
+                    <xacro:if value="${is_front}">
+                        <xacro:unless value="${is_right}">
+                            <!-- LF_BS -->
+                        	<geometry>
+                        	    <box size="0.00651 0.0707 0.07002"/>
+                        	</geometry>
+                        </xacro:unless>
+                        <xacro:if value="${is_right}">
+                            <!-- RF_BS -->
+                        	<geometry>
+                        	    <box size="0.0707 0.00651 0.07002"/>
+                        	</geometry>
+                        </xacro:if>
+                    </xacro:if>
+                    <xacro:unless value="${is_front}">
+                        <xacro:unless value="${is_right}">
+                            <!-- LH_BS -->
+                        	<geometry>
+                        	    <box size="0.0707 0.00651 0.07002"/>
+                        	</geometry>
+                        </xacro:unless>
+                        <xacro:if value="${is_right}">
+                            <!-- RH_BS -->
+                        	<geometry>
+                        	    <box size="0.00651 0.0707 0.07002"/>
+                        	</geometry>
+                        </xacro:if>
+                    </xacro:unless>
+	                <material name="shoulder_collision_color">
+      				<color rgba="0.8 0.8 0.8 1.0"/>
+    			</material>
+	            </collision>
+	            <!--INERTIAL -->
+	            <inertial>
+	            	<origin xyz="0 0 0" rpy="0 0 0" />
+	                <mass value="0.01"/>
+	                <inertia ixx="0" ixy="0" ixz="0" iyy="0" iyz="0" izz="0"/>
+	            </inertial>
+	        </link>
         <!-- Extensions -->
         <xacro:leg_transmission name="${name}"/>
