Commit message: fix order of the legs

File: robots/starbot.urdf.xacro (robot description, xacro)
@@ -48,5 +48,23 @@
       </collision>
     </link>
-    <!-- LEFT FRONT LEG -->
+    <!-- if we imagine to place a line between the two positive direction of axis x and y -->
+    <!--
+      legs are align with axis x and y as shown below
+          is right?
+             |
+     y       |        x
+       o     |     o
+    	o    |    o
+    	 o___|___o
+    	 |   |   |
+  _______|___|___|_________ is front?
+         |   |   |
+    	 |___|___|
+    	 o   |   o
+    	o    |    o
+       o     |     o
+    -x       |       -y
+    -->
+    <!-- LEFT FRONT LEG = leg align with axis y -->
      <xacro:leg
     	name="lf"
@@ -55,7 +73,7 @@
     	is_right="false"
     	robot_name="$(arg robot_name)">
-    	<origin xyz="0.14142 0.00035 2e-05" rpy="0 0 0"/>
+    	<origin xyz="-0.00035 0.14142 2e-05" rpy="0 0 0"/>
     </xacro:leg>
-    <!-- RIGHT FRONT LEG -->
+    <!-- RIGHT FRONT LEG = leg align with axis x -->
     <xacro:leg
     	name="rf"
@@ -64,7 +82,7 @@
     	is_right="true"
     	robot_name="$(arg robot_name)">
-    	<origin xyz="-0.00035 0.14142 2e-05" rpy="0 0 0"/>
+    	<origin xyz="0.14142 0.00035 2e-05" rpy="0 0 0"/>
     </xacro:leg>
-    <!-- LEFT HIND LEG -->
+    <!-- LEFT HIND LEG = leg align with axis neg x -->
      <xacro:leg
     	name="lh"
@@ -73,7 +91,7 @@
     	is_right="false"
     	robot_name="$(arg robot_name)">
-    	<origin xyz="-0.00035 -0.14142 2e-05" rpy="0 0 0"/>
+    	<origin xyz="-0.14142 0.00035 2e-05" rpy="0 0 0"/>
     </xacro:leg>
-    <!-- RIGHT HIND LEG -->
+    <!-- RIGHT HIND LEG = leg align with axis neg y -->
     <xacro:leg
     	name="rh"
@@ -82,5 +100,5 @@
     	is_right="true"
     	robot_name="$(arg robot_name)">
-    	<origin xyz="-0.14142 0.00035 2e-05" rpy="0 0 0"/>
+    	<origin xyz="-0.00035 -0.14142 2e-05" rpy="0 0 0"/>
     </xacro:leg>
 </robot>

File: urdfs/leg.xacro (robot description, xacro)
@@ -33,5 +33,5 @@
                             <!-- LF SHOULDER -->
                         	<geometry>
-                        	    <mesh filename="package://starbot_description/meshes/stl/shoulder.stl"/>
+                        	    <mesh filename="package://starbot_description/meshes/stl/shoulder_y.stl"/>
                         	</geometry>
                         </xacro:unless>
@@ -39,5 +39,5 @@
                             <!-- RF SHOULDER-->
                         	<geometry>
-                        	    <mesh filename="package://starbot_description/meshes/stl/shoulder.001.stl"/>
+                        	    <mesh filename="package://starbot_description/meshes/stl/shoulder_x.stl"/>
                         	</geometry>
                         </xacro:if>
@@ -47,5 +47,5 @@
                             <!-- LH SHOULDER -->
                         	<geometry>
-                        	    <mesh filename="package://starbot_description/meshes/stl/shoulder.002.stl"/>
+                        	    <mesh filename="package://starbot_description/meshes/stl/shoulder_nx.stl"/>
                         	</geometry>
                         </xacro:unless>
@@ -53,5 +53,5 @@
                             <!-- RH SHOULDER -->
                         	<geometry>
-                        	    <mesh filename="package://starbot_description/meshes/stl/shoulder.003.stl"/>
+                        	    <mesh filename="package://starbot_description/meshes/stl/shoulder_ny.stl"/>
                         	</geometry>
                         </xacro:if>
@@ -68,25 +68,25 @@
                             <!-- LF_BS -->
                         	<geometry>
+                        	    <box size="0.0707 0.00651 0.07002"/>
+                        	</geometry>
+                        </xacro:unless>
+                        <xacro:if value="${is_right}">
+                            <!-- RF_BS -->
+                        	<geometry>
                         	    <box size="0.00651 0.0707 0.07002"/>
                         	</geometry>
-                        </xacro:unless>
-                        <xacro:if value="${is_right}">
-                            <!-- RF_BS -->
+                        </xacro:if>
+                    </xacro:if>
+                    <xacro:unless value="${is_front}">
+                        <xacro:unless value="${is_right}">
+                            <!-- LH_BS -->
+                        	<geometry>
+                        	    <box size="0.00651 0.0707 0.07002"/>
+                        	</geometry>
+                        </xacro:unless>
+                        <xacro:if value="${is_right}">
+                            <!-- RH_BS -->
                         	<geometry>
                         	    <box size="0.0707 0.00651 0.07002"/>
-                        	</geometry>
-                        </xacro:if>
-                    </xacro:if>
-                    <xacro:unless value="${is_front}">
-                        <xacro:unless value="${is_right}">
-                            <!-- LH_BS -->
-                        	<geometry>
-                        	    <box size="0.0707 0.00651 0.07002"/>
-                        	</geometry>
-                        </xacro:unless>
-                        <xacro:if value="${is_right}">
-                            <!-- RH_BS -->
-                        	<geometry>
-                        	    <box size="0.00651 0.0707 0.07002"/>
                         	</geometry>
                         </xacro:if>
@@ -99,5 +99,5 @@
 	            <inertial>
 	            	<origin xyz="0 0 0" rpy="0 0 0" />
-	                <mass value="0.01"/>
+	                <mass value="0.0001"/>
 	                <inertia ixx="0" ixy="0" ixz="0" iyy="0" iyz="0" izz="0"/>
 	            </inertial>
@@ -113,13 +113,13 @@
                     <xacro:unless value="${is_right}">
                         <!-- LF_UPPER_LEG_JOINT -->
-                        <axis xyz="0 1 0"/>
+                        <axis xyz="1 0 0"/>
                         <limit effort="${MAX_TORQUE}" lower="-3.14" upper="3.14" velocity="${VELOCITY}"/>
-                        <origin xyz="-${UPPER_LEG} 0 0" rpy="0 0 0" />
+                        <origin xyz="0 ${UPPER_LEG}  0" rpy="0 0 0" />
                     </xacro:unless>
                     <xacro:if value="${is_right}">
                         <!-- RF_UPPER_LEG_JOINT -->
-                        <axis xyz="-1 0 0"/>
-			<limit effort="${MAX_TORQUE}" lower="-3.14" upper="3.14" velocity="${VELOCITY}"/>
-                        <origin xyz="0 -${UPPER_LEG} 0" rpy="0 0 0" />
+                        <axis xyz="0 1 0"/>
+			<limit effort="${MAX_TORQUE}" lower="-3.14" upper="3.14" velocity="${VELOCITY}"/>
+                        <origin xyz="${UPPER_LEG} 0 0" rpy="0 0 0" />
                     </xacro:if>
                 </xacro:if>
@@ -127,13 +127,13 @@
                     <xacro:unless value="${is_right}">
                         <!-- LH_UPPER_LEG_JOINT -->
-                        <axis xyz="1 0 0"/>
-			<limit effort="${MAX_TORQUE}" lower="-3.14" upper="3.14" velocity="${VELOCITY}"/>
-                        <origin xyz="0 ${UPPER_LEG} 0" rpy="0 0 0" />
+                        <axis xyz="0 -1 0"/>
+			<limit effort="${MAX_TORQUE}" lower="-3.14" upper="3.14" velocity="${VELOCITY}"/>
+                        <origin xyz="-${UPPER_LEG} 0 0" rpy="0 0 0" />
                     </xacro:unless>
                     <xacro:if value="${is_right}">
-                        <!-- RF_UPPER_LEG_JOINT -->
-                        <axis xyz="0 -1 0"/>
-			<limit effort="${MAX_TORQUE}" lower="-3.14" upper="3.14" velocity="${VELOCITY}"/>
-                        <origin xyz="${UPPER_LEG} 0 0" rpy="0 0 0" />
+                        <!-- RH_UPPER_LEG_JOINT -->
+                        <axis xyz="-1 0 0"/>
+			<limit effort="${MAX_TORQUE}" lower="-3.14" upper="3.14" velocity="${VELOCITY}"/>
+                        <origin xyz="0 -${UPPER_LEG} 0" rpy="0 0 0" />
                     </xacro:if>
                 </xacro:unless>
@@ -150,5 +150,5 @@
                             <!-- LF UPPER_LEG -->
                         	<geometry>
-                        	    <mesh filename="package://starbot_description/meshes/stl/upper_leg.stl"/>
+                        	    <mesh filename="package://starbot_description/meshes/stl/upper_leg_y.stl"/>
                         	</geometry>
                         </xacro:unless>
@@ -156,5 +156,5 @@
                             <!-- RF UPPER_LEG-->
                         	<geometry>
-                        	    <mesh filename="package://starbot_description/meshes/stl/upper_leg.001.stl"/>
+                        	    <mesh filename="package://starbot_description/meshes/stl/upper_leg_x.stl"/>
                         	</geometry>
                         </xacro:if>
@@ -164,5 +164,5 @@
                             <!-- LH UPPER_LEG -->
                         	<geometry>
-                        	    <mesh filename="package://starbot_description/meshes/stl/upper_leg.002.stl"/>
+                        	    <mesh filename="package://starbot_description/meshes/stl/upper_leg_nx.stl"/>
                         	</geometry>
                         </xacro:unless>
@@ -170,5 +170,5 @@
                             <!-- RH UPPER_LEG -->
                         	<geometry>
-                        	    <mesh filename="package://starbot_description/meshes/stl/upper_leg.003.stl"/>
+                        	    <mesh filename="package://starbot_description/meshes/stl/upper_leg_ny.stl"/>
                         	</geometry>
                         </xacro:if>
@@ -185,25 +185,25 @@
                             <!-- LF UPPER_LEG -->
                         	<geometry>
+                        	    <box size="0.07002 0.30016 0.0707"/>
+                        	</geometry>
+                        </xacro:unless>
+                        <xacro:if value="${is_right}">
+                            <!-- RF UPPER_LEG -->
+                        	<geometry>
                         	    <box size="0.30016 0.07002 0.0707"/>
                         	</geometry>
-                        </xacro:unless>
-                        <xacro:if value="${is_right}">
-                            <!-- RF UPPER_LEG -->
+                        </xacro:if>
+                    </xacro:if>
+                    <xacro:unless value="${is_front}">
+                        <xacro:unless value="${is_right}">
+                            <!-- LH UPPER_LEG -->
+                        	<geometry>
+                        	    <box size="0.30016 0.07002 0.0707"/>
+                        	</geometry>
+                        </xacro:unless>
+                        <xacro:if value="${is_right}">
+                            <!-- RH UPPER_LEG-->
                         	<geometry>
                         	    <box size="0.07002 0.30016 0.0707"/>
-                        	</geometry>
-                        </xacro:if>
-                    </xacro:if>
-                    <xacro:unless value="${is_front}">
-                        <xacro:unless value="${is_right}">
-                            <!-- LH UPPER_LEG -->
-                        	<geometry>
-                        	    <box size="0.07002 0.30016 0.0707"/>
-                        	</geometry>
-                        </xacro:unless>
-                        <xacro:if value="${is_right}">
-                            <!-- RH UPPER_LEG-->
-                        	<geometry>
-                        	    <box size="0.30016 0.07002 0.0707"/>
                         	</geometry>
                         </xacro:if>
@@ -219,5 +219,5 @@
                      <origin xyz="0 0 0" rpy="0 0 0"/>
                     <mass value="2.3"/>
-                    <inertia ixx="0.00148" ixy="0" ixz="0" iyy="0.01286" iyz="0" izz="0.01286"/>
+                     <inertia ixx="0.01259" ixy="0" ixz="0" iyy="0.00147" iyz="0" izz="0.01259"/>
                 </inertial>
             	</xacro:unless>
@@ -227,5 +227,5 @@
                      <origin xyz="0 0 0" rpy="0 0 0"/>
                     <mass value="2.3"/>
-                    <inertia ixx="0.01259" ixy="0" ixz="0" iyy="0.00147" iyz="0" izz="0.01259"/>
+                    <inertia ixx="0.00147" ixy="0" ixz="0" iyy="0.01259" iyz="0" izz="0.01259"/>
                 </inertial>
             	</xacro:if>
@@ -236,32 +236,32 @@
                 <child link="${name}_lowerleg"/>
                 <xacro:insert_block name="origin"/>
-                <!-- joints rotates around the x-axis -->
+                <!-- joints rotates around the x-axis (refer to the x-axis align leg) -->
                 <!-- limit and placement of the joint -->
                 <xacro:if value="${is_front}">
                     <xacro:unless value="${is_right}">
                         <!-- LF_LOWER_LEG_JOINT -->
-                        <axis xyz="1 0 0"/>
+                        <axis xyz="0 1 0"/>
                         <limit effort="${MAX_TORQUE}" lower="-3.14" upper="3.14" velocity="${VELOCITY}"/>
+                        <origin xyz="${LOWER_LEG_y} ${LOWER_LEG_x} -${LOWER_LEG_z}" rpy="0 0 0" />
+                    </xacro:unless>
+                    <xacro:if value="${is_right}">
+                    	<axis xyz="1 0 0"/>
+                        <!-- RF_LOWER_LEG_JOINT -->
+			<limit effort="${MAX_TORQUE}" lower="-3.14" upper="3.14" velocity="${VELOCITY}"/>
                         <origin xyz="${LOWER_LEG_x} -${LOWER_LEG_y} -${LOWER_LEG_z}" rpy="0 0 0" />
-                    </xacro:unless>
-                    <xacro:if value="${is_right}">
-                    	<axis xyz="0 1 0"/>
-                        <!-- RF_LOWER_LEG_JOINT -->
-			<limit effort="${MAX_TORQUE}" lower="-3.14" upper="3.14" velocity="${VELOCITY}"/>
-                        <origin xyz="${LOWER_LEG_y} ${LOWER_LEG_x} -${LOWER_LEG_z}" rpy="0 0 0" />
                     </xacro:if>
                 </xacro:if>
                 <xacro:unless value="${is_front}">
                     <xacro:unless value="${is_right}">
-                    	<axis xyz="0 -1 0"/>
+                    	<axis xyz="-1 0 0"/>
                         <!-- LH_LOWER_LEG_JOINT -->
 			<limit effort="${MAX_TORQUE}" lower="-3.14" upper="3.14" velocity="${VELOCITY}"/>
-                        <origin xyz="${LOWER_LEG_y} -${LOWER_LEG_x} -${LOWER_LEG_z}" rpy="0 0 0" />
+                        <origin xyz="$-{LOWER_LEG_x} -${LOWER_LEG_y} -${LOWER_LEG_z}" rpy="0 0 0" />
                     </xacro:unless>
                     <xacro:if value="${is_right}">
                         <!-- RF_LOWER_LEG_JOINT -->
-                        <axis xyz="-1 0 0"/>
-			<limit effort="${MAX_TORQUE}" lower="-3.14" upper="3.14" velocity="${VELOCITY}"/>
-                        <origin xyz="-${LOWER_LEG_x} -${LOWER_LEG_y} -${LOWER_LEG_z}" rpy="0 0 0" />
+                        <axis xyz="0 -1 0"/>
+			<limit effort="${MAX_TORQUE}" lower="-3.14" upper="3.14" velocity="${VELOCITY}"/>
+                        <origin xyz="${LOWER_LEG_y} -${LOWER_LEG_x} -${LOWER_LEG_z}" rpy="0 0 0" />
                     </xacro:if>
                 </xacro:unless>
@@ -279,5 +279,5 @@
                             <!--we need mesh geometry otherwise strange behaviour happens-->
                         	<geometry>
-                        	    <mesh filename="package://starbot_description/meshes/stl/upper_leg.stl" scale="0.7 0.7 0.7"/>
+                        	    <mesh filename="package://starbot_description/meshes/stl/upper_leg_y.stl"/>
                         	</geometry>
                         </xacro:unless>
@@ -285,5 +285,5 @@
                             <!-- RF LOWER_LEG-->
                         	<geometry>
-                        	    <mesh filename="package://starbot_description/meshes/stl/upper_leg.001.stl" scale="0.7 0.7 0.7"/>
+                        	    <cylinder radius="0.02029" length="0.4002"/>
                         	</geometry>
                         </xacro:if>
@@ -293,5 +293,5 @@
                             <!-- LH LOWER_LEG -->
                         	<geometry>
-                        	    <mesh filename="package://starbot_description/meshes/stl/upper_leg.002.stl" scale="0.7 0.7 0.7"/>
+                        	    <cylinder radius="0.02029" length="0.4002"/>
                         	</geometry>
                         </xacro:unless>
@@ -299,5 +299,5 @@
                             <!-- RH LOWER_LEG -->
                         	<geometry>
-                        	    <mesh filename="package://starbot_description/meshes/stl/upper_leg.003.stl" scale="0.7 0.7 0.7"/>
+                        	    <cylinder radius="0.02029" length="0.4002"/>
                         	</geometry>
                         </xacro:if>
@@ -314,25 +314,25 @@
                             <!-- LF LOWER_LEG -->
                         	<geometry>
+                        	    <box size="0.04058 0.25009 0.04002"/>
+                        	</geometry>
+                        </xacro:unless>
+                        <xacro:if value="${is_right}">
+                            <!-- RF LOWER_LEG -->
+                        	<geometry>
                         	    <box size="0.25009 0.04058 0.04002"/>
                         	</geometry>
-                        </xacro:unless>
-                        <xacro:if value="${is_right}">
-                            <!-- RF LOWER_LEG -->
+                        </xacro:if>
+                    </xacro:if>
+                    <xacro:unless value="${is_front}">
+                        <xacro:unless value="${is_right}">
+                            <!-- LH LOWER_LEG -->
+                        	<geometry>
+                        	     <box size="0.25009 0.04058 0.04002"/>
+                        	</geometry>
+                        </xacro:unless>
+                        <xacro:if value="${is_right}">
+                            <!-- RH LOWER_LEG-->
                         	<geometry>
                         	    <box size="0.04058 0.25009 0.04002"/>
-                        	</geometry>
-                        </xacro:if>
-                    </xacro:if>
-                    <xacro:unless value="${is_front}">
-                        <xacro:unless value="${is_right}">
-                            <!-- LH LOWER_LEG -->
-                        	<geometry>
-                        	     <box size="0.04058 0.25009 0.04002"/>
-                        	</geometry>
-                        </xacro:unless>
-                        <xacro:if value="${is_right}">
-                            <!-- RH LOWER_LEG-->
-                        	<geometry>
-                        	    <box size="0.25009 0.04058 0.04002"/>
                         	</geometry>
                         </xacro:if>
@@ -344,17 +344,17 @@
 	            <!-- LOWER LEG LINK INERTIAL -->
             	<xacro:unless value="${is_right}">
-                <!-- Left upper leg inertia -->
+                <!-- Left lower leg inertia -->
                 <inertial>
                     <origin xyz="0 0 0" rpy="0 0 0"/>
         	    <mass value="2.36"/>
-        	    <inertia ixx="0.00954" ixy="0" ixz="0" iyy="0.00954" iyz="0" izz="0.01845"/>
+        	    <inertia ixx="0.00056" ixy="0" ixz="0" iyy="0.00056" iyz="0" izz="0.00049"/>
                 </inertial>
             	</xacro:unless>
             	<xacro:if value="${is_right}">
-            	<!-- Right upper leg inertia -->
+            	<!-- Right lower leg inertia -->
                 <inertial>
                      <origin xyz="0 0 0" rpy="0 0 0"/>
         	     <mass value="2.36"/>
-        	     <inertia ixx="0.00056" ixy="0" ixz="0" iyy="0.00056" iyz="0" izz="0.00049"/>
+        	     <inertia ixx="0.00954" ixy="0" ixz="0" iyy="0.00954" iyz="0" izz="0.01845"/>
                 </inertial>
             	</xacro:if>
