Commit message: fixed joints origin

File: robots/starbot.urdf.xacro (robot description, xacro)
@@ -73,5 +73,4 @@
     	is_right="false"
     	robot_name="$(arg robot_name)">
-    	<origin xyz="-0.00035 0.14142 2e-05" rpy="0 0 0"/>
     </xacro:leg>
     <!-- RIGHT FRONT LEG = leg align with axis x -->
@@ -82,5 +81,4 @@
     	is_right="true"
     	robot_name="$(arg robot_name)">
-    	<origin xyz="0.14142 0.00035 2e-05" rpy="0 0 0"/>
     </xacro:leg>
     <!-- LEFT HIND LEG = leg align with axis neg x -->
@@ -91,5 +89,4 @@
     	is_right="false"
     	robot_name="$(arg robot_name)">
-    	<origin xyz="-0.14142 0.00035 2e-05" rpy="0 0 0"/>
     </xacro:leg>
     <!-- RIGHT HIND LEG = leg align with axis neg y -->
@@ -100,5 +97,4 @@
     	is_right="true"
     	robot_name="$(arg robot_name)">
-    	<origin xyz="-0.00035 -0.14142 2e-05" rpy="0 0 0"/>
     </xacro:leg>
 </robot>

File: urdfs/leg.xacro (robot description, xacro)
@@ -6,13 +6,12 @@
     <!-- These are absoulte distance value, the sign are decided below -->
     <xacro:property name="MAX_TORQUE" value="0" />
+    <xacro:property name="SHOULDER" value="0.14142" />
     <xacro:property name="VELOCITY" value="0" />
     <xacro:property name="UPPER_LEG" value="0.15312" />
-    <xacro:property name="LOWER_LEG_x" value="0.22546" />
-    <xacro:property name="LOWER_LEG_y" value="0.00035" />
-    <xacro:property name="LOWER_LEG_z" value="2e-05" />
+    <xacro:property name="LOWER_LEG_pos" value="0.02546" />
     <xacro:property name="PRE_WHEEL_pos" value="0.16173" />
     <xacro:property name="WHEEL_pos" value="0.10183" />
     <!-- This macro has for purpose to define a leg -->
-    <xacro:macro name="leg" params="name parent is_front is_right robot_name *origin">
+    <xacro:macro name="leg" params="name parent is_front is_right robot_name">
         <!-- Starbot 1.0 -->
         <!--BS_JOINT: Joint between the body and the shoulder -->
@@ -20,9 +19,35 @@
             <parent link="${parent}"/>
             <child link="${name}_shoulder"/>
-            <xacro:insert_block name="origin"/>
-            <!-- joints rotates around the z-axis -->
-            <axis xyz="0 0 1"/>
-            <!-- limit of the joint -->
-            <limit effort="${MAX_TORQUE}" lower="-3.14" upper="3.14" velocity="${VELOCITY}"/>
+            <!-- limit and placement of the joint -->
+            <xacro:if value="${is_front}">
+                <xacro:unless value="${is_right}">
+                    <!-- LF_UPPER_LEG_JOINT -->
+                    <axis xyz="1 0 0"/>
+                    <limit effort="${MAX_TORQUE}" lower="-0.785" upper="0.785" velocity="${VELOCITY}"/>
+                    <origin xyz="0 ${SHOULDER}  0" rpy="0 0 0" />
+                </xacro:unless>
+                <xacro:if value="${is_right}">
+                    <!-- RF_UPPER_LEG_JOINT -->
+                    <axis xyz="0 1 0"/>
+                    <limit effort="${MAX_TORQUE}" lower="-0.785" upper="0.785" velocity="${VELOCITY}"/>
+                    <origin xyz="${SHOULDER} 0 0" rpy="0 0 0" />
+                </xacro:if>
+            </xacro:if>
+            <xacro:unless value="${is_front}">
+                <xacro:unless value="${is_right}">
+                    <!-- LH_UPPER_LEG_JOINT -->
+                    <axis xyz="0 -1 0"/>
+                    <limit effort="${MAX_TORQUE}" lower="-0.785" upper="0.785" velocity="${VELOCITY}"/>
+                    <origin xyz="-${SHOULDER} 0 0" rpy="0 0 0" />
+                </xacro:unless>
+                <xacro:if value="${is_right}">
+                    <!-- RH_UPPER_LEG_JOINT -->
+                    <axis xyz="-1 0 0"/>
+                    <limit effort="${MAX_TORQUE}" lower="-0.785" upper="0.785" velocity="${VELOCITY}"/>
+                    <origin xyz="0 -${SHOULDER} 0" rpy="0 0 0" />
+                </xacro:if>
+            </xacro:unless>
+            <!-- pybullet simulation parameters -->
+            <dynamics damping="0.0" friction="0.0"/>
         </joint>
         <!-- SHOULDER ASSEMBLY -->
@@ -109,5 +134,4 @@
             <parent link="${name}_shoulder"/>
             <child link="${name}_upperleg"/>
-            <xacro:insert_block name="origin"/>
             <!-- joints rotates around the y-axis -->
             <!-- limit and placement of the joint -->
@@ -116,5 +140,5 @@
                     <!-- LF_UPPER_LEG_JOINT -->
                     <axis xyz="1 0 0"/>
-                    <limit effort="${MAX_TORQUE}" lower="-3.14" upper="3.14" velocity="${VELOCITY}"/>
+                    <limit effort="${MAX_TORQUE}" lower="-0.785" upper="0.785" velocity="${VELOCITY}"/>
                     <origin xyz="0 ${UPPER_LEG}  0" rpy="0 0 0" />
                 </xacro:unless>
@@ -122,5 +146,5 @@
                     <!-- RF_UPPER_LEG_JOINT -->
                     <axis xyz="0 1 0"/>
-                    <limit effort="${MAX_TORQUE}" lower="-3.14" upper="3.14" velocity="${VELOCITY}"/>
+                    <limit effort="${MAX_TORQUE}" lower="-0.785" upper="0.785" velocity="${VELOCITY}"/>
                     <origin xyz="${UPPER_LEG} 0 0" rpy="0 0 0" />
                 </xacro:if>
@@ -130,5 +154,5 @@
                     <!-- LH_UPPER_LEG_JOINT -->
                     <axis xyz="0 -1 0"/>
-                    <limit effort="${MAX_TORQUE}" lower="-3.14" upper="3.14" velocity="${VELOCITY}"/>
+                    <limit effort="${MAX_TORQUE}" lower="-0.785" upper="0.785" velocity="${VELOCITY}"/>
                     <origin xyz="-${UPPER_LEG} 0 0" rpy="0 0 0" />
                 </xacro:unless>
@@ -136,5 +160,5 @@
                     <!-- RH_UPPER_LEG_JOINT -->
                     <axis xyz="-1 0 0"/>
-                    <limit effort="${MAX_TORQUE}" lower="-3.14" upper="3.14" velocity="${VELOCITY}"/>
+                    <limit effort="${MAX_TORQUE}" lower="-0.785" upper="0.785" velocity="${VELOCITY}"/>
                     <origin xyz="0 -${UPPER_LEG} 0" rpy="0 0 0" />
                 </xacro:if>
@@ -237,5 +261,4 @@
             <parent link="${name}_upperleg"/>
             <child link="${name}_lowerleg"/>
-            <xacro:insert_block name="origin"/>
             <!-- joints rotates around the x-axis (refer to the x-axis align leg) -->
             <!-- limit and placement of the joint -->
@@ -244,12 +267,12 @@
                     <!-- LF_LOWER_LEG_JOINT -->
                     <axis xyz="0 1 0"/>
-                    <limit effort="${MAX_TORQUE}" lower="0" upper="0" velocity="${VELOCITY}"/>
-                    <origin xyz="${LOWER_LEG_y} ${LOWER_LEG_x} -${LOWER_LEG_z}" rpy="0 0 0" />
+                    <limit effort="${MAX_TORQUE}" lower="0" upper="0.20" velocity="${VELOCITY}"/>
+                    <origin xyz="0 ${LOWER_LEG_pos} 0" rpy="0 0 0" />
                 </xacro:unless>
                 <xacro:if value="${is_right}">
                     <axis xyz="1 0 0"/>
                     <!-- RF_LOWER_LEG_JOINT -->
-                    <limit effort="${MAX_TORQUE}" lower="0" upper="0" velocity="${VELOCITY}"/>
-                    <origin xyz="${LOWER_LEG_x} -${LOWER_LEG_y} -${LOWER_LEG_z}" rpy="0 0 0" />
+                    <limit effort="${MAX_TORQUE}" lower="0" upper="0.20" velocity="${VELOCITY}"/>
+                    <origin xyz="${LOWER_LEG_pos} 0 0" rpy="0 0 0" />
                 </xacro:if>
             </xacro:if>
@@ -258,12 +281,12 @@
                     <axis xyz="-1 0 0"/>
                     <!-- LH_LOWER_LEG_JOINT -->
-                    <limit effort="${MAX_TORQUE}" lower="0" upper="0" velocity="${VELOCITY}"/>
-                    <origin xyz="$-{LOWER_LEG_x} -${LOWER_LEG_y} -${LOWER_LEG_z}" rpy="0 0 0" />
+                    <limit effort="${MAX_TORQUE}" lower="0" upper="0.20" velocity="${VELOCITY}"/>
+                    <origin xyz="-${LOWER_LEG_pos} 0 0" rpy="0 0 0" />
                 </xacro:unless>
                 <xacro:if value="${is_right}">
                     <!-- RF_LOWER_LEG_JOINT -->
                     <axis xyz="0 -1 0"/>
-                    <limit effort="${MAX_TORQUE}" lower="0" upper="0" velocity="${VELOCITY}"/>
-                    <origin xyz="${LOWER_LEG_y} -${LOWER_LEG_x} -${LOWER_LEG_z}" rpy="0 0 0" />
+                    <limit effort="${MAX_TORQUE}" lower="0" upper="0.20" velocity="${VELOCITY}"/>
+                    <origin xyz="0 -${LOWER_LEG_pos} 0" rpy="0 0 0" />
                 </xacro:if>
             </xacro:unless>
@@ -366,5 +389,4 @@
             <parent link="${name}_lowerleg"/>
             <child link="${name}_pre_wheel"/>
-            <xacro:insert_block name="origin"/>
             <!-- joints rotates around the x-axis (refer to the x-axis align leg) -->
             <!-- limit and placement of the joint -->
@@ -373,5 +395,5 @@
                     <!-- LF_PRE_WHEEL_JOINT -->
                     <axis xyz="1 0 0"/>
-                    <limit effort="${MAX_TORQUE}" lower="-3.14" upper="3.14" velocity="${VELOCITY}"/>
+                    <limit effort="${MAX_TORQUE}" lower="-1.57" upper="1.57" velocity="${VELOCITY}"/>
                     <origin xyz="0 ${PRE_WHEEL_pos} 0" rpy="0 0 0" />
                 </xacro:unless>
@@ -379,5 +401,5 @@
                     <axis xyz="0 1 0"/>
                     <!-- RF_PRE_WHEEL_JOINT -->
-                    <limit effort="${MAX_TORQUE}" lower="-3.14" upper="3.14" velocity="${VELOCITY}"/>
+                    <limit effort="${MAX_TORQUE}" lower="-1.57" upper="1.57" velocity="${VELOCITY}"/>
                     <origin xyz="${PRE_WHEEL_pos} 0 0" rpy="0 0 0" />
                 </xacro:if>
@@ -387,11 +409,11 @@
                     <axis xyz="0 -1 0"/>
                     <!-- LH_PRE_WHEEL_JOINT -->
-                    <limit effort="${MAX_TORQUE}" lower="-3.14" upper="3.14" velocity="${VELOCITY}"/>
-                    <origin xyz="$-{PRE_WHEEL_pos} 0 0" rpy="0 0 0" />
+                    <limit effort="${MAX_TORQUE}" lower="-1.57" upper="1.57" velocity="${VELOCITY}"/>
+                    <origin xyz="-${PRE_WHEEL_pos} 0 0" rpy="0 0 0" />
                 </xacro:unless>
                 <xacro:if value="${is_right}">
                     <!-- RF_PRE_WHEEL_JOINT -->
                     <axis xyz="-1 0 0"/>
-                    <limit effort="${MAX_TORQUE}" lower="-3.14" upper="3.14" velocity="${VELOCITY}"/>
+                    <limit effort="${MAX_TORQUE}" lower="-1.57" upper="1.57" velocity="${VELOCITY}"/>
                     <origin xyz="0 -${PRE_WHEEL_pos} 0" rpy="0 0 0" />
                 </xacro:if>
@@ -495,5 +517,4 @@
             <parent link="${name}_pre_wheel"/>
             <child link="${name}_wheel"/>
-            <xacro:insert_block name="origin"/>
             <!-- joints rotates around the x-axis (refer to the x-axis align leg) -->
             <!-- limit and placement of the joint -->
@@ -502,5 +523,4 @@
                     <!-- LF_WHEEL_JOINT -->
                     <axis xyz="1 0 0"/>
-                    <limit effort="${MAX_TORQUE}" lower="-3.14" upper="3.14" velocity="${VELOCITY}"/>
                     <origin xyz="0 ${WHEEL_pos} 0" rpy="0 0 0" />
                 </xacro:unless>
@@ -508,5 +528,4 @@
                     <axis xyz="0 1 0"/>
                     <!-- RF_WHEEL_JOINT -->
-                    <limit effort="${MAX_TORQUE}" lower="-3.14" upper="3.14" velocity="${VELOCITY}"/>
                     <origin xyz="${WHEEL_pos} 0 0" rpy="0 0 0" />
                 </xacro:if>
@@ -516,11 +535,9 @@
                     <axis xyz="0 -1 0"/>
                     <!-- LH_WHEEL_JOINT -->
-                    <limit effort="${MAX_TORQUE}" lower="-3.14" upper="3.14" velocity="${VELOCITY}"/>
-                    <origin xyz="$-{WHEEL_pos} 0 0" rpy="0 0 0" />
+                    <origin xyz="-${WHEEL_pos} 0 0" rpy="0 0 0" />
                 </xacro:unless>
                 <xacro:if value="${is_right}">
                     <!-- RF_WHEEL_JOINT -->
                     <axis xyz="-1 0 0"/>
-                    <limit effort="${MAX_TORQUE}" lower="-3.14" upper="3.14" velocity="${VELOCITY}"/>
                     <origin xyz="0 -${WHEEL_pos} 0" rpy="0 0 0" />
                 </xacro:if>

Commit message: continuous joints cannot be used with Pinocchio

File: robots/starbot.urdf.xacro (robot description, xacro)
@@ -29,5 +29,5 @@
         <inertial>
         <origin xyz="0 0 0" rpy="0 0 0"/>
-        <mass value="20.0"/>
+        <mass value="10.0"/>
         <inertia ixx="0.16574" ixy="0" ixz="0" iyy="0.16574" iyz="0" izz="0.24057"/>
       </inertial>
@@ -41,10 +41,4 @@
         </material>
       </visual>
-      <collision>
-        <origin xyz="0 0 0" rpy="0 0 0"/>
-        <geometry>
-          <box size="0.27816 0.27816 0.2"/>
-        </geometry>
-      </collision>
     </link>
     <!-- if we imagine to place a line between the two positive direction of axis x and y -->
@@ -69,5 +63,5 @@
      <xacro:leg
     	name="lf"
-    	parent="base_link"
+    	parent="trunk"
     	is_front="true"
     	is_right="false"
@@ -77,5 +71,5 @@
     <xacro:leg
     	name="rf"
-    	parent="base_link"
+    	parent="trunk"
     	is_front="true"
     	is_right="true"
@@ -85,5 +79,5 @@
      <xacro:leg
     	name="lh"
-    	parent="base_link"
+    	parent="trunk"
     	is_front="false"
     	is_right="false"
@@ -93,5 +87,5 @@
     <xacro:leg
     	name="rh"
-    	parent="base_link"
+    	parent="trunk"
     	is_front="false"
     	is_right="true"

File: urdfs/leg.xacro (robot description, xacro)
@@ -573,5 +573,5 @@
         </link>
         <!--WHEEL JOINT-->
-        <joint name="${name}_wheel_joint" type="continuous">
+        <joint name="${name}_wheel_joint" type="revolute">
             <parent link="${name}_pre_wheel"/>
             <child link="${name}_wheel"/>
@@ -602,4 +602,5 @@
                 </xacro:if>
             </xacro:unless>
+            <limit effort="100" lower="-1e10" upper="1e10" velocity="100"/>
             <!-- pybullet simulation parameters -->
             <dynamics damping="0.0" friction="0.0"/>
