Commit message: fixed wheel intersection

File: robots/starbot.urdf.xacro (robot description, xacro)
@@ -41,4 +41,10 @@
         </material>
       </visual>
+      <collision>
+            <origin xyz="0 0 0" rpy="0 0 0" />
+            <geometry>
+                <mesh filename="package://starbot_description/meshes/stl/octagon.stl"/>
+            </geometry>
+        </collision>
     </link>
     <!-- if we imagine to place a line between the two positive direction of axis x and y -->

File: urdfs/leg.xacro (robot description, xacro)
@@ -65,4 +65,5 @@
             <!--VISUAL-->
             <visual>
+            <origin xyz="0 0 0" rpy="0 0 0" />
                 <xacro:if value="${is_front}">
                     <xacro:unless value="${is_right}">
@@ -145,5 +146,5 @@
                     <axis xyz="0 0 1"/>
                     <limit effort="${MAX_TORQUE}" lower="-0.785" upper="0.785" velocity="${VELOCITY}"/>
-                    <origin xyz="0 0  0" rpy="0 0 0" />
+                    <origin xyz="0 ${UPPER_LEG} 0" rpy="0 0 0" />
                 </xacro:unless>
                 <xacro:if value="${is_right}">
@@ -151,5 +152,5 @@
                     <axis xyz="0 0 1"/>
                     <limit effort="${MAX_TORQUE}" lower="-0.785" upper="0.785" velocity="${VELOCITY}"/>
-                    <origin xyz="0 0 0" rpy="0 0 0" />
+                    <origin xyz="${UPPER_LEG} 0 0" rpy="0 0 0" />
                 </xacro:if>
             </xacro:if>
@@ -159,5 +160,5 @@
                     <axis xyz="0 0 1"/>
                     <limit effort="${MAX_TORQUE}" lower="-0.785" upper="0.785" velocity="${VELOCITY}"/>
-                    <origin xyz="0 0 0" rpy="0 0 0" />
+                    <origin xyz="-${UPPER_LEG} 0 0" rpy="0 0 0" />
                 </xacro:unless>
                 <xacro:if value="${is_right}">
@@ -165,5 +166,5 @@
                     <axis xyz="0 0 1"/>
                     <limit effort="${MAX_TORQUE}" lower="-0.785" upper="0.785" velocity="${VELOCITY}"/>
-                    <origin xyz="0 0 0" rpy="0 0 0" />
+                    <origin xyz="0 -${UPPER_LEG} 0" rpy="0 0 0" />
                 </xacro:if>
             </xacro:unless>
@@ -175,8 +176,8 @@
             <!--VISUAL-->
             <visual>
+                <origin xyz="0 0 0" rpy="0 0 0" />
                 <xacro:if value="${is_front}">
                     <xacro:unless value="${is_right}">
 			<!-- LF UPPER_LEG -->
-                      		<origin xyz="0 ${UPPER_LEG} 0" rpy="0 0 0" />
                         <geometry>
                             <mesh filename="package://starbot_description/meshes/stl/upper_leg_y.stl"/>
@@ -185,5 +186,4 @@
                     <xacro:if value="${is_right}">
 			<!-- RF UPPER_LEG-->
-                        <origin xyz="${UPPER_LEG} 0 0" rpy="0 0 0" />
                         <geometry>
                             <mesh filename="package://starbot_description/meshes/stl/upper_leg_x.stl"/>
@@ -194,5 +194,4 @@
                     <xacro:unless value="${is_right}">
 			<!-- LH UPPER_LEG -->
-			<origin xyz="-${UPPER_LEG} 0  0" rpy="0 0 0" />
                         <geometry>
                             <mesh filename="package://starbot_description/meshes/stl/upper_leg_nx.stl"/>
@@ -201,5 +200,4 @@
                     <xacro:if value="${is_right}">
 		        <!-- RH UPPER_LEG -->
-					<origin xyz=" 0 -${UPPER_LEG} 0" rpy="0 0 0" />
                         <geometry>
                             <mesh filename="package://starbot_description/meshes/stl/upper_leg_ny.stl"/>
@@ -214,5 +212,5 @@
                     <xacro:unless value="${is_right}">
                         <!-- LF UPPER_LEG -->
-			<origin xyz="0 ${UPPER_LEG}  0" rpy="0 0 0" />
+			<origin xyz="0 0 0" rpy="0 0 0" />
                         <geometry>
                             <mesh filename="package://starbot_description/meshes/stl/upper_leg_y.stl"/>
@@ -221,5 +219,5 @@
                     <xacro:if value="${is_right}">
                         <!-- RF UPPER_LEG -->
-       			<origin xyz="${UPPER_LEG} 0 0" rpy="0 0 0" />
+       			<origin xyz="0 0 0" rpy="0 0 0" />
                         <geometry>
                             <mesh filename="package://starbot_description/meshes/stl/upper_leg_x.stl"/>
@@ -230,5 +228,5 @@
                     <xacro:unless value="${is_right}">
                         <!-- LH UPPER_LEG -->
-			<origin xyz="-${UPPER_LEG} 0  0" rpy="0 0 0" />
+			<origin xyz="0 0  0" rpy="0 0 0" />
                         <geometry>
                             <mesh filename="package://starbot_description/meshes/stl/upper_leg_nx.stl"/>
@@ -237,5 +235,5 @@
                     <xacro:if value="${is_right}">
                         <!-- RH UPPER_LEG-->
-			<origin xyz=" 0 -${UPPER_LEG} 0" rpy="0 0 0" />
+			<origin xyz=" 0 0 0" rpy="0 0 0" />
                         <geometry>
                             <mesh filename="package://starbot_description/meshes/stl/upper_leg_ny.stl"/>
@@ -249,5 +247,5 @@
                         <!-- LF UPPER_LEG -->
                         <inertial>
-                    		<origin xyz="0 0 0" rpy="0 0 0"/>
+                    		<origin xyz="0 ${UPPER_LEG} 0" rpy="0 0 0"/>
                     		<mass value="2.3"/>
                     		<inertia ixx="0.01246" ixy="0" ixz="0" iyy="0.00148" iyz="0" izz="0.01246"/>
@@ -257,5 +255,5 @@
                         <!-- RF UPPER_LEG -->
                         <inertial>
-                    		<origin xyz="0 0 0" rpy="0 0 0"/>
+                    		<origin xyz="${UPPER_LEG} 0 0" rpy="0 0 0"/>
                     		<mass value="2.3"/>
                     		<inertia ixx="0.00148" ixy="0" ixz="0" iyy="0.01246" iyz="0" izz="0.00148"/>
@@ -267,5 +265,5 @@
                         <!-- LH UPPER_LEG -->
                         <inertial>
-                    		<origin xyz="0 0 0" rpy="0 0 0"/>
+                    		<origin xyz="-${UPPER_LEG} 0 0" rpy="0 0 0"/>
                     		<mass value="2.3"/>
                     		<inertia ixx="0.00148" ixy="0" ixz="0" iyy="0.01246" iyz="0" izz="0.00148"/>
@@ -275,5 +273,5 @@
                         <!-- RH UPPER_LEG-->
                         <inertial>
-                    		<origin xyz="0 0 0" rpy="0 0 0"/>
+                    		<origin xyz="0 -${UPPER_LEG} 0" rpy="0 0 0"/>
                     		<mass value="2.3"/>
                     		<inertia ixx="0.01246" ixy="0" ixz="0" iyy="0.00148" iyz="0" izz="0.01246"/>
@@ -286,12 +284,10 @@
             <parent link="${name}_upperleg"/>
             <child link="${name}_lowerleg"/>
-            <!-- joints rotates around the x-axis (refer to the x-axis align leg) -->
             <!-- limit and placement of the joint -->
             <xacro:if value="${is_front}">
                 <xacro:unless value="${is_right}">
                     <!-- LF_LOWER_LEG_JOINT -->
-			<origin xyz="0 ${UPPER_LEG} 0" rpy="0 0 0" />
                     <axis xyz="0 1 0"/>
-                    <limit effort="${MAX_TORQUE}" lower="0" upper="0.20" velocity="${VELOCITY}"/>
+                    <limit effort="${MAX_TORQUE}" lower="0.02" upper="0.20" velocity="${VELOCITY}"/>
                     <origin xyz="0 ${LOWER_LEG_pos} 0" rpy="0 0 0" />
                 </xacro:unless>
@@ -299,6 +295,5 @@
                     <axis xyz="1 0 0"/>
                     <!-- RF_LOWER_LEG_JOINT -->
-		<origin xyz="${UPPER_LEG} 0 0" rpy="0 0 0" />
-                    <limit effort="${MAX_TORQUE}" lower="0" upper="0.20" velocity="${VELOCITY}"/>
+                    <limit effort="${MAX_TORQUE}" lower="0.02" upper="0.20" velocity="${VELOCITY}"/>
                     <origin xyz="${LOWER_LEG_pos} 0 0" rpy="0 0 0" />
                 </xacro:if>
@@ -308,13 +303,11 @@
                     <axis xyz="-1 0 0"/>
                     <!-- LH_LOWER_LEG_JOINT -->
-		<origin xyz="-${UPPER_LEG} 0  0" rpy="0 0 0" />
-                    <limit effort="${MAX_TORQUE}" lower="0" upper="0.20" velocity="${VELOCITY}"/>
+                    <limit effort="${MAX_TORQUE}" lower="0.02" upper="0.20" velocity="${VELOCITY}"/>
                     <origin xyz="-${LOWER_LEG_pos} 0 0" rpy="0 0 0" />
                 </xacro:unless>
                 <xacro:if value="${is_right}">
                     <!-- RF_LOWER_LEG_JOINT -->
-			<origin xyz=" 0 -${UPPER_LEG} 0" rpy="0 0 0" />
                     <axis xyz="0 -1 0"/>
-                    <limit effort="${MAX_TORQUE}" lower="0" upper="0.20" velocity="${VELOCITY}"/>
+                    <limit effort="${MAX_TORQUE}" lower="0.02" upper="0.20" velocity="${VELOCITY}"/>
                     <origin xyz="0 -${LOWER_LEG_pos} 0" rpy="0 0 0" />
                 </xacro:if>
@@ -327,9 +320,8 @@
             <!--VISUAL-->
             <visual>
+		<origin xyz="0 0 0" rpy="0 0 0" />
                 <xacro:if value="${is_front}">
                     <xacro:unless value="${is_right}">
                         <!-- LF LOWER_LEG -->
-			<origin xyz="0 ${UPPER_LEG}  0" rpy="0 0 0" />
-           <!--we need mesh geometry otherwise strange behaviour happens-->
                         <geometry>
                             <mesh filename="package://starbot_description/meshes/stl/lower_leg_y.stl"/>
@@ -396,5 +388,5 @@
                         <!-- LF LOWER_LEG -->
                         <inertial>
-                    		<origin xyz="0 0 0" rpy="0 0 0"/>
+                    		<origin xyz="0 ${LOWER_LEG_pos} 0" rpy="0 0 0"/>
                     		<mass value="2.36"/>
                     		<inertia ixx="0.00767" ixy="0" ixz="0" iyy="0.00056" iyz="0" izz="0.00767"/>
@@ -404,5 +396,5 @@
                         <!-- RF LOWER_LEG -->
                         <inertial>
-                    		<origin xyz="0 0 0" rpy="0 0 0"/>
+                    		<origin xyz="${LOWER_LEG_pos} 0 0" rpy="0 0 0"/>
                     		<mass value="2.36"/>
                     		<inertia ixx="0.00056" ixy="0" ixz="0" iyy="0.00767" iyz="0" izz="0.00056"/>
@@ -414,5 +406,5 @@
                         <!-- LH LOWER_LEG -->
                         <inertial>
-                    		<origin xyz="0 0 0" rpy="0 0 0"/>
+                    		<origin xyz="-${LOWER_LEG_pos} 0 0" rpy="0 0 0"/>
                     		<mass value="2.36"/>
                     		<inertia ixx="0.00056" ixy="0" ixz="0" iyy="0.00767" iyz="0" izz="0.00056"/>
@@ -422,5 +414,5 @@
                         <!-- RH LOWER_LEG-->
                         <inertial>
-                    		<origin xyz="0 0 0" rpy="0 0 0"/>
+                    		<origin xyz="0 -${LOWER_LEG_pos} 0" rpy="0 0 0"/>
                     		<mass value="2.36"/>
                     		<inertia ixx="0.00767" ixy="0" ixz="0" iyy="0.00056" iyz="0" izz="0.00767"/>
@@ -539,5 +531,5 @@
                         <!-- PRE_WHEEL_LEG -->
                         <inertial>
-                    		<origin xyz="0 0 0" rpy="0 0 0"/>
+                    		<origin xyz="0 ${PRE_WHEEL_pos} 0" rpy="0 0 0"/>
                     		<mass value="0.66"/>
                     		<inertia ixx="0.00024" ixy="0" ixz="0" iyy="0.00016" iyz="0" izz="0.00024"/>
@@ -547,5 +539,5 @@
                         <!-- PRE_WHEEL_LEG -->
                         <inertial>
-                    		<origin xyz="0 0 0" rpy="0 0 0"/>
+                    		<origin xyz="${PRE_WHEEL_pos} 0 0" rpy="0 0 0"/>
                     		<mass value="0.66"/>
                     		<inertia ixx="0.00016" ixy="0" ixz="0" iyy="0.00024" iyz="0" izz="0.00016"/>
@@ -557,5 +549,5 @@
                         <!-- PRE_WHEEL_LEG -->
                         <inertial>
-                    		<origin xyz="0 0 0" rpy="0 0 0"/>
+                    		<origin xyz="-${PRE_WHEEL_pos} 0 0" rpy="0 0 0"/>
                     		<mass value="0.66"/>
                     		<inertia ixx="0.00016" ixy="0" ixz="0" iyy="0.00024" iyz="0" izz="0.00016"/>
@@ -565,5 +557,5 @@
                         <!-- PRE_WHEEL_LEG-->
                         <inertial>
-                    		<origin xyz="0 0 0" rpy="0 0 0"/>
+                    		<origin xyz="0 -${PRE_WHEEL_pos} 0" rpy="0 0 0"/>
                     		<mass value="0.66"/>
                     		<inertia ixx="0.00024" ixy="0" ixz="0" iyy="0.00016" iyz="0" izz="0.00024"/>
@@ -679,5 +671,5 @@
                         <!-- PRE_WHEEL_LEG -->
                         <inertial>
-                    		<origin xyz="0 0 0" rpy="0 0 0"/>
+                    		<origin xyz="0 ${WHEEL_pos} 0" rpy="0 0 0"/>
                     		<mass value="1.0"/>
                     		<inertia ixx="0.00224" ixy="0" ixz="0" iyy="0.00121" iyz="0" izz="0.00224"/>
@@ -687,5 +679,5 @@
                         <!-- PRE_WHEEL_LEG -->
                         <inertial>
-                    		<origin xyz="0 0 0" rpy="0 0 0"/>
+                    		<origin xyz="${WHEEL_pos} 0 0" rpy="0 0 0"/>
                     		<mass value="1.0"/>
                     		<inertia ixx="0.00121" ixy="0" ixz="0" iyy="0.00224" iyz="0" izz="0.00121"/>
@@ -697,5 +689,5 @@
                         <!-- PRE_WHEEL_LEG -->
                         <inertial>
-                    		<origin xyz="0 0 0" rpy="0 0 0"/>
+                    		<origin xyz="-${WHEEL_pos}  0 0" rpy="0 0 0"/>
                     		<mass value="1.0"/>
                     		<inertia ixx="0.00121" ixy="0" ixz="0" iyy="0.00224" iyz="0" izz="0.00121"/>
@@ -705,5 +697,5 @@
                         <!-- PRE_WHEEL_LEG-->
                         <inertial>
-                    		<origin xyz="0 0 0" rpy="0 0 0"/>
+                    		<origin xyz="0 -${WHEEL_pos} 0" rpy="0 0 0"/>
                     		<mass value="1.0"/>
                     		<inertia ixx="0.00224" ixy="0" ixz="0" iyy="0.00121" iyz="0" izz="0.00224"/>
