Commit message: fixed inertia matrices and scaled collisions meshes

File: robots/starbot.urdf.xacro (robot description, xacro)
@@ -29,6 +29,6 @@
         <inertial>
         <origin xyz="0 0 0" rpy="0 0 0"/>
-        <mass value="10.0"/>
-        <inertia ixx="0.16574" ixy="0" ixz="0" iyy="0.16574" iyz="0" izz="0.24057"/>
+        <mass value="20.0"/>
+        <inertia ixx="0.1956" ixy="0" ixz="0" iyy="0.1956" iyz="0" izz="0.2579"/>
       </inertial>
       <visual>

File: urdfs/common.xacro (robot description, xacro)
@@ -7,12 +7,12 @@
     <xacro:property name="UPPER_LIMIT_PRI" value="0.2" />
     <!-- center of mass of each part besides shoulder (for inertia) -->
-    <xacro:property name="CM_XY_UPPER" value="0.076" />
-    <xacro:property name="CM_Z_UPPER" value="0.0" />
-    <xacro:property name="CM_XY_LOWER" value="0.113" />
-    <xacro:property name="CM_Z_LOWER" value="0.0" />
-    <xacro:property name="CM_XY_PRE_WHEEL" value="0.081" />
-    <xacro:property name="CM_Z_PRE_WHEEL" value="0.0" />
-    <xacro:property name="CM_XY_WHEEL" value="0.051" />
-    <xacro:property name="CM_Z_WHEEL" value="0.0" />
+    <xacro:property name="CM_XY_UPPER" value="${UPPER_LEG_pos/2}" />
+    <xacro:property name="CM_Z_UPPER" value="0" />
+    <xacro:property name="CM_XY_LOWER" value="${LOWER_LEG_pos + LOWER_LEG_joint_pos}" />
+    <xacro:property name="CM_Z_LOWER" value="0" />
+    <xacro:property name="CM_XY_PRE_WHEEL" value="0" />
+    <xacro:property name="CM_Z_PRE_WHEEL" value="0" />
+    <xacro:property name="CM_XY_WHEEL" value="0" />
+    <xacro:property name="CM_Z_WHEEL" value="0" />
     <!-- These are absolute distance value, the sign are decided in leg.xacro -->
     <xacro:property name="SHOULDER_pos" value="0.14142" />
@@ -28,11 +28,11 @@
     <!-- material colors -->
      <material name="orange">
-     <color rgba="0.800 0.331 0.183 1.0"/>
+     <color rgba="0.800 0.331 0.183 0.4"/>
     </material>
     <material name="blue">
-     <color rgba="0.051 0.144 0.800 1.0"/>
+     <color rgba="0.051 0.144 0.800 0.4"/>
     </material>
     <material name="gray">
-     <color rgba="0.638 0.779 0.819 1.0"/>
+     <color rgba="0.638 0.779 0.819 0.4"/>
     </material>
 </robot>

File: urdfs/leg.xacro (robot description, xacro)
@@ -87,5 +87,5 @@
                         <!-- LF_BS -->
                         <geometry>
-                            <mesh filename="package://starbot_description/meshes/stl/shoulder_y.stl"/>
+                            <mesh filename="package://starbot_description/meshes/stl/shoulder_y.stl" scale = "0.8 0.8 0.8" />
                         </geometry>
                     </xacro:unless>
@@ -93,5 +93,5 @@
                         <!-- RF_BS -->
                         <geometry>
-                            <mesh filename="package://starbot_description/meshes/stl/shoulder_x.stl"/>
+                            <mesh filename="package://starbot_description/meshes/stl/shoulder_x.stl" scale = "0.8 0.8 0.8" />
                         </geometry>
                     </xacro:if>
@@ -101,5 +101,5 @@
                         <!-- LH_BS -->
                         <geometry>
-                            <mesh filename="package://starbot_description/meshes/stl/shoulder_nx.stl"/>
+                            <mesh filename="package://starbot_description/meshes/stl/shoulder_nx.stl" scale = "0.8 0.8 0.8" />
                         </geometry>
                     </xacro:unless>
@@ -107,5 +107,5 @@
                         <!-- RH_BS -->
                         <geometry>
-                            <mesh filename="package://starbot_description/meshes/stl/shoulder_ny.stl"/>
+                            <mesh filename="package://starbot_description/meshes/stl/shoulder_ny.stl" scale = "0.8 0.8 0.8" />
                         </geometry>
                     </xacro:if>
@@ -199,14 +199,14 @@
                     <xacro:unless value="${is_right}">
                         <!-- LF UPPER_LEG -->
-			<origin xyz="0 ${UPPER_LEG_pos} 0" rpy="0 0 0" />
-                        <geometry>
-                            <mesh filename="package://starbot_description/meshes/stl/upper_leg_y.stl"/>
+			<origin xyz="0 ${CM_XY_UPPER} ${CM_Z_UPPER}" rpy="0 0 0" />
+                        <geometry>
+                            <mesh filename="package://starbot_description/meshes/stl/upper_leg_y.stl" scale = "0.8 0.8 0.8" />
                         </geometry>
                     </xacro:unless>
                     <xacro:if value="${is_right}">
                         <!-- RF UPPER_LEG -->
-       			<origin xyz="${UPPER_LEG_pos} 0 0" rpy="0 0 0" />
-                        <geometry>
-                            <mesh filename="package://starbot_description/meshes/stl/upper_leg_x.stl"/>
+       			<origin xyz="${CM_XY_UPPER} 0 ${CM_Z_UPPER}" rpy="0 0 0" />
+                        <geometry>
+                            <mesh filename="package://starbot_description/meshes/stl/upper_leg_x.stl" scale = "0.8 0.8 0.8" />
                         </geometry>
                     </xacro:if>
@@ -215,14 +215,14 @@
                     <xacro:unless value="${is_right}">
                         <!-- LH UPPER_LEG -->
-			<origin xyz="-${UPPER_LEG_pos} 0 0" rpy="0 0 0" />
-                        <geometry>
-                            <mesh filename="package://starbot_description/meshes/stl/upper_leg_nx.stl"/>
+			<origin xyz="-${CM_XY_UPPER} 0 ${CM_Z_UPPER}" rpy="0 0 0" />
+                        <geometry>
+                            <mesh filename="package://starbot_description/meshes/stl/upper_leg_nx.stl" scale = "0.8 0.8 0.8" />
                         </geometry>
                     </xacro:unless>
                     <xacro:if value="${is_right}">
                         <!-- RH UPPER_LEG-->
-			<origin xyz="0 -${UPPER_LEG_pos} 0" rpy="0 0 0" />
-                        <geometry>
-                            <mesh filename="package://starbot_description/meshes/stl/upper_leg_ny.stl"/>
+			<origin xyz="0 -${CM_XY_UPPER} ${CM_Z_UPPER}" rpy="0 0 0" />
+                        <geometry>
+                            <mesh filename="package://starbot_description/meshes/stl/upper_leg_ny.stl" scale = "0.8 0.8 0.8" />
                         </geometry>
                     </xacro:if>
@@ -234,7 +234,7 @@
                         <!-- LF UPPER_LEG -->
                         <inertial>
-                    		<origin xyz="0 ${UPPER_LEG_pos} 0" rpy="0 0 0"/>
+                    		<origin xyz="0 ${UPPER_LEG_pos} 0" rpy="0 0 1.57"/>
                     		<mass value="2.3"/>
-                    		<inertia ixx="0.01246" ixy="0" ixz="0" iyy="0.00148" iyz="0" izz="0.01246"/>
+                    		<inertia ixx="0.001878" ixy="0" ixz="0" iyy="0.0182" iyz="0" izz="0.0182"/>
                 	</inertial>
                     </xacro:unless>
@@ -244,5 +244,5 @@
                     		<origin xyz="${UPPER_LEG_pos} 0 0" rpy="0 0 0"/>
                     		<mass value="2.3"/>
-                    		<inertia ixx="0.00148" ixy="0" ixz="0" iyy="0.01246" iyz="0" izz="0.00148"/>
+                    		<inertia ixx="0.001878" ixy="0" ixz="0" iyy="0.0182" iyz="0" izz="0.0182"/>
                 	</inertial>
                     </xacro:if>
@@ -254,5 +254,5 @@
                     		<origin xyz="-${UPPER_LEG_pos} 0 0" rpy="0 0 0"/>
                     		<mass value="2.3"/>
-                    		<inertia ixx="0.00148" ixy="0" ixz="0" iyy="0.01246" iyz="0" izz="0.00148"/>
+                    		<inertia ixx="0.001878" ixy="0" ixz="0" iyy="0.0182" iyz="0" izz="0.0182"/>
                 	</inertial>
                     </xacro:unless>
@@ -260,7 +260,7 @@
                         <!-- RH UPPER_LEG-->
                         <inertial>
-                    		<origin xyz="0 -${UPPER_LEG_pos} 0" rpy="0 0 0"/>
+                    		<origin xyz="0 -${UPPER_LEG_pos} 0" rpy="0 0 1.57"/>
                     		<mass value="2.3"/>
-                    		<inertia ixx="0.01246" ixy="0" ixz="0" iyy="0.00148" iyz="0" izz="0.01246"/>
+                    		<inertia ixx="0.001878" ixy="0" ixz="0" iyy="0.0182" iyz="0" izz="0.0182"/>
                 	</inertial>
                     </xacro:if>
@@ -348,5 +348,5 @@
                          <origin xyz="0 ${LOWER_LEG_pos} 0" rpy="0 0 0" />
                         <geometry>
-                            <mesh filename="package://starbot_description/meshes/stl/lower_leg_y.stl"/>
+                            <mesh filename="package://starbot_description/meshes/stl/lower_leg_y.stl" scale = "0.8 0.8 0.8"/>
                         </geometry>
                     </xacro:unless>
@@ -355,5 +355,5 @@
                         <origin xyz="${LOWER_LEG_pos} 0 0" rpy="0 0 0" />
                         <geometry>
-                            <mesh filename="package://starbot_description/meshes/stl/lower_leg_x.stl"/>
+                            <mesh filename="package://starbot_description/meshes/stl/lower_leg_x.stl" scale = "0.8 0.8 0.8" />
                         </geometry>
                     </xacro:if>
@@ -364,5 +364,5 @@
                         <origin xyz="-${LOWER_LEG_pos} 0 0" rpy="0 0 0" />
                         <geometry>
-                            <mesh filename="package://starbot_description/meshes/stl/lower_leg_nx.stl"/>
+                            <mesh filename="package://starbot_description/meshes/stl/lower_leg_nx.stl" scale = "0.8 0.8 0.8"/>
                         </geometry>
                     </xacro:unless>
@@ -371,5 +371,5 @@
                          <origin xyz="0 -${LOWER_LEG_pos} 0" rpy="0 0 0" />
                         <geometry>
-                            <mesh filename="package://starbot_description/meshes/stl/lower_leg_ny.stl"/>
+                            <mesh filename="package://starbot_description/meshes/stl/lower_leg_ny.stl" scale = "0.8 0.8 0.8"/>
                         </geometry>
                     </xacro:if>
@@ -381,7 +381,7 @@
                         <!-- LF LOWER_LEG -->
                         <inertial>
-                    		<origin xyz="0 ${LOWER_LEG_pos} 0" rpy="0 0 0"/>
+                    		<origin xyz="0 ${CM_XY_LOWER} ${CM_Z_LOWER}" rpy="0 0 1.57"/>
                     		<mass value="2.36"/>
-                    		<inertia ixx="0.00767" ixy="0" ixz="0" iyy="0.00056" iyz="0" izz="0.00767"/>
+                    		<inertia ixx="0.000639" ixy="0" ixz="0" iyy="0.0126" iyz="0" izz="0.0126"/>
                 	</inertial>
                     </xacro:unless>
@@ -389,7 +389,7 @@
                         <!-- RF LOWER_LEG -->
                         <inertial>
-                    		<origin xyz="${LOWER_LEG_pos} 0 0" rpy="0 0 0"/>
+                    		<origin xyz="${CM_XY_LOWER} 0 ${CM_Z_LOWER}" rpy="0 0 0"/>
                     		<mass value="2.36"/>
-                    		<inertia ixx="0.00056" ixy="0" ixz="0" iyy="0.00767" iyz="0" izz="0.00056"/>
+                    		<inertia ixx="0.000639" ixy="0" ixz="0" iyy="0.0126" iyz="0" izz="0.0126"/>
                 	</inertial>
                     </xacro:if>
@@ -399,7 +399,7 @@
                         <!-- LH LOWER_LEG -->
                         <inertial>
-                    		<origin xyz="-${LOWER_LEG_pos} 0 0" rpy="0 0 0"/>
+                    		<origin xyz="-${CM_XY_LOWER} 0 ${CM_Z_LOWER}" rpy="0 0 0"/>
                     		<mass value="2.36"/>
-                    		<inertia ixx="0.00056" ixy="0" ixz="0" iyy="0.00767" iyz="0" izz="0.00056"/>
+                    		<inertia ixx="0.000639" ixy="0" ixz="0" iyy="0.0126" iyz="0" izz="0.0126"/>
                 	</inertial>
                     </xacro:unless>
@@ -407,7 +407,7 @@
                         <!-- RH LOWER_LEG-->
                         <inertial>
-                    		<origin xyz="0 -${LOWER_LEG_pos} 0" rpy="0 0 0"/>
+                    		<origin xyz="0 -${CM_XY_LOWER} ${CM_Z_LOWER}" rpy="0 0 1.57"/>
                     		<mass value="2.36"/>
-                    		<inertia ixx="0.00767" ixy="0" ixz="0" iyy="0.00056" iyz="0" izz="0.00767"/>
+                    		<inertia ixx="0.000639" ixy="0" ixz="0" iyy="0.0126" iyz="0" izz="0.0126"/>
                 	</inertial>
                     </xacro:if>
@@ -494,5 +494,5 @@
                         <!-- LF PRE_WHEEL -->
                         <geometry>
-                            <mesh filename="package://starbot_description/meshes/stl/joint_wheel_y.stl"/>
+                            <mesh filename="package://starbot_description/meshes/stl/joint_wheel_y.stl" scale = "0.8 0.8 0.8"/>
                         </geometry>
                     </xacro:unless>
@@ -500,5 +500,5 @@
                         <!-- RF PRE_WHEEL -->
                         <geometry>
-                            <mesh filename="package://starbot_description/meshes/stl/joint_wheel_x.stl"/>
+                            <mesh filename="package://starbot_description/meshes/stl/joint_wheel_x.stl" scale = "0.8 0.8 0.8"/>
                         </geometry>
                     </xacro:if>
@@ -508,5 +508,5 @@
                         <!-- LH PRE_WHEEL -->
                         <geometry>
-                            <mesh filename="package://starbot_description/meshes/stl/joint_wheel_nx.stl"/>
+                            <mesh filename="package://starbot_description/meshes/stl/joint_wheel_nx.stl" scale = "0.8 0.8 0.8"/>
                         </geometry>
                     </xacro:unless>
@@ -514,5 +514,5 @@
                         <!-- RH PRE_WHEEL-->
                         <geometry>
-                            <mesh filename="package://starbot_description/meshes/stl/joint_wheel_ny.stl"/>
+                            <mesh filename="package://starbot_description/meshes/stl/joint_wheel_ny.stl" scale = "0.8 0.8 0.8"/>
                         </geometry>
                     </xacro:if>
@@ -522,35 +522,35 @@
             <xacro:if value="${is_front}">
                     <xacro:unless value="${is_right}">
-                        <!-- PRE_WHEEL_LEG -->
-                        <inertial>
-                    		<origin xyz="0 ${PRE_WHEEL_pos} 0" rpy="0 0 0"/>
+                        <!-- LF PRE_WHEEL_LEG -->
+                        <inertial>
+                    		<origin xyz="0 ${CM_XY_PRE_WHEEL} ${CM_Z_PRE_WHEEL}" rpy="0 0 1.57"/>
                     		<mass value="0.66"/>
-                    		<inertia ixx="0.00024" ixy="0" ixz="0" iyy="0.00016" iyz="0" izz="0.00024"/>
-                	</inertial>
-                    </xacro:unless>
-                    <xacro:if value="${is_right}">
-                        <!-- PRE_WHEEL_LEG -->
-                        <inertial>
-                    		<origin xyz="${PRE_WHEEL_pos} 0 0" rpy="0 0 0"/>
+                    		<inertia ixx="0.00017674" ixy="0" ixz="0" iyy="0.000358" iyz="0" izz="0.000358"/>
+                	</inertial>
+                    </xacro:unless>
+                    <xacro:if value="${is_right}">
+                        <!-- RF PRE_WHEEL_LEG -->
+                        <inertial>
+                    		<origin xyz="${CM_XY_PRE_WHEEL} 0 ${CM_Z_PRE_WHEEL}" rpy="0 0 0"/>
                     		<mass value="0.66"/>
-                    		<inertia ixx="0.00016" ixy="0" ixz="0" iyy="0.00024" iyz="0" izz="0.00016"/>
-                	</inertial>
-                    </xacro:if>
-                </xacro:if>
-                <xacro:unless value="${is_front}">
-                    <xacro:unless value="${is_right}">
-                        <!-- PRE_WHEEL_LEG -->
-                        <inertial>
-                    		<origin xyz="-${PRE_WHEEL_pos} 0 0" rpy="0 0 0"/>
+                    		<inertia ixx="0.00017674" ixy="0" ixz="0" iyy="0.000358" iyz="0" izz="0.000358"/>
+                	</inertial>
+                    </xacro:if>
+                </xacro:if>
+                <xacro:unless value="${is_front}">
+                    <xacro:unless value="${is_right}">
+                        <!-- LH PRE_WHEEL_LEG -->
+                        <inertial>
+                    		<origin xyz="-${CM_XY_PRE_WHEEL} 0 ${CM_Z_PRE_WHEEL}" rpy="0 0 0"/>
                     		<mass value="0.66"/>
-                    		<inertia ixx="0.00016" ixy="0" ixz="0" iyy="0.00024" iyz="0" izz="0.00016"/>
-                	</inertial>
-                    </xacro:unless>
-                    <xacro:if value="${is_right}">
-                        <!-- PRE_WHEEL_LEG-->
-                        <inertial>
-                    		<origin xyz="0 -${PRE_WHEEL_pos} 0" rpy="0 0 0"/>
+                    		<inertia ixx="0.00017674" ixy="0" ixz="0" iyy="0.000358" iyz="0" izz="0.000358"/>
+                	</inertial>
+                    </xacro:unless>
+                    <xacro:if value="${is_right}">
+                        <!-- RH PRE_WHEEL_LEG-->
+                        <inertial>
+                    		<origin xyz="0 -${CM_XY_PRE_WHEEL} ${CM_Z_PRE_WHEEL}" rpy="0 0 1.57"/>
                     		<mass value="0.66"/>
-                    		<inertia ixx="0.00024" ixy="0" ixz="0" iyy="0.00016" iyz="0" izz="0.00024"/>
+                    		<inertia ixx="0.00017674" ixy="0" ixz="0" iyy="0.000358" iyz="0" izz="0.000358"/>
                 	</inertial>
                     </xacro:if>
@@ -582,5 +582,5 @@
                 </xacro:unless>
                 <xacro:if value="${is_right}">
-                    <!-- RF_WHEEL_JOINT -->
+                    <!-- RH_WHEEL_JOINT -->
                     <axis xyz="-1 0 0"/>
                     <origin xyz="0 -${WHEEL_pos} 0" rpy="0 0 0" />
@@ -662,35 +662,35 @@
             <xacro:if value="${is_front}">
                     <xacro:unless value="${is_right}">
-                        <!-- PRE_WHEEL_LEG -->
-                        <inertial>
-                    		<origin xyz="0 ${WHEEL_pos} 0" rpy="0 0 0"/>
+                        <!--LF WHEEL_LEG -->
+                        <inertial>
+                    		<origin xyz="0 ${CM_XY_WHEEL} ${CM_Z_WHEEL}" rpy="0 0 1.57"/>
                     		<mass value="1.0"/>
-                    		<inertia ixx="0.00224" ixy="0" ixz="0" iyy="0.00121" iyz="0" izz="0.00224"/>
-                	</inertial>
-                    </xacro:unless>
-                    <xacro:if value="${is_right}">
-                        <!-- PRE_WHEEL_LEG -->
-                        <inertial>
-                    		<origin xyz="${WHEEL_pos} 0 0" rpy="0 0 0"/>
+                    		<inertia ixx="0.00177" ixy="0" ixz="0" iyy="0.00326" iyz="0" izz="0.00177"/>
+                	</inertial>
+                    </xacro:unless>
+                    <xacro:if value="${is_right}">
+                        <!--RF WHEEL_LEG -->
+                        <inertial>
+                    		<origin xyz="${CM_XY_WHEEL} 0 ${CM_Z_WHEEL}" rpy="0 0 0"/>
                     		<mass value="1.0"/>
-                    		<inertia ixx="0.00121" ixy="0" ixz="0" iyy="0.00224" iyz="0" izz="0.00121"/>
-                	</inertial>
-                    </xacro:if>
-                </xacro:if>
-                <xacro:unless value="${is_front}">
-                    <xacro:unless value="${is_right}">
-                        <!-- PRE_WHEEL_LEG -->
-                        <inertial>
-                    		<origin xyz="-${WHEEL_pos}  0 0" rpy="0 0 0"/>
+                    		<inertia ixx="0.00177" ixy="0" ixz="0" iyy="0.00326" iyz="0" izz="0.00177"/>
+                	</inertial>
+                    </xacro:if>
+                </xacro:if>
+                <xacro:unless value="${is_front}">
+                    <xacro:unless value="${is_right}">
+                        <!--LH WHEEL_LEG -->
+                        <inertial>
+                    		<origin xyz="-${CM_XY_WHEEL}  0 ${CM_Z_WHEEL}" rpy="0 0 0"/>
                     		<mass value="1.0"/>
-                    		<inertia ixx="0.00121" ixy="0" ixz="0" iyy="0.00224" iyz="0" izz="0.00121"/>
-                	</inertial>
-                    </xacro:unless>
-                    <xacro:if value="${is_right}">
-                        <!-- PRE_WHEEL_LEG-->
-                        <inertial>
-                    		<origin xyz="0 -${WHEEL_pos} 0" rpy="0 0 0"/>
+                    		<inertia ixx="0.00177" ixy="0" ixz="0" iyy="0.00326" iyz="0" izz="0.00177"/>
+                	</inertial>
+                    </xacro:unless>
+                    <xacro:if value="${is_right}">
+                        <!--RH WHEEL_LEG-->
+                        <inertial>
+                    		<origin xyz="0 -${CM_XY_WHEEL} ${CM_Z_WHEEL}" rpy="0 0 1.57"/>
                     		<mass value="1.0"/>
-                    		<inertia ixx="0.00224" ixy="0" ixz="0" iyy="0.00121" iyz="0" izz="0.00224"/>
+                    		<inertia ixx="0.00177" ixy="0" ixz="0" iyy="0.00326" iyz="0" izz="0.00177"/>
                 	</inertial>
                     </xacro:if>
