Commit message: fix collisions

File: robots/starbot.urdf.xacro (robot description, xacro)
@@ -44,5 +44,5 @@
             <origin xyz="0 0 0" rpy="0 0 0" />
             <geometry>
-                <mesh filename="package://starbot_description/meshes/stl/octagon.stl"/>
+                <mesh filename="package://starbot_description/meshes/stl/octagon.stl" scale = "0.8 0.8 0.8" />
             </geometry>
         </collision>

File: urdfs/leg.xacro (robot description, xacro)
@@ -87,5 +87,5 @@
                         <!-- LF_BS -->
                         <geometry>
-                            <mesh filename="package://starbot_description/meshes/stl/shoulder_y.stl" scale = "0.8 0.8 0.8" />
+                            <mesh filename="package://starbot_description/meshes/stl/shoulder_y.stl" />
                         </geometry>
                     </xacro:unless>
@@ -93,5 +93,5 @@
                         <!-- RF_BS -->
                         <geometry>
-                            <mesh filename="package://starbot_description/meshes/stl/shoulder_x.stl" scale = "0.8 0.8 0.8" />
+                            <mesh filename="package://starbot_description/meshes/stl/shoulder_x.stl"/>
                         </geometry>
                     </xacro:if>
@@ -101,5 +101,5 @@
                         <!-- LH_BS -->
                         <geometry>
-                            <mesh filename="package://starbot_description/meshes/stl/shoulder_nx.stl" scale = "0.8 0.8 0.8" />
+                            <mesh filename="package://starbot_description/meshes/stl/shoulder_nx.stl" />
                         </geometry>
                     </xacro:unless>
@@ -107,5 +107,5 @@
                         <!-- RH_BS -->
                         <geometry>
-                            <mesh filename="package://starbot_description/meshes/stl/shoulder_ny.stl" scale = "0.8 0.8 0.8" />
+                            <mesh filename="package://starbot_description/meshes/stl/shoulder_ny.stl" />
                         </geometry>
                     </xacro:if>
@@ -201,5 +201,5 @@
 			<origin xyz="0 ${CM_XY_UPPER} ${CM_Z_UPPER}" rpy="0 0 0" />
                         <geometry>
-                            <mesh filename="package://starbot_description/meshes/stl/upper_leg_y.stl" scale = "0.8 0.8 0.8" />
+                            <mesh filename="package://starbot_description/meshes/stl/upper_leg_y.stl" />
                         </geometry>
                     </xacro:unless>
@@ -208,5 +208,5 @@
        			<origin xyz="${CM_XY_UPPER} 0 ${CM_Z_UPPER}" rpy="0 0 0" />
                         <geometry>
-                            <mesh filename="package://starbot_description/meshes/stl/upper_leg_x.stl" scale = "0.8 0.8 0.8" />
+                            <mesh filename="package://starbot_description/meshes/stl/upper_leg_x.stl" />
                         </geometry>
                     </xacro:if>
@@ -217,5 +217,5 @@
 			<origin xyz="-${CM_XY_UPPER} 0 ${CM_Z_UPPER}" rpy="0 0 0" />
                         <geometry>
-                            <mesh filename="package://starbot_description/meshes/stl/upper_leg_nx.stl" scale = "0.8 0.8 0.8" />
+                            <mesh filename="package://starbot_description/meshes/stl/upper_leg_nx.stl"/>
                         </geometry>
                     </xacro:unless>
@@ -224,5 +224,5 @@
 			<origin xyz="0 -${CM_XY_UPPER} ${CM_Z_UPPER}" rpy="0 0 0" />
                         <geometry>
-                            <mesh filename="package://starbot_description/meshes/stl/upper_leg_ny.stl" scale = "0.8 0.8 0.8" />
+                            <mesh filename="package://starbot_description/meshes/stl/upper_leg_ny.stl"  />
                         </geometry>
                     </xacro:if>
@@ -348,5 +348,5 @@
                          <origin xyz="0 ${LOWER_LEG_pos} 0" rpy="0 0 0" />
                         <geometry>
-                            <mesh filename="package://starbot_description/meshes/stl/lower_leg_y.stl" scale = "0.8 0.8 0.8"/>
+                            <mesh filename="package://starbot_description/meshes/stl/lower_leg_y.stl" />
                         </geometry>
                     </xacro:unless>
@@ -355,5 +355,5 @@
                         <origin xyz="${LOWER_LEG_pos} 0 0" rpy="0 0 0" />
                         <geometry>
-                            <mesh filename="package://starbot_description/meshes/stl/lower_leg_x.stl" scale = "0.8 0.8 0.8" />
+                            <mesh filename="package://starbot_description/meshes/stl/lower_leg_x.stl"/>
                         </geometry>
                     </xacro:if>
@@ -364,5 +364,5 @@
                         <origin xyz="-${LOWER_LEG_pos} 0 0" rpy="0 0 0" />
                         <geometry>
-                            <mesh filename="package://starbot_description/meshes/stl/lower_leg_nx.stl" scale = "0.8 0.8 0.8"/>
+                            <mesh filename="package://starbot_description/meshes/stl/lower_leg_nx.stl" />
                         </geometry>
                     </xacro:unless>
@@ -371,5 +371,5 @@
                          <origin xyz="0 -${LOWER_LEG_pos} 0" rpy="0 0 0" />
                         <geometry>
-                            <mesh filename="package://starbot_description/meshes/stl/lower_leg_ny.stl" scale = "0.8 0.8 0.8"/>
+                            <mesh filename="package://starbot_description/meshes/stl/lower_leg_ny.stl"/>
                         </geometry>
                     </xacro:if>
@@ -494,5 +494,5 @@
                         <!-- LF PRE_WHEEL -->
                         <geometry>
-                            <mesh filename="package://starbot_description/meshes/stl/joint_wheel_y.stl" scale = "0.8 0.8 0.8"/>
+                            <mesh filename="package://starbot_description/meshes/stl/joint_wheel_y.stl"/>
                         </geometry>
                     </xacro:unless>
@@ -500,5 +500,5 @@
                         <!-- RF PRE_WHEEL -->
                         <geometry>
-                            <mesh filename="package://starbot_description/meshes/stl/joint_wheel_x.stl" scale = "0.8 0.8 0.8"/>
+                            <mesh filename="package://starbot_description/meshes/stl/joint_wheel_x.stl"/>
                         </geometry>
                     </xacro:if>
@@ -508,5 +508,5 @@
                         <!-- LH PRE_WHEEL -->
                         <geometry>
-                            <mesh filename="package://starbot_description/meshes/stl/joint_wheel_nx.stl" scale = "0.8 0.8 0.8"/>
+                            <mesh filename="package://starbot_description/meshes/stl/joint_wheel_nx.stl" />
                         </geometry>
                     </xacro:unless>
@@ -514,5 +514,5 @@
                         <!-- RH PRE_WHEEL-->
                         <geometry>
-                            <mesh filename="package://starbot_description/meshes/stl/joint_wheel_ny.stl" scale = "0.8 0.8 0.8"/>
+                            <mesh filename="package://starbot_description/meshes/stl/joint_wheel_ny.stl"/>
                         </geometry>
                     </xacro:if>

Commit message: commented upper leg collision and reduced body size to avoid issues

File: robots/starbot.urdf.xacro (robot description, xacro)
@@ -35,5 +35,5 @@
         <origin xyz="0 0 0" rpy="0 0 0"/>
         <geometry>
-           <mesh filename="package://starbot_description/meshes/stl/octagon.stl"/>
+           <mesh filename="package://starbot_description/meshes/stl/octagon.stl" scale = "0.7 0.7 0.7"/>
         </geometry>
         <material name="yellow">
@@ -44,5 +44,5 @@
             <origin xyz="0 0 0" rpy="0 0 0" />
             <geometry>
-                <mesh filename="package://starbot_description/meshes/stl/octagon.stl" scale = "0.8 0.8 0.8" />
+                <mesh filename="package://starbot_description/meshes/stl/octagon.stl" scale = "0.7 0.7 0.7" />
             </geometry>
         </collision>

File: urdfs/leg.xacro (robot description, xacro)
@@ -80,36 +80,4 @@
                 <material name="orange"/>
             </visual>
-            <!--COLLISION-->
-            <collision>
-                <origin xyz="0 0 0" rpy="0 0 0" />
-                <xacro:if value="${is_front}">
-                    <xacro:unless value="${is_right}">
-                        <!-- LF_BS -->
-                        <geometry>
-                            <mesh filename="package://starbot_description/meshes/stl/shoulder_y.stl" />
-                        </geometry>
-                    </xacro:unless>
-                    <xacro:if value="${is_right}">
-                        <!-- RF_BS -->
-                        <geometry>
-                            <mesh filename="package://starbot_description/meshes/stl/shoulder_x.stl"/>
-                        </geometry>
-                    </xacro:if>
-                </xacro:if>
-                <xacro:unless value="${is_front}">
-                    <xacro:unless value="${is_right}">
-                        <!-- LH_BS -->
-                        <geometry>
-                            <mesh filename="package://starbot_description/meshes/stl/shoulder_nx.stl" />
-                        </geometry>
-                    </xacro:unless>
-                    <xacro:if value="${is_right}">
-                        <!-- RH_BS -->
-                        <geometry>
-                            <mesh filename="package://starbot_description/meshes/stl/shoulder_ny.stl" />
-                        </geometry>
-                    </xacro:if>
-                </xacro:unless>
-            </collision>
             <!--INERTIAL -->
             <inertial>
@@ -195,44 +163,44 @@
             </visual>
             <!--COLLISION-->
-            <collision>
-                <xacro:if value="${is_front}">
+            <!--<collision>
+                <xacro:if value="${is_front}">
+                    <xacro:unless value="${is_right}">
+                        &lt;!&ndash; LF UPPER_LEG &ndash;&gt;
+			            <origin xyz="0 ${UPPER_LEG_pos} 0" rpy="0 0 0" />
+                        <geometry>
+                            <mesh filename="package://starbot_description/meshes/stl/upper_leg_y.stl" />
+                        </geometry>
+                    </xacro:unless>
+                    <xacro:if value="${is_right}">
+                        &lt;!&ndash; RF UPPER_LEG &ndash;&gt;
+       			        <origin xyz="${UPPER_LEG_pos} 0 0" rpy="0 0 0" />
+                        <geometry>
+                            <mesh filename="package://starbot_description/meshes/stl/upper_leg_x.stl" />
+                        </geometry>
+                    </xacro:if>
+                </xacro:if>
+                <xacro:unless value="${is_front}">
+                    <xacro:unless value="${is_right}">
+                        &lt;!&ndash; LH UPPER_LEG &ndash;&gt;
+			            <origin xyz="-${UPPER_LEG_pos} 0 0" rpy="0 0 0" />
+                        <geometry>
+                            <mesh filename="package://starbot_description/meshes/stl/upper_leg_nx.stl"/>
+                        </geometry>
+                    </xacro:unless>
+                    <xacro:if value="${is_right}">
+                        &lt;!&ndash; RH UPPER_LEG&ndash;&gt;
+			            <origin xyz="0 -${UPPER_LEG_pos} 0" rpy="0 0 0" />
+                        <geometry>
+                            <mesh filename="package://starbot_description/meshes/stl/upper_leg_ny.stl"  />
+                        </geometry>
+                    </xacro:if>
+                </xacro:unless>
+            </collision>-->
+            <!-- UPPER LEG LINK INERTIAL -->
+            <xacro:if value="${is_front}">
                     <xacro:unless value="${is_right}">
                         <!-- LF UPPER_LEG -->
-			<origin xyz="0 ${CM_XY_UPPER} ${CM_Z_UPPER}" rpy="0 0 0" />
-                        <geometry>
-                            <mesh filename="package://starbot_description/meshes/stl/upper_leg_y.stl" />
-                        </geometry>
-                    </xacro:unless>
-                    <xacro:if value="${is_right}">
-                        <!-- RF UPPER_LEG -->
-       			<origin xyz="${CM_XY_UPPER} 0 ${CM_Z_UPPER}" rpy="0 0 0" />
-                        <geometry>
-                            <mesh filename="package://starbot_description/meshes/stl/upper_leg_x.stl" />
-                        </geometry>
-                    </xacro:if>
-                </xacro:if>
-                <xacro:unless value="${is_front}">
-                    <xacro:unless value="${is_right}">
-                        <!-- LH UPPER_LEG -->
-			<origin xyz="-${CM_XY_UPPER} 0 ${CM_Z_UPPER}" rpy="0 0 0" />
-                        <geometry>
-                            <mesh filename="package://starbot_description/meshes/stl/upper_leg_nx.stl"/>
-                        </geometry>
-                    </xacro:unless>
-                    <xacro:if value="${is_right}">
-                        <!-- RH UPPER_LEG-->
-			<origin xyz="0 -${CM_XY_UPPER} ${CM_Z_UPPER}" rpy="0 0 0" />
-                        <geometry>
-                            <mesh filename="package://starbot_description/meshes/stl/upper_leg_ny.stl"  />
-                        </geometry>
-                    </xacro:if>
-                </xacro:unless>
-            </collision>
-            <!-- UPPER LEG LINK INERTIAL -->
-            <xacro:if value="${is_front}">
-                    <xacro:unless value="${is_right}">
-                        <!-- LF UPPER_LEG -->
-                        <inertial>
-                    		<origin xyz="0 ${UPPER_LEG_pos} 0" rpy="0 0 1.57"/>
+                        <inertial>
+                    		<origin xyz="0 ${CM_XY_UPPER} ${CM_Z_UPPER}" rpy="0 0 1.57"/>
                     		<mass value="2.3"/>
                     		<inertia ixx="0.001878" ixy="0" ixz="0" iyy="0.0182" iyz="0" izz="0.0182"/>
@@ -242,5 +210,5 @@
                         <!-- RF UPPER_LEG -->
                         <inertial>
-                    		<origin xyz="${UPPER_LEG_pos} 0 0" rpy="0 0 0"/>
+                    		<origin xyz="${CM_XY_UPPER} 0 ${CM_Z_UPPER}" rpy="0 0 0"/>
                     		<mass value="2.3"/>
                     		<inertia ixx="0.001878" ixy="0" ixz="0" iyy="0.0182" iyz="0" izz="0.0182"/>
@@ -252,5 +220,5 @@
                         <!-- LH UPPER_LEG -->
                         <inertial>
-                    		<origin xyz="-${UPPER_LEG_pos} 0 0" rpy="0 0 0"/>
+                    		<origin xyz="-${CM_XY_UPPER} 0 ${CM_Z_UPPER}" rpy="0 0 0"/>
                     		<mass value="2.3"/>
                     		<inertia ixx="0.001878" ixy="0" ixz="0" iyy="0.0182" iyz="0" izz="0.0182"/>
@@ -260,5 +228,5 @@
                         <!-- RH UPPER_LEG-->
                         <inertial>
-                    		<origin xyz="0 -${UPPER_LEG_pos} 0" rpy="0 0 1.57"/>
+                    		<origin xyz="0 -${CM_XY_UPPER} ${CM_Z_UPPER}" rpy="0 0 1.57"/>
                     		<mass value="2.3"/>
                     		<inertia ixx="0.001878" ixy="0" ixz="0" iyy="0.0182" iyz="0" izz="0.0182"/>

Commit message: reduced base link mass to 10 kg to make orientation control work, changed joint definition to match the pinocchio leg definition

File: robots/starbot.urdf.xacro (robot description, xacro)
@@ -29,5 +29,5 @@
         <inertial>
         <origin xyz="0 0 0" rpy="0 0 0"/>
-        <mass value="20.0"/>
+        <mass value="10.0"/>
         <inertia ixx="0.1956" ixy="0" ixz="0" iyy="0.1956" iyz="0" izz="0.2579"/>
       </inertial>

Commit message: finally fixing the hack of new_gazebo_version to set root joint for pinocchio as per robot_control commit fccb58b1fb819f6c18701ba5d1a20bd6d21af330

File: robots/starbot.urdf.xacro (robot description, xacro)
@@ -3,5 +3,4 @@
     <!--- new_gazebo_version should be false by default because pinocchio needs it!-->
     <xacro:arg name="robot_name" default="starbot"/>
-    <xacro:arg name="new_gazebo_version" default="false"/>
     <xacro:include filename="$(find starbot_description)/gazebo/gazebo.urdf.xacro">
         <xacro:arg name="task_period" value="$(arg task_period)"/>
@@ -9,15 +8,4 @@
     </xacro:include>
     <xacro:include filename="$(find starbot_description)/urdfs/leg.xacro"/>
-    <!-- BASE LINK -->
-    <!-- floating type is supported in older versions of Gazebo. In new Gazebo if a link has no parent, it is supposed to be attached to a floating joint -->
-    <xacro:unless value="$(arg new_gazebo_version)">
-        <!-- Floating-base Joint -->
-        <link name="world"/>
-        <joint name="floating_base_joint" type="floating" >
-            <origin rpy="0 0 0" xyz="0 0 0"/>
-            <parent link="world"/>
-            <child link="base_link"/>
-        </joint>
-    </xacro:unless>
     <link name="base_link" />
     <joint name="floating_base" type="fixed">
